File: midnight-sun-2019/midnight-sun-2019.kicad_pcb (KiCad board)
At the start: 2 copper layers, 8 parts, among them J1 Conn_01x02, J2 USB_A, U1 74HC14, U2 74HC86, U3 74HC595, U4 74HC595, U5 74HC595

Commit message: WIP: schematic
Parts:
- removed C1: C, Capacitor_THT:CP_Radial_D4.0mm_P1.50mm
- removed J1: Conn_01x02, Connector_PinSocket_2.54mm:PinSocket_1x02_P2.54mm_Vertical
- removed J2: USB_A, electrokit:USB_Micro-B_Electrokit_anr41011019
- removed U1: 74HC14, Package_DIP:DIP-14_W7.62mm_Socket
- removed U2: 74HC86, Package_DIP:DIP-14_W7.62mm_Socket
- removed U3, U4, U5: 74HC595, Package_DIP:DIP-16_W7.62mm_Socket
- added C101: C, Capacitor_THT:CP_Radial_D5.0mm_P2.00mm, F.Cu at (193.6, 35.6)
- added C102: C, Capacitor_THT:CP_Radial_D5.0mm_P2.00mm, F.Cu at (236.2, 35.6)
- added D101: LED, LED_SMD:LED_0805_2012Metric_Castellated, F.Cu at (167.3, 22.9)
- added D102: LED, LED_SMD:LED_0805_2012Metric_Castellated, F.Cu at (207.0, 23.8)
- added D103: LED, LED_SMD:LED_0805_2012Metric_Castellated, F.Cu at (248.9, 23.8)
- added D104: LED, LED_SMD:LED_0805_2012Metric_Castellated, F.Cu at (232.1, 101.6)
- added D105: LED, LED_SMD:LED_0805_2012Metric_Castellated, F.Cu at (232.7, 132.1)
- added D106: LED, LED_SMD:LED_0805_2012Metric_Castellated, F.Cu at (216.8, 129.5)
- added D107: LED, LED_SMD:LED_0805_2012Metric_Castellated, F.Cu at (216.8, 132.1)
- added D108: LED, LED_SMD:LED_0805_2012Metric_Castellated, F.Cu at (216.8, 134.6)
- added D109: LED, LED_SMD:LED_0805_2012Metric_Castellated, F.Cu at (216.8, 137.2)
- added D110: LED, LED_SMD:LED_0805_2012Metric_Castellated, F.Cu at (216.8, 139.7)
- added D111: LED, LED_SMD:LED_0805_2012Metric_Castellated, F.Cu at (216.8, 142.2)
- added D112: LED, LED_SMD:LED_0805_2012Metric_Castellated, F.Cu at (216.8, 144.8)
- added D113: LED, LED_SMD:LED_0805_2012Metric_Castellated, F.Cu at (232.7, 157.5)
- added D114: LED, LED_SMD:LED_0805_2012Metric_Castellated, F.Cu at (216.8, 154.9)
- added D115: LED, LED_SMD:LED_0805_2012Metric_Castellated, F.Cu at (216.8, 157.5)
- added D116: LED, LED_SMD:LED_0805_2012Metric_Castellated, F.Cu at (216.8, 160.0)
- added D117: LED, LED_SMD:LED_0805_2012Metric_Castellated, F.Cu at (216.8, 162.6)
- added D118: LED, LED_SMD:LED_0805_2012Metric_Castellated, F.Cu at (216.8, 165.1)
- added D119: LED, LED_SMD:LED_0805_2012Metric_Castellated, F.Cu at (216.8, 167.6)
- added D120: LED, LED_SMD:LED_0805_2012Metric_Castellated, F.Cu at (216.8, 170.2)
- added D201: LED, LED_SMD:LED_0805_2012Metric_Castellated, F.Cu at (71.1, 116.9)
- added D202: LED, LED_SMD:LED_0805_2012Metric_Castellated, F.Cu at (95.4, 93.4)
- added D203: LED, LED_SMD:LED_0805_2012Metric_Castellated, F.Cu at (105.1, 84.6)
- added D204: LED, LED_SMD:LED_0805_2012Metric_Castellated, F.Cu at (109.9, 93.4)
- added D205: LED, LED_SMD:LED_0805_2012Metric_Castellated, F.Cu at (114.8, 108.1)
- added D206: LED, LED_SMD:LED_0805_2012Metric_Castellated, F.Cu at (100.2, 122.8)
- added D207: LED, LED_SMD:LED_0805_2012Metric_Castellated, F.Cu at (119.6, 102.2)
- added D208: LED, LED_SMD:LED_0805_2012Metric_Castellated, F.Cu at (90.5, 131.6)
- added D209: LED, LED_SMD:LED_0805_2012Metric_Castellated, F.Cu at (105.1, 116.9)
- added D210: LED, LED_SMD:LED_0805_2012Metric_Castellated, F.Cu at (129.3, 93.4)
- added D211: LED, LED_SMD:LED_0805_2012Metric_Castellated, F.Cu at (124.5, 96.3)
- added D212: LED, LED_SMD:LED_0805_2012Metric_Castellated, F.Cu at (95.4, 125.7)
- added D213: LED, LED_SMD:LED_0805_2012Metric_Castellated, F.Cu at (56.6, 131.6)
- added D214: LED, LED_SMD:LED_0805_2012Metric_Castellated, F.Cu at (80.8, 140.4)
- added D215: LED, LED_SMD:LED_0805_2012Metric_Castellated, F.Cu at (109.9, 111.0)
- added D216: LED, LED_SMD:LED_0805_2012Metric_Castellated, F.Cu at (95.4, 122.8)
- added D217: LED, LED_SMD:LED_0805_2012Metric_Castellated, F.Cu at (85.7, 134.5)
- added D218: LED, LED_SMD:LED_0805_2012Metric_Castellated, F.Cu at (129.3, 90.4)
- added D219: LED, LED_SMD:LED_0805_2012Metric_Castellated, F.Cu at (105.1, 114.0)
- added D220: LED, LED_SMD:LED_0805_2012Metric_Castellated, F.Cu at (76.0, 143.4)
- added D221: LED, LED_SMD:LED_0805_2012Metric_Castellated, F.Cu at (90.5, 128.7)
- added D222: LED, LED_SMD:LED_0805_2012Metric_Castellated, F.Cu at (119.6, 99.3)
- added D223: LED, LED_SMD:LED_0805_2012Metric_Castellated, F.Cu at (114.8, 105.1)
- added D224: LED, LED_SMD:LED_0805_2012Metric_Castellated, F.Cu at (37.2, 125.7)
- added D225: LED, LED_SMD:LED_0805_2012Metric_Castellated, F.Cu at (27.5, 87.5)
- added D226: LED, LED_SMD:LED_0805_2012Metric_Castellated, F.Cu at (32.3, 84.6)
- added D227: LED, LED_SMD:LED_0805_2012Metric_Castellated, F.Cu at (22.6, 93.4)
- added D228: LED, LED_SMD:LED_0805_2012Metric_Castellated, F.Cu at (37.2, 81.6)
- added D229: LED, LED_SMD:LED_0805_2012Metric_Castellated, F.Cu at (27.5, 90.4)
- added D230: LED, LED_SMD:LED_0805_2012Metric_Castellated, F.Cu at (32.3, 87.5)
- added D231: LED, LED_SMD:LED_0805_2012Metric_Castellated, F.Cu at (22.6, 96.3)
- added D232: LED, LED_SMD:LED_0805_2012Metric_Castellated, F.Cu at (22.6, 81.6)
- added D233: LED, LED_SMD:LED_0805_2012Metric_Castellated, F.Cu at (27.5, 93.4)
- added D234: LED, LED_SMD:LED_0805_2012Metric_Castellated, F.Cu at (42.0, 81.6)
- added D235: LED, LED_SMD:LED_0805_2012Metric_Castellated, F.Cu at (22.6, 99.3)
- added D236: LED, LED_SMD:LED_0805_2012Metric_Castellated, F.Cu at (32.3, 90.4)
- added D237: LED, LED_SMD:LED_0805_2012Metric_Castellated, F.Cu at (37.2, 87.5)
- added D238: LED, LED_SMD:LED_0805_2012Metric_Castellated, F.Cu at (46.9, 105.1)
- added D239: LED, LED_SMD:LED_0805_2012Metric_Castellated, F.Cu at (42.0, 84.6)
- added D240: LED, LED_SMD:LED_0805_2012Metric_Castellated, F.Cu at (32.3, 93.4)
- added D241: LED, LED_SMD:LED_0805_2012Metric_Castellated, F.Cu at (22.6, 102.2)
- added D242: LED, LED_SMD:LED_0805_2012Metric_Castellated, F.Cu at (46.9, 81.6)
- added D243: LED, LED_SMD:LED_0805_2012Metric_Castellated, F.Cu at (22.6, 105.1)
- added D244: LED, LED_SMD:LED_0805_2012Metric_Castellated, F.Cu at (27.5, 99.3)
- added D245: LED, LED_SMD:LED_0805_2012Metric_Castellated, F.Cu at (37.2, 90.4)
- added D246: LED, LED_SMD:LED_0805_2012Metric_Castellated, F.Cu at (42.0, 93.4)
- added D247: LED, LED_SMD:LED_0805_2012Metric_Castellated, F.Cu at (56.6, 93.4)
- added D248: LED, LED_SMD:LED_0805_2012Metric_Castellated, F.Cu at (32.3, 116.9)
- added D249: LED, LED_SMD:LED_0805_2012Metric_Castellated, F.Cu at (46.9, 102.2)
- added D250: LED, LED_SMD:LED_0805_2012Metric_Castellated, F.Cu at (27.5, 122.8)
- added D251: LED, LED_SMD:LED_0805_2012Metric_Castellated, F.Cu at (42.0, 108.1)
- added D252: LED, LED_SMD:LED_0805_2012Metric_Castellated, F.Cu at (71.1, 81.6)
- added D253: LED, LED_SMD:LED_0805_2012Metric_Castellated, F.Cu at (27.5, 96.3)
- added D254: LED, LED_SMD:LED_0805_2012Metric_Castellated, F.Cu at (51.7, 81.6)
- added D255: LED, LED_SMD:LED_0805_2012Metric_Castellated, F.Cu at (27.5, 105.1)
- added D256: LED, LED_SMD:LED_0805_2012Metric_Castellated, F.Cu at (32.3, 99.3)
- added D257: LED, LED_SMD:LED_0805_2012Metric_Castellated, F.Cu at (42.0, 90.4)
- added D258: LED, LED_SMD:LED_0805_2012Metric_Castellated, F.Cu at (46.9, 87.5)
- added D259: LED, LED_SMD:LED_0805_2012Metric_Castellated, F.Cu at (22.6, 111.0)
- added D260: LED, LED_SMD:LED_0805_2012Metric_Castellated, F.Cu at (37.2, 96.3)
- added D261: LED, LED_SMD:LED_0805_2012Metric_Castellated, F.Cu at (51.7, 84.6)
- added D262: LED, LED_SMD:LED_0805_2012Metric_Castellated, F.Cu at (42.0, 87.5)
- added D263: LED, LED_SMD:LED_0805_2012Metric_Castellated, F.Cu at (32.3, 102.2)
- added D264: LED, LED_SMD:LED_0805_2012Metric_Castellated, F.Cu at (27.5, 108.1)
- added D265: LED, LED_SMD:LED_0805_2012Metric_Castellated, F.Cu at (56.6, 81.6)
- added D266: LED, LED_SMD:LED_0805_2012Metric_Castellated, F.Cu at (32.3, 105.1)
- added D267: LED, LED_SMD:LED_0805_2012Metric_Castellated, F.Cu at (22.6, 90.4)
- added D268: LED, LED_SMD:LED_0805_2012Metric_Castellated, F.Cu at (22.6, 114.0)
- added D269: LED, LED_SMD:LED_0805_2012Metric_Castellated, F.Cu at (46.9, 90.4)
- added D270: LED, LED_SMD:LED_0805_2012Metric_Castellated, F.Cu at (51.7, 87.5)
- added D271: LED, LED_SMD:LED_0805_2012Metric_Castellated, F.Cu at (27.5, 111.0)
- added D272: LED, LED_SMD:LED_0805_2012Metric_Castellated, F.Cu at (42.0, 96.3)
- added D273: LED, LED_SMD:LED_0805_2012Metric_Castellated, F.Cu at (56.6, 84.6)
- added D274: LED, LED_SMD:LED_0805_2012Metric_Castellated, F.Cu at (46.9, 93.4)
- added D275: LED, LED_SMD:LED_0805_2012Metric_Castellated, F.Cu at (37.2, 84.6)
- added D276: LED, LED_SMD:LED_0805_2012Metric_Castellated, F.Cu at (22.6, 84.6)
- added D277: LED, LED_SMD:LED_0805_2012Metric_Castellated, F.Cu at (27.5, 81.6)
- added D278: LED, LED_SMD:LED_0805_2012Metric_Castellated, F.Cu at (22.6, 87.5)
- added D279: LED, LED_SMD:LED_0805_2012Metric_Castellated, F.Cu at (27.5, 84.6)
- added D280: LED, LED_SMD:LED_0805_2012Metric_Castellated, F.Cu at (32.3, 81.6)
- added D281: LED, LED_SMD:LED_0805_2012Metric_Castellated, F.Cu at (51.7, 102.2)
- added D282: LED, LED_SMD:LED_0805_2012Metric_Castellated, F.Cu at (32.3, 111.0)
- added D283: LED, LED_SMD:LED_0805_2012Metric_Castellated, F.Cu at (46.9, 96.3)
- added D284: LED, LED_SMD:LED_0805_2012Metric_Castellated, F.Cu at (61.4, 84.6)
- added D285: LED, LED_SMD:LED_0805_2012Metric_Castellated, F.Cu at (51.7, 93.4)
- added D286: LED, LED_SMD:LED_0805_2012Metric_Castellated, F.Cu at (22.6, 116.9)
- added D287: LED, LED_SMD:LED_0805_2012Metric_Castellated, F.Cu at (42.0, 102.2)
- added D288: LED, LED_SMD:LED_0805_2012Metric_Castellated, F.Cu at (22.6, 122.8)
- added D289: LED, LED_SMD:LED_0805_2012Metric_Castellated, F.Cu at (37.2, 108.1)
- added D290: LED, LED_SMD:LED_0805_2012Metric_Castellated, F.Cu at (66.3, 81.6)
- added D291: LED, LED_SMD:LED_0805_2012Metric_Castellated, F.Cu at (42.0, 105.1)
- added D292: LED, LED_SMD:LED_0805_2012Metric_Castellated, F.Cu at (27.5, 119.8)
- added D293: LED, LED_SMD:LED_0805_2012Metric_Castellated, F.Cu at (46.9, 99.3)
- added D294: LED, LED_SMD:LED_0805_2012Metric_Castellated, F.Cu at (32.3, 114.0)
- added D295: LED, LED_SMD:LED_0805_2012Metric_Castellated, F.Cu at (109.9, 105.1)
- added D296: LED, LED_SMD:LED_0805_2012Metric_Castellated, F.Cu at (61.4, 87.5)
- added D297: LED, LED_SMD:LED_0805_2012Metric_Castellated, F.Cu at (37.2, 111.0)
- added D298: LED, LED_SMD:LED_0805_2012Metric_Castellated, F.Cu at (22.6, 125.7)
- added D299: LED, LED_SMD:LED_0805_2012Metric_Castellated, F.Cu at (51.7, 96.3)
- added D300: LED, LED_SMD:LED_0805_2012Metric_Castellated, F.Cu at (85.7, 93.4)
- added D301: LED, LED_SMD:LED_0805_2012Metric_Castellated, F.Cu at (114.8, 96.3)
- added D302: LED, LED_SMD:LED_0805_2012Metric_Castellated, F.Cu at (129.3, 84.6)
- added D303: LED, LED_SMD:LED_0805_2012Metric_Castellated, F.Cu at (119.6, 93.4)
- added D304: LED, LED_SMD:LED_0805_2012Metric_Castellated, F.Cu at (95.4, 116.9)
- added D305: LED, LED_SMD:LED_0805_2012Metric_Castellated, F.Cu at (80.8, 131.6)
- added D306: LED, LED_SMD:LED_0805_2012Metric_Castellated, F.Cu at (109.9, 102.2)
- added D307: LED, LED_SMD:LED_0805_2012Metric_Castellated, F.Cu at (90.5, 122.8)
- added D308: LED, LED_SMD:LED_0805_2012Metric_Castellated, F.Cu at (76.0, 137.5)
- added D309: LED, LED_SMD:LED_0805_2012Metric_Castellated, F.Cu at (105.1, 108.1)
- added D310: LED, LED_SMD:LED_0805_2012Metric_Castellated, F.Cu at (56.6, 90.4)
- added D311: LED, LED_SMD:LED_0805_2012Metric_Castellated, F.Cu at (32.3, 119.8)
- added D312: LED, LED_SMD:LED_0805_2012Metric_Castellated, F.Cu at (51.7, 99.3)
- added D313: LED, LED_SMD:LED_0805_2012Metric_Castellated, F.Cu at (22.6, 128.7)
- added D314: LED, LED_SMD:LED_0805_2012Metric_Castellated, F.Cu at (37.2, 114.0)
- added D315: LED, LED_SMD:LED_0805_2012Metric_Castellated, F.Cu at (61.4, 90.4)
- added D316: LED, LED_SMD:LED_0805_2012Metric_Castellated, F.Cu at (66.3, 87.5)
- added D317: LED, LED_SMD:LED_0805_2012Metric_Castellated, F.Cu at (66.3, 84.6)
- added D318: LED, LED_SMD:LED_0805_2012Metric_Castellated, F.Cu at (27.5, 125.7)
- added D319: LED, LED_SMD:LED_0805_2012Metric_Castellated, F.Cu at (56.6, 96.3)
- added D320: LED, LED_SMD:LED_0805_2012Metric_Castellated, F.Cu at (71.1, 84.6)
- added D321: LED, LED_SMD:LED_0805_2012Metric_Castellated, F.Cu at (61.4, 93.4)
- added D322: LED, LED_SMD:LED_0805_2012Metric_Castellated, F.Cu at (37.2, 116.9)
- added D323: LED, LED_SMD:LED_0805_2012Metric_Castellated, F.Cu at (22.6, 131.6)
- added D324: LED, LED_SMD:LED_0805_2012Metric_Castellated, F.Cu at (56.6, 87.5)
- added D325: LED, LED_SMD:LED_0805_2012Metric_Castellated, F.Cu at (32.3, 122.8)
- added D326: LED, LED_SMD:LED_0805_2012Metric_Castellated, F.Cu at (46.9, 108.1)
- added D327: LED, LED_SMD:LED_0805_2012Metric_Castellated, F.Cu at (76.0, 81.6)
- added D328: LED, LED_SMD:LED_0805_2012Metric_Castellated, F.Cu at (51.7, 105.1)
- added D329: LED, LED_SMD:LED_0805_2012Metric_Castellated, F.Cu at (22.6, 134.5)
- added D330: LED, LED_SMD:LED_0805_2012Metric_Castellated, F.Cu at (27.5, 116.9)
- added D331: LED, LED_SMD:LED_0805_2012Metric_Castellated, F.Cu at (37.2, 102.2)
- added D332: LED, LED_SMD:LED_0805_2012Metric_Castellated, F.Cu at (32.3, 108.1)
- added D333: LED, LED_SMD:LED_0805_2012Metric_Castellated, F.Cu at (61.4, 81.6)
- added D334: LED, LED_SMD:LED_0805_2012Metric_Castellated, F.Cu at (37.2, 105.1)
- added D335: LED, LED_SMD:LED_0805_2012Metric_Castellated, F.Cu at (22.6, 119.8)
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Routing:
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- added copper zone on B.Cu, net GND
- added copper zone on F.Cu, net VCC
Other:
- copper layers 2 -> 4

Commit message: Wire up all the logic
Parts:
- added C103: 10 uF, Capacitor_THT:CP_Radial_D5.0mm_P2.00mm, F.Cu at (274.3, 29.2)
- added D324: LED, LED_SMD:LED_0805_2012Metric_Castellated, F.Cu at (64.2, 43.9)
- added D325: LED, LED_SMD:LED_0805_2012Metric_Castellated, F.Cu at (78.7, 38.1)
- added D326: LED, LED_SMD:LED_0805_2012Metric_Castellated, F.Cu at (73.9, 41.0)
- added D327: LED, LED_SMD:LED_0805_2012Metric_Castellated, F.Cu at (64.2, 32.2)
- added D328: LED, LED_SMD:LED_0805_2012Metric_Castellated, F.Cu at (69.0, 43.9)
- added D329: LED, LED_SMD:LED_0805_2012Metric_Castellated, F.Cu at (78.7, 35.1)
- added D330: LED, LED_SMD:LED_0805_2012Metric_Castellated, F.Cu at (64.2, 46.9)
- added D331: LED, LED_SMD:LED_0805_2012Metric_Castellated, F.Cu at (73.9, 38.1)
- added D332: LED, LED_SMD:LED_0805_2012Metric_Castellated, F.Cu at (69.0, 41.0)
- added D333: LED, LED_SMD:LED_0805_2012Metric_Castellated, F.Cu at (78.7, 32.2)
- added D334: LED, LED_SMD:LED_0805_2012Metric_Castellated, F.Cu at (69.0, 46.9)
- added D335: LED, LED_SMD:LED_0805_2012Metric_Castellated, F.Cu at (73.9, 35.1)
- added D336: LED, LED_SMD:LED_0805_2012Metric_Castellated, F.Cu at (69.0, 38.1)
- added D337: LED, LED_SMD:LED_0805_2012Metric_Castellated, F.Cu at (64.2, 41.0)
- added D338: LED, LED_SMD:LED_0805_2012Metric_Castellated, F.Cu at (73.9, 32.2)
- added D339: LED, LED_SMD:LED_0805_2012Metric_Castellated, F.Cu at (69.0, 35.1)
- added D340: LED, LED_SMD:LED_0805_2012Metric_Castellated, F.Cu at (64.2, 38.1)
- added D341: LED, LED_SMD:LED_0805_2012Metric_Castellated, F.Cu at (69.0, 32.2)
- added D342: LED, LED_SMD:LED_0805_2012Metric_Castellated, F.Cu at (64.2, 35.1)
- added D343: LED, LED_SMD:LED_0805_2012Metric_Castellated, F.Cu at (78.7, 41.0)
- added D344: LED, LED_SMD:LED_0805_2012Metric_Castellated, F.Cu at (83.6, 32.2)
- added D345: LED, LED_SMD:LED_0805_2012Metric_Castellated, F.Cu at (88.4, 32.2)
- added D346: LED, LED_SMD:LED_0805_2012Metric_Castellated, F.Cu at (73.9, 43.9)
- added D347: LED, LED_SMD:LED_0805_2012Metric_Castellated, F.Cu at (83.6, 35.1)
- added J103: USB_B_Micro, electrokit:USB_Micro-B_Electrokit_anr41011019, F.Cu at (248.9, 180.3)
- added R212: R, Resistor_SMD:R_0805_2012Metric_Pad1.15x1.40mm_HandSolder, F.Cu at (88.3, 38.1)
- added R213: R, Resistor_SMD:R_0805_2012Metric_Pad1.15x1.40mm_HandSolder, F.Cu at (78.6, 46.9)
- added R214: R, Resistor_SMD:R_0805_2012Metric_Pad1.15x1.40mm_HandSolder, F.Cu at (83.5, 41.0)
- added R215: R, Resistor_SMD:R_0805_2012Metric_Pad1.15x1.40mm_HandSolder, F.Cu at (93.2, 32.2)
- added R216: R, Resistor_SMD:R_0805_2012Metric_Pad1.15x1.40mm_HandSolder, F.Cu at (78.7, 44.0)
- added R217: R, Resistor_SMD:R_0805_2012Metric_Pad1.15x1.40mm_HandSolder, F.Cu at (88.4, 35.1)
- added R218: R, Resistor_SMD:R_0805_2012Metric_Pad1.15x1.40mm_HandSolder, F.Cu at (73.8, 46.9)
- added R219: R, Resistor_SMD:R_0805_2012Metric_Pad1.15x1.40mm_HandSolder, F.Cu at (83.5, 38.1)
- added U116: 74HC14, Package_DIP:DIP-14_W7.62mm_Socket, F.Cu at (152.4, 172.7)
- C101: value C -> 100 nF; footprint Capacitor_THT:CP_Radial_D5.0mm_P2.00mm -> Capacitor_THT:C_Disc_D7.5mm_W2.5mm_P5.00mm
- C102: value C -> 10 uF
- D101, D103: footprint LED_SMD:LED_0805_2012Metric_Castellated -> LED_THT:LED_D5.0mm
- D102: footprint LED_SMD:LED_0805_2012Metric_Castellated -> LED_THT:LED_D5.0mm_Clear
- J102: value USB_B_Micro -> Conn_01x02; footprint electrokit:USB_Micro-B_Electrokit_anr41011019 -> Connector_PinHeader_2.54mm:PinHeader_1x02_P2.54mm_Vertical
- R101, R104, R105: value R -> 10k
- R102, R103: value R -> 1k
- SW101: footprint Button_Switch_THT:SW_CuK_JS202011CQN_DPDT_Straight -> electrokit:SW_SPDT_MTS-102-A2
- SW102, SW103: value SW_Push -> SW_SPDT; footprint Button_Switch_THT:SW_DIP_SPSTx03_Slide_9.78x9.8mm_W7.62mm_P2.54mm -> electrokit:SW_PUSH_DPDT_CW_Industries_GPBS850L
- U113: value 74HC14 -> 74HC86
- U115: value 74HC86 -> 74HC14
- moved U110 172.9 mm to (167.6, 27.9)
- moved D201 170.3 mm to (-91.4, 66.1)
- moved D202 170.3 mm to (-67.2, 42.6)
- moved D203 170.3 mm to (-57.5, 33.8)
- moved D204 170.3 mm to (-52.6, 42.6)
- moved D205 170.3 mm to (-47.8, 57.3)
- moved D206 170.3 mm to (-62.3, 72.0)
- moved D207 170.3 mm to (-42.9, 51.4)
- moved D208 170.3 mm to (-72.0, 80.8)
- moved D209 170.3 mm to (-57.5, 66.1)
- moved D210 170.3 mm to (-33.2, 42.6)
- moved D211 170.3 mm to (-38.1, 45.5)
- moved D212 170.3 mm to (-67.2, 74.9)
- moved D213 170.3 mm to (-106.0, 80.8)
- moved D214 170.3 mm to (-81.7, 89.6)
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- renumbered D324 to D348, D325 to D349, D326 to D350, D327 to D351, D328 to D352, D329 to D353, D330 to D354, D331 to D355, D332 to D356, D333 to D357, D334 to D358, D335 to D359, D336 to D360, D337 to D361, D338 to D362, D339 to D363, D340 to D364, D341 to D365, D342 to D366, D343 to D367, D344 to D368, D345 to D369, D346 to D370, D347 to D371, D348 to D372, D349 to D373, D350 to D374, D351 to D375, D352 to D376, D353 to D377, D354 to D378, D355 to D379, D356 to D380, D357 to D381, D358 to D382, D359 to D383, D360 to D384, D361 to D385, D362 to D386, D363 to D387, D364 to D388, D365 to D389, D366 to D390, D367 to D391, D368 to D392, D369 to D393, D370 to D394, D371 to D395, D372 to D396, D373 to D397, D374 to D398, D375 to D399, D376 to D400, D377 to D401, D378 to D402, D379 to D403, D380 to D404, D381 to D405, D382 to D406, D383 to D407, D384 to D408, D385 to D409, D386 to D410, D387 to D411, D388 to D412, D389 to D413, D390 to D414, D391 to D415, D392 to D416, D393 to D417, D394 to D418, D395 to D419, D396 to D420, D397 to D421, D398 to D422, D399 to D423, D400 to D424, D401 to D425, D402 to D426, D403 to D427, D404 to D428, D405 to D429, D406 to D430, D407 to D431, D408 to D432, D409 to D433, D410 to D434, D411 to D435, D412 to D436, D413 to D437, D414 to D438, D415 to D439, D416 to D440, D417 to D441, D418 to D442, D419 to D443, D420 to D444, D421 to D445, D422 to D446, D423 to D447, D424 to D448, D425 to D449, D426 to D450, D427 to D451, D428 to D452, D429 to D453, D430 to D454, D431 to D455, D432 to D456, D433 to D457, D434 to D458, D435 to D459, D436 to D460, D437 to D461, D438 to D462, D439 to D463, D440 to D464, D441 to D465, D442 to D466, D443 to D467, D444 to D468, D445 to D469, D446 to D470, D447 to D471, D448 to D472, D449 to D473, D450 to D474, D451 to D475, D452 to D476, D453 to D477, D454 to D478, D455 to D479, D456 to D480, D457 to D481, D458 to D482, D459 to D483, D460 to D484, D461 to D485, D462 to D486, D463 to D487, D464 to D488, D465 to D489, D466 to D490, D467 to D491, D468 to D492, D469 to D493, D470 to D494, D471 to D495, D472 to D496, D473 to D497, D474 to D498, D475 to D499, D476 to D500, D477 to D501, D478 to D502, D479 to D503, D480 to D504, D481 to D505, D482 to D506, D483 to D507, D484 to D508, D485 to D509, D486 to D510, D487 to D511, D488 to D512, D489 to D513, D490 to D514, D491 to D515, D492 to D516, D493 to D517, D494 to D518, D495 to D519, D496 to D520, D497 to D521, D498 to D522, D499 to D523, D500 to D524, D501 to D525, D502 to D526, D503 to D527, D504 to D528, D505 to D529, D506 to D530, D507 to D531, D508 to D532, D509 to D533, D510 to D534, D511 to D535, D512 to D536, D513 to D537, D514 to D538, D515 to D539, D516 to D540, D517 to D541, D518 to D542, D519 to D543, D520 to D544, D521 to D545, D522 to D546, D523 to D547, D524 to D548, D525 to D549, D526 to D550, D527 to D551, D528 to D552, D529 to D553, D530 to D554, D531 to D555, D532 to D556, D533 to D557, D534 to D558, D535 to D559, D536 to D560, D537 to D561, D538 to D562, D539 to D563, D540 to D564, D541 to D565, D542 to D566, D543 to D567, D544 to D568, D545 to D569, D546 to D570, D547 to D571, D548 to D572, D549 to D573, D550 to D574, D551 to D575, D552 to D576, D553 to D577, D554 to D578, D555 to D579, D556 to D580, D557 to D581, D558 to D582, D559 to D583, D560 to D584, D561 to D585, D562 to D586, D563 to D587, D564 to D588, D565 to D589, D566 to D590, D567 to D591, D568 to D592, D569 to D593, D570 to D594, D571 to D595, D572 to D596, D573 to D597, D574 to D598, D575 to D599, D576 to D600, D577 to D601, D578 to D602, D579 to D603, D580 to D604, D581 to D605, D582 to D606, D583 to D607, D584 to D608, D585 to D609, D586 to D610, D587 to D611, D588 to D612, D589 to D613, D590 to D614, D591 to D615, D592 to D616, D593 to D617, D594 to D618, D595 to D619, D596 to D620, D597 to D621, D598 to D622, D599 to D623, D600 to D624, D601 to D625, D602 to D626, D603 to D627, D604 to D628, D605 to D629, D606 to D630, D607 to D631, D608 to D632, D609 to D633, D610 to D634, D611 to D635, D612 to D636, D613 to D637, R212 to R220, R213 to R221, R214 to R222, R215 to R223, R216 to R224, R217 to R225, R218 to R226, R219 to R227, R220 to R228, R221 to R229, R222 to R230, R223 to R231, R224 to R232, R225 to R233, R226 to R234, R227 to R235
Connections:
- C101 pad 2: Net-(C101-Pad2) -> VCC
- C102 pad 1: GND -> Net-(C102-Pad1)
- C102 pad 2: Net-(C102-Pad2) -> GND
- J102 pad 1: VCC -> GND
- J102 pad 2: Net-(J102-Pad2) -> VCC
- R102 pad 1: Net-(C101-Pad2) -> Net-(C102-Pad1)
- R103 pad 1: Net-(C102-Pad2) -> Net-(C103-Pad1)
- SW102 pad 3: (no net) -> VCC
- SW103 pad 3: (no net) -> VCC
- U101 pad 1: Net-(C101-Pad2) -> Net-(C102-Pad1)
- U101 pad 14: VCC -> (no net)
- U101 pad 3: Net-(C102-Pad2) -> Net-(C103-Pad1)
- U101 pad 7: GND -> (no net)
- U105 pad 14: VCC -> (no net)
- U105 pad 7: GND -> (no net)
- U106 pad 14: VCC -> (no net)
- U106 pad 7: GND -> (no net)
- U107 pad 14: VCC -> (no net)
- U107 pad 7: GND -> (no net)
- U108 pad 14: VCC -> (no net)
- U108 pad 7: GND -> (no net)
- U109 pad 14: VCC -> (no net)
- U109 pad 7: GND -> (no net)
- U110 pad 10: /z1 -> Net-(U110-Pad10)
- U110 pad 14: VCC -> (no net)
- U110 pad 7: GND -> (no net)
- U110 pad 8: /z0 -> Net-(U110-Pad8)
- U111 pad 1: /b9 -> /b12
- U111 pad 10: /h3 -> /h6
- U111 pad 11: Net-(U111-Pad11) -> /o3
- U111 pad 12: /b14 -> /b12
- U111 pad 13: /h4 -> /h7
- U111 pad 14: VCC -> (no net)
- U111 pad 2: /h6 -> /h5
- U111 pad 3: Net-(U110-Pad9) -> /o0
- U111 pad 4: /b15 -> /b14
- U111 pad 5: /h4 -> /h3
- U111 pad 6: Net-(U110-Pad11) -> /o1
- U111 pad 7: GND -> (no net)
- U111 pad 8: Net-(U111-Pad8) -> /o2
- U111 pad 9: /b12 -> /b9
- U112 pad 1: /b13 -> /b12
- U112 pad 10: /h7 -> /h1
- U112 pad 11: Net-(U112-Pad11) -> /o7
- U112 pad 12: /b14 -> /b11
- U112 pad 13: /h3 -> /h1
- U112 pad 14: VCC -> (no net)
- U112 pad 2: /h4 -> /h3
- U112 pad 3: Net-(U112-Pad3) -> /o4
- U112 pad 4: /b10 -> /b15
- U112 pad 5: /h0 -> /h6
- U112 pad 6: Net-(U112-Pad6) -> /o5
- U112 pad 7: GND -> (no net)
- U112 pad 8: Net-(U112-Pad8) -> /o6
- U113 pad 1: Net-(U111-Pad8) -> /b9
- U113 pad 10: /z6 -> /h3
- U113 pad 11: Net-(U112-Pad8) -> Net-(U113-Pad11)
- U113 pad 12: /z7 -> /b14
- U113 pad 13: Net-(U112-Pad11) -> /h4
- U113 pad 14: VCC -> (no net)
- U113 pad 2: /z2 -> /h6
- U113 pad 3: Net-(U111-Pad11) -> Net-(U113-Pad3)
- U113 pad 4: /z3 -> /b15
- U113 pad 5: Net-(U112-Pad3) -> /h4
- U113 pad 6: /z4 -> Net-(U113-Pad6)
- U113 pad 7: GND -> (no net)
- U113 pad 8: /z5 -> Net-(U113-Pad8)
- U113 pad 9: Net-(U112-Pad6) -> /b12
- U114 pad 1: /b12 -> /b13
- U114 pad 10: /h6 -> /h7
- U114 pad 11: /o3 -> Net-(U114-Pad11)
- U114 pad 12: /b12 -> /b14
- U114 pad 13: /h7 -> /h3
- U114 pad 14: VCC -> (no net)
- U114 pad 2: /h5 -> /h4
- U114 pad 3: /o0 -> Net-(U114-Pad3)
- U114 pad 4: /b14 -> /b10
- U114 pad 5: /h3 -> /h0
- U114 pad 6: /o1 -> Net-(U114-Pad6)
- U114 pad 7: GND -> (no net)
- U114 pad 8: /o2 -> Net-(U114-Pad8)
- U114 pad 9: /b9 -> /b8
- U115 pad 1: /b12 -> Net-(U113-Pad8)
- U115 pad 10: /h1 -> Net-(U115-Pad10)
- U115 pad 11: /o7 -> Net-(U115-Pad11)
- U115 pad 12: /b11 -> Net-(U115-Pad12)
- U115 pad 13: /h1 -> Net-(U115-Pad13)
- U115 pad 14: VCC -> (no net)
- U115 pad 2: /h3 -> /z2
- U115 pad 3: /o4 -> Net-(U113-Pad6)
- U115 pad 4: /b15 -> /z1
- U115 pad 5: /h6 -> Net-(U113-Pad3)
- U115 pad 6: /o5 -> /z0
- U115 pad 7: GND -> (no net)
- U115 pad 8: /o6 -> /z3
- U115 pad 9: /b8 -> Net-(U113-Pad11)
Routing:
- net /h3: track 21.0 -> 386.6 mm, vias 1 -> 14
- net /h4: track 27.8 -> 368.6 mm, vias 1 -> 13
- net /b14: track 35.5 -> 359.0 mm, vias 1 -> 9
- net /b12: track 40.4 -> 351.7 mm, vias 1 -> 11
- net /h6: track 32.9 -> 313.6 mm, vias 1 -> 9
- net /b9: track 16.5 -> 292.8 mm, vias 1 -> 6
- net /b15: track 39.3 -> 301.4 mm, vias 1 -> 6
- net /b8: track 16.5 -> 272.7 mm, vias 1 -> 6
- net /b13: track 25.3 -> 275.4 mm, vias 1 -> 4
- net /b10: track 16.5 -> 266.2 mm, vias 1 -> 5
- net /h0: track 34.8 -> 273.1 mm, vias 1 -> 9
- net /h7: track 41.8 -> 275.1 mm, vias 1 -> 9
- net /b11: track 16.5 -> 236.7 mm, vias 1 -> 5
- net /h1: track 16.5 -> 223.4 mm, vias 1 -> 9
- net /h5: track 29.7 -> 186.5 mm, vias 1 -> 5
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Other:
- board text added: ""Crazy Circuit Conundrum" Midnight Sun CtF 2019 finals"
- board text added: "Design: Emil Lundberg emil@emlun.se"

Commit message: Experiment with rearranging ICs
Parts:
- moved U111 101.6 mm to (111.8, 116.8)
- moved U112 69.1 mm to (111.8, 157.5)
Routing:
- net /o3: track 106.4 -> 212.7 mm
- net /o2: track 91.1 -> 182.2 mm
- net /o0: track 84.8 -> 169.5 mm
- net /o1: track 78.4 -> 156.8 mm
- net /b12: track 351.7 -> 397.4 mm, vias 11 -> 13
- net /h3: track 386.6 -> 427.2 mm, vias 14 -> 16

Commit message: Update QR code to real flag
Parts:
- added D638: LED, LED_SMD:LED_0805_2012Metric_Castellated, F.Cu at (-19.1, 18.4)
- added D639: LED, LED_SMD:LED_0805_2012Metric_Castellated, F.Cu at (-19.1, 21.4)
- added D640: LED, LED_SMD:LED_0805_2012Metric_Castellated, F.Cu at (-14.2, 18.4)
- added D641: LED, LED_SMD:LED_0805_2012Metric_Castellated, F.Cu at (-14.2, 21.4)
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Connections:
- D369 pad 2: Net-(D369-Pad2) -> Net-(D348-Pad2)
- D370 pad 2: Net-(D369-Pad2) -> Net-(D370-Pad2)
- D371 pad 2: Net-(D369-Pad2) -> Net-(D370-Pad2)
- D372 pad 2: Net-(D369-Pad2) -> Net-(D370-Pad2)
- D373 pad 2: Net-(D369-Pad2) -> Net-(D370-Pad2)
- D374 pad 2: Net-(D369-Pad2) -> Net-(D370-Pad2)
- D375 pad 2: Net-(D369-Pad2) -> Net-(D370-Pad2)
- D376 pad 2: Net-(D369-Pad2) -> Net-(D370-Pad2)
- D377 pad 2: Net-(D369-Pad2) -> Net-(D370-Pad2)
- D378 pad 2: Net-(D369-Pad2) -> Net-(D370-Pad2)
- D379 pad 2: Net-(D369-Pad2) -> Net-(D370-Pad2)
- D380 pad 2: Net-(D369-Pad2) -> Net-(D370-Pad2)
- D381 pad 2: Net-(D369-Pad2) -> Net-(D370-Pad2)
- D382 pad 2: Net-(D369-Pad2) -> Net-(D370-Pad2)
- D383 pad 2: Net-(D369-Pad2) -> Net-(D370-Pad2)
- D384 pad 2: Net-(D369-Pad2) -> Net-(D370-Pad2)
- D385 pad 2: Net-(D369-Pad2) -> Net-(D370-Pad2)
- D386 pad 2: Net-(D369-Pad2) -> Net-(D370-Pad2)
- D387 pad 2: Net-(D369-Pad2) -> Net-(D370-Pad2)
- D388 pad 2: Net-(D369-Pad2) -> Net-(D370-Pad2)
- D389 pad 2: Net-(D389-Pad2) -> Net-(D370-Pad2)
- D390 pad 2: Net-(D389-Pad2) -> Net-(D370-Pad2)
- D391 pad 2: Net-(D389-Pad2) -> Net-(D370-Pad2)
- D392 pad 2: Net-(D389-Pad2) -> Net-(D392-Pad2)
- D393 pad 2: Net-(D389-Pad2) -> Net-(D392-Pad2)
- D394 pad 2: Net-(D389-Pad2) -> Net-(D392-Pad2)
- D395 pad 2: Net-(D389-Pad2) -> Net-(D392-Pad2)
- D396 pad 2: Net-(D389-Pad2) -> Net-(D392-Pad2)
- D397 pad 2: Net-(D389-Pad2) -> Net-(D392-Pad2)
- D398 pad 2: Net-(D389-Pad2) -> Net-(D392-Pad2)
- D399 pad 2: Net-(D389-Pad2) -> Net-(D392-Pad2)
- D400 pad 2: Net-(D389-Pad2) -> Net-(D392-Pad2)
- D401 pad 2: Net-(D389-Pad2) -> Net-(D392-Pad2)
- D402 pad 2: Net-(D389-Pad2) -> Net-(D392-Pad2)
- D403 pad 2: Net-(D389-Pad2) -> Net-(D392-Pad2)
- D404 pad 2: Net-(D389-Pad2) -> Net-(D392-Pad2)
- D405 pad 2: Net-(D389-Pad2) -> Net-(D392-Pad2)
- D406 pad 2: Net-(D389-Pad2) -> Net-(D392-Pad2)
- D407 pad 2: Net-(D389-Pad2) -> Net-(D392-Pad2)
- D408 pad 2: Net-(D389-Pad2) -> Net-(D392-Pad2)
- D409 pad 2: Net-(D409-Pad2) -> Net-(D392-Pad2)
- D410 pad 2: Net-(D409-Pad2) -> Net-(D392-Pad2)
- D411 pad 2: Net-(D409-Pad2) -> Net-(D392-Pad2)
- D412 pad 2: Net-(D409-Pad2) -> Net-(D392-Pad2)
- D413 pad 2: Net-(D409-Pad2) -> Net-(D392-Pad2)
- D414 pad 2: Net-(D409-Pad2) -> Net-(D414-Pad2)
- D415 pad 2: Net-(D409-Pad2) -> Net-(D414-Pad2)
- D416 pad 2: Net-(D409-Pad2) -> Net-(D414-Pad2)
- D417 pad 2: Net-(D409-Pad2) -> Net-(D414-Pad2)
- D418 pad 2: Net-(D409-Pad2) -> Net-(D414-Pad2)
- D419 pad 2: Net-(D409-Pad2) -> Net-(D414-Pad2)
- D420 pad 2: Net-(D409-Pad2) -> Net-(D414-Pad2)
- D421 pad 2: Net-(D409-Pad2) -> Net-(D414-Pad2)
- D422 pad 2: Net-(D409-Pad2) -> Net-(D414-Pad2)
- D423 pad 2: Net-(D409-Pad2) -> Net-(D414-Pad2)
- D424 pad 2: Net-(D409-Pad2) -> Net-(D414-Pad2)
- D425 pad 2: Net-(D409-Pad2) -> Net-(D414-Pad2)
- D426 pad 2: Net-(D409-Pad2) -> Net-(D414-Pad2)
- D427 pad 2: Net-(D409-Pad2) -> Net-(D414-Pad2)
- D428 pad 2: Net-(D409-Pad2) -> Net-(D414-Pad2)
- D429 pad 2: Net-(D429-Pad2) -> Net-(D414-Pad2)
- D430 pad 2: Net-(D429-Pad2) -> Net-(D414-Pad2)
- D431 pad 2: Net-(D429-Pad2) -> Net-(D414-Pad2)
- D432 pad 2: Net-(D429-Pad2) -> Net-(D414-Pad2)
- D433 pad 2: Net-(D429-Pad2) -> Net-(D414-Pad2)
- D434 pad 2: Net-(D429-Pad2) -> Net-(D414-Pad2)
- D435 pad 2: Net-(D429-Pad2) -> Net-(D435-Pad2)
- D436 pad 2: Net-(D429-Pad2) -> Net-(D435-Pad2)
- D437 pad 2: Net-(D429-Pad2) -> Net-(D435-Pad2)
- D438 pad 2: Net-(D429-Pad2) -> Net-(D435-Pad2)
- D439 pad 2: Net-(D429-Pad2) -> Net-(D435-Pad2)
- D440 pad 2: Net-(D429-Pad2) -> Net-(D435-Pad2)
- D441 pad 2: Net-(D429-Pad2) -> Net-(D435-Pad2)
- D442 pad 2: Net-(D429-Pad2) -> Net-(D435-Pad2)
- D443 pad 2: Net-(D429-Pad2) -> Net-(D435-Pad2)
- D444 pad 2: Net-(D429-Pad2) -> Net-(D435-Pad2)
- D445 pad 2: Net-(D429-Pad2) -> Net-(D435-Pad2)
- D446 pad 2: Net-(D429-Pad2) -> Net-(D435-Pad2)
- D447 pad 2: Net-(D429-Pad2) -> Net-(D435-Pad2)
- D448 pad 2: Net-(D429-Pad2) -> Net-(D435-Pad2)
- D449 pad 2: Net-(D449-Pad2) -> Net-(D435-Pad2)
- D450 pad 2: Net-(D449-Pad2) -> Net-(D435-Pad2)
- D451 pad 2: Net-(D449-Pad2) -> Net-(D435-Pad2)
- D452 pad 2: Net-(D449-Pad2) -> Net-(D435-Pad2)
- D453 pad 2: Net-(D449-Pad2) -> Net-(D435-Pad2)
- D454 pad 2: Net-(D449-Pad2) -> Net-(D435-Pad2)
- D455 pad 2: Net-(D449-Pad2) -> Net-(D435-Pad2)
- D456 pad 2: Net-(D449-Pad2) -> Net-(D456-Pad2)
- D457 pad 2: Net-(D449-Pad2) -> Net-(D456-Pad2)
- D458 pad 2: Net-(D449-Pad2) -> Net-(D456-Pad2)
- D459 pad 2: Net-(D449-Pad2) -> Net-(D456-Pad2)
- D460 pad 2: Net-(D449-Pad2) -> Net-(D456-Pad2)
- D461 pad 2: Net-(D449-Pad2) -> Net-(D456-Pad2)
- D462 pad 2: Net-(D449-Pad2) -> Net-(D456-Pad2)
- D463 pad 2: Net-(D449-Pad2) -> Net-(D456-Pad2)
- D464 pad 2: Net-(D449-Pad2) -> Net-(D456-Pad2)
- D465 pad 2: Net-(D449-Pad2) -> Net-(D456-Pad2)
- D466 pad 2: Net-(D449-Pad2) -> Net-(D456-Pad2)
- D467 pad 2: Net-(D449-Pad2) -> Net-(D456-Pad2)
- D468 pad 2: Net-(D449-Pad2) -> Net-(D456-Pad2)
- D469 pad 2: Net-(D469-Pad2) -> Net-(D456-Pad2)
- D470 pad 2: Net-(D469-Pad2) -> Net-(D456-Pad2)
- D471 pad 2: Net-(D469-Pad2) -> Net-(D456-Pad2)
- D472 pad 2: Net-(D469-Pad2) -> Net-(D456-Pad2)
- D473 pad 2: Net-(D469-Pad2) -> Net-(D456-Pad2)
- D474 pad 2: Net-(D469-Pad2) -> Net-(D456-Pad2)
- D475 pad 2: Net-(D469-Pad2) -> Net-(D456-Pad2)
- D476 pad 2: Net-(D469-Pad2) -> Net-(D456-Pad2)
- D477 pad 2: Net-(D469-Pad2) -> Net-(D477-Pad2)
- D478 pad 2: Net-(D469-Pad2) -> Net-(D477-Pad2)
- D479 pad 2: Net-(D469-Pad2) -> Net-(D477-Pad2)
- D480 pad 2: Net-(D469-Pad2) -> Net-(D477-Pad2)
- D481 pad 2: Net-(D469-Pad2) -> Net-(D477-Pad2)
- D482 pad 2: Net-(D469-Pad2) -> Net-(D477-Pad2)
- D483 pad 2: Net-(D469-Pad2) -> Net-(D477-Pad2)
- D484 pad 2: Net-(D469-Pad2) -> Net-(D477-Pad2)
- D485 pad 2: Net-(D469-Pad2) -> Net-(D477-Pad2)
- D486 pad 2: Net-(D469-Pad2) -> Net-(D477-Pad2)
- D487 pad 2: Net-(D469-Pad2) -> Net-(D477-Pad2)
- D488 pad 2: Net-(D469-Pad2) -> Net-(D477-Pad2)
- D489 pad 2: Net-(D489-Pad2) -> Net-(D477-Pad2)
- D490 pad 2: Net-(D489-Pad2) -> Net-(D477-Pad2)
- D491 pad 2: Net-(D489-Pad2) -> Net-(D477-Pad2)
- D492 pad 2: Net-(D489-Pad2) -> Net-(D477-Pad2)
- D493 pad 2: Net-(D489-Pad2) -> Net-(D477-Pad2)
- D494 pad 2: Net-(D489-Pad2) -> Net-(D477-Pad2)
- D495 pad 2: Net-(D489-Pad2) -> Net-(D477-Pad2)
- D496 pad 2: Net-(D489-Pad2) -> Net-(D477-Pad2)
- D497 pad 2: Net-(D489-Pad2) -> Net-(D477-Pad2)
- D498 pad 2: Net-(D489-Pad2) -> Net-(D498-Pad2)
- D499 pad 2: Net-(D489-Pad2) -> Net-(D498-Pad2)
- D500 pad 2: Net-(D489-Pad2) -> Net-(D498-Pad2)
- D501 pad 2: Net-(D489-Pad2) -> Net-(D498-Pad2)
- D502 pad 2: Net-(D489-Pad2) -> Net-(D498-Pad2)
- D503 pad 2: Net-(D489-Pad2) -> Net-(D498-Pad2)
- D504 pad 2: Net-(D489-Pad2) -> Net-(D498-Pad2)
- D505 pad 2: Net-(D489-Pad2) -> Net-(D498-Pad2)
- D506 pad 2: Net-(D489-Pad2) -> Net-(D498-Pad2)
- D507 pad 2: Net-(D489-Pad2) -> Net-(D498-Pad2)
- D508 pad 2: Net-(D489-Pad2) -> Net-(D498-Pad2)
- D509 pad 2: Net-(D509-Pad2) -> Net-(D498-Pad2)
- D510 pad 2: Net-(D509-Pad2) -> Net-(D498-Pad2)
- D511 pad 2: Net-(D509-Pad2) -> Net-(D498-Pad2)
- D512 pad 2: Net-(D509-Pad2) -> Net-(D498-Pad2)
- D513 pad 2: Net-(D509-Pad2) -> Net-(D498-Pad2)
- D514 pad 2: Net-(D509-Pad2) -> Net-(D498-Pad2)
- D515 pad 2: Net-(D509-Pad2) -> Net-(D498-Pad2)
- D516 pad 2: Net-(D509-Pad2) -> Net-(D498-Pad2)
- D517 pad 2: Net-(D509-Pad2) -> Net-(D498-Pad2)
- D518 pad 2: Net-(D509-Pad2) -> Net-(D498-Pad2)
- D519 pad 2: Net-(D509-Pad2) -> Net-(D519-Pad2)
- D520 pad 2: Net-(D509-Pad2) -> Net-(D519-Pad2)
- D521 pad 2: Net-(D509-Pad2) -> Net-(D519-Pad2)
- D522 pad 2: Net-(D509-Pad2) -> Net-(D519-Pad2)
- D523 pad 2: Net-(D509-Pad2) -> Net-(D519-Pad2)
- D524 pad 2: Net-(D509-Pad2) -> Net-(D519-Pad2)
- D525 pad 2: Net-(D509-Pad2) -> Net-(D519-Pad2)
- D526 pad 2: Net-(D526-Pad2) -> Net-(D519-Pad2)
- D527 pad 2: Net-(D526-Pad2) -> Net-(D519-Pad2)
- D528 pad 2: Net-(D526-Pad2) -> Net-(D519-Pad2)
- D529 pad 2: Net-(D526-Pad2) -> Net-(D519-Pad2)
- D530 pad 2: Net-(D526-Pad2) -> Net-(D519-Pad2)
- D531 pad 2: Net-(D526-Pad2) -> Net-(D519-Pad2)
- D532 pad 2: Net-(D526-Pad2) -> Net-(D519-Pad2)
- D533 pad 2: Net-(D526-Pad2) -> Net-(D519-Pad2)
- D534 pad 2: Net-(D526-Pad2) -> Net-(D519-Pad2)
- D535 pad 2: Net-(D526-Pad2) -> Net-(D535-Pad2)
- D536 pad 2: Net-(D526-Pad2) -> Net-(D535-Pad2)
- D537 pad 2: Net-(D526-Pad2) -> Net-(D535-Pad2)
- D538 pad 2: Net-(D526-Pad2) -> Net-(D535-Pad2)
- D539 pad 2: Net-(D526-Pad2) -> Net-(D535-Pad2)
- D540 pad 2: Net-(D526-Pad2) -> Net-(D535-Pad2)
- D541 pad 2: Net-(D526-Pad2) -> Net-(D535-Pad2)
- D542 pad 2: Net-(D542-Pad2) -> Net-(D535-Pad2)
- D543 pad 2: Net-(D542-Pad2) -> Net-(D535-Pad2)
- D544 pad 2: Net-(D542-Pad2) -> Net-(D535-Pad2)
- D545 pad 2: Net-(D542-Pad2) -> Net-(D535-Pad2)
- D546 pad 2: Net-(D542-Pad2) -> Net-(D535-Pad2)
- D547 pad 2: Net-(D542-Pad2) -> Net-(D535-Pad2)
- D548 pad 2: Net-(D542-Pad2) -> Net-(D535-Pad2)
- D549 pad 2: Net-(D542-Pad2) -> Net-(D535-Pad2)
- D550 pad 2: Net-(D542-Pad2) -> Net-(D535-Pad2)
- D551 pad 2: Net-(D542-Pad2) -> Net-(D551-Pad2)
- D552 pad 2: Net-(D542-Pad2) -> Net-(D551-Pad2)
- D553 pad 2: Net-(D542-Pad2) -> Net-(D551-Pad2)
- D554 pad 2: Net-(D542-Pad2) -> Net-(D551-Pad2)
- D555 pad 2: Net-(D542-Pad2) -> Net-(D551-Pad2)
- D556 pad 2: Net-(D542-Pad2) -> Net-(D551-Pad2)
- D557 pad 2: Net-(D542-Pad2) -> Net-(D551-Pad2)
- D558 pad 2: Net-(D558-Pad2) -> Net-(D551-Pad2)
- D559 pad 2: Net-(D558-Pad2) -> Net-(D551-Pad2)
- D560 pad 2: Net-(D558-Pad2) -> Net-(D551-Pad2)
- D561 pad 2: Net-(D558-Pad2) -> Net-(D551-Pad2)
- D562 pad 2: Net-(D558-Pad2) -> Net-(D551-Pad2)
- D563 pad 2: Net-(D558-Pad2) -> Net-(D551-Pad2)
- D564 pad 2: Net-(D558-Pad2) -> Net-(D551-Pad2)
- D565 pad 2: Net-(D558-Pad2) -> Net-(D551-Pad2)
- D566 pad 2: Net-(D558-Pad2) -> Net-(D551-Pad2)
- D567 pad 2: Net-(D558-Pad2) -> Net-(D567-Pad2)
- D568 pad 2: Net-(D558-Pad2) -> Net-(D567-Pad2)
- D569 pad 2: Net-(D558-Pad2) -> Net-(D567-Pad2)
- D570 pad 2: Net-(D558-Pad2) -> Net-(D567-Pad2)
- D571 pad 2: Net-(D558-Pad2) -> Net-(D567-Pad2)
- D572 pad 2: Net-(D558-Pad2) -> Net-(D567-Pad2)
- D573 pad 2: Net-(D558-Pad2) -> Net-(D567-Pad2)
- D574 pad 2: Net-(D574-Pad2) -> Net-(D567-Pad2)
- D575 pad 2: Net-(D574-Pad2) -> Net-(D567-Pad2)
- D576 pad 2: Net-(D574-Pad2) -> Net-(D567-Pad2)
- D577 pad 2: Net-(D574-Pad2) -> Net-(D567-Pad2)
- D578 pad 2: Net-(D574-Pad2) -> Net-(D567-Pad2)
- D579 pad 2: Net-(D574-Pad2) -> Net-(D567-Pad2)
- D580 pad 2: Net-(D574-Pad2) -> Net-(D567-Pad2)
- D581 pad 2: Net-(D574-Pad2) -> Net-(D567-Pad2)
- D582 pad 2: Net-(D574-Pad2) -> Net-(D582-Pad2)
- D583 pad 2: Net-(D574-Pad2) -> Net-(D582-Pad2)
- D584 pad 2: Net-(D574-Pad2) -> Net-(D582-Pad2)
- D585 pad 2: Net-(D574-Pad2) -> Net-(D582-Pad2)
- D586 pad 2: Net-(D574-Pad2) -> Net-(D582-Pad2)
- D587 pad 2: Net-(D574-Pad2) -> Net-(D582-Pad2)
- D588 pad 2: Net-(D574-Pad2) -> Net-(D582-Pad2)
- D589 pad 2: Net-(D574-Pad2) -> Net-(D582-Pad2)
- D590 pad 2: Net-(D590-Pad2) -> Net-(D582-Pad2)
- D591 pad 2: Net-(D590-Pad2) -> Net-(D582-Pad2)
- D592 pad 2: Net-(D590-Pad2) -> Net-(D582-Pad2)
- D593 pad 2: Net-(D590-Pad2) -> Net-(D582-Pad2)
- D594 pad 2: Net-(D590-Pad2) -> Net-(D582-Pad2)
- D595 pad 2: Net-(D590-Pad2) -> Net-(D582-Pad2)
- D596 pad 2: Net-(D590-Pad2) -> Net-(D582-Pad2)
- D597 pad 2: Net-(D590-Pad2) -> Net-(D597-Pad2)
- D598 pad 2: Net-(D590-Pad2) -> Net-(D597-Pad2)
- D599 pad 2: Net-(D590-Pad2) -> Net-(D597-Pad2)
- D600 pad 2: Net-(D590-Pad2) -> Net-(D597-Pad2)
- D601 pad 2: Net-(D590-Pad2) -> Net-(D597-Pad2)
- D602 pad 2: Net-(D590-Pad2) -> Net-(D597-Pad2)
- D603 pad 2: Net-(D590-Pad2) -> Net-(D597-Pad2)
- D604 pad 2: Net-(D590-Pad2) -> Net-(D597-Pad2)
- D605 pad 2: Net-(D590-Pad2) -> Net-(D597-Pad2)
- D606 pad 2: Net-(D606-Pad2) -> Net-(D597-Pad2)
- D607 pad 2: Net-(D606-Pad2) -> Net-(D597-Pad2)
- D608 pad 2: Net-(D606-Pad2) -> Net-(D597-Pad2)
- D609 pad 2: Net-(D606-Pad2) -> Net-(D597-Pad2)
- D610 pad 2: Net-(D606-Pad2) -> Net-(D597-Pad2)
- D611 pad 2: Net-(D606-Pad2) -> Net-(D597-Pad2)
- D612 pad 2: Net-(D606-Pad2) -> Net-(D612-Pad2)
- D613 pad 2: Net-(D606-Pad2) -> Net-(D612-Pad2)
- D614 pad 2: Net-(D606-Pad2) -> Net-(D612-Pad2)
- D615 pad 2: Net-(D606-Pad2) -> Net-(D612-Pad2)
- D616 pad 2: Net-(D606-Pad2) -> Net-(D612-Pad2)
- D617 pad 2: Net-(D606-Pad2) -> Net-(D612-Pad2)
- D618 pad 2: Net-(D606-Pad2) -> Net-(D612-Pad2)
- D619 pad 2: Net-(D606-Pad2) -> Net-(D612-Pad2)
- D620 pad 2: Net-(D606-Pad2) -> Net-(D612-Pad2)
- D621 pad 2: Net-(D606-Pad2) -> Net-(D612-Pad2)
- D622 pad 2: Net-(D622-Pad2) -> Net-(D612-Pad2)
- D623 pad 2: Net-(D623-Pad2) -> Net-(D612-Pad2)
- D624 pad 2: Net-(D623-Pad2) -> Net-(D612-Pad2)
- D625 pad 2: Net-(D623-Pad2) -> Net-(D612-Pad2)
- D626 pad 2: Net-(D623-Pad2) -> Net-(D612-Pad2)
- D627 pad 2: Net-(D623-Pad2) -> Net-(D627-Pad2)
- D628 pad 2: Net-(D623-Pad2) -> Net-(D628-Pad2)
- D629 pad 2: Net-(D623-Pad2) -> Net-(D628-Pad2)
- D630 pad 2: Net-(D623-Pad2) -> Net-(D628-Pad2)
- D631 pad 2: Net-(D623-Pad2) -> Net-(D628-Pad2)
- D632 pad 2: Net-(D623-Pad2) -> Net-(D628-Pad2)
- D633 pad 2: Net-(D623-Pad2) -> Net-(D628-Pad2)
- D634 pad 2: Net-(D623-Pad2) -> Net-(D628-Pad2)
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Routing:
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
Commit message: Finish wiring up the logic
Parts:
- moved U112 56.8 mm to (167.6, 147.3)
- moved U111 55.9 mm to (167.6, 116.8)
Routing:
- net /o3: track 114.0 -> 38.1 mm, vias 0 -> 3
- net /o1: track 86.0 -> 17.0 mm, vias 0 -> 1
- net /o0: track 92.4 -> 23.4 mm, vias 0 -> 1
- net /o2: track 98.7 -> 29.7 mm, vias 0 -> 1
- net /h6: track 245.0 -> 307.3 mm, vias 6 -> 9
- net /h5: track 162.3 -> 224.6 mm, vias 4 -> 6
- net /h1: track 203.1 -> 253.9 mm, vias 7 -> 9
- net /b9: track 220.4 -> 262.1 mm, vias 5 -> 7
- net /o6: track 7.62 -> 47.0 mm, vias 0 -> 3
- net /b11: track 229.1 -> 267.2 mm
- net /b15: track 251.9 -> 288.7 mm, vias 5 -> 6
- net /b8: track 291.8 -> 327.3 mm, vias 6 -> 7
- net /h4: track 284.6 -> 254.1 mm, vias 12 -> 11
- net /o7: track 7.62 -> 35.6 mm, vias 0 -> 3
- net /o5: track 7.62 -> 30.5 mm, vias 0 -> 3
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