File: midnight-sun-2019/midnight-sun-2019.kicad_pcb (KiCad board)
At the start: 4 copper layers, 546 parts, among them J101 Conn_01x02, J102 Conn_01x02, J103 USB_B_Micro, SW101 SW_SPDT, SW102 SW_SPDT, SW103 SW_SPDT, U101 74HC14, U102 74HC595, U103 74HC595, U104 74HC595, U105 74HC86, U106 74HC86, U107 74HC86, U108 74HC86, U109 74HC14, U110 74HC14, U111 74HC86, U112 74HC86, U113 74HC86, U114 74HC86, U115 74HC14, U116 74HC14

Commit message: Swap positions of LEDs and Rs in matrix
Connections:
- D201 pad 1: GND -> Net-(D201-Pad1)
- D201 pad 2: Net-(D201-Pad2) -> /a0
- D202 pad 1: GND -> Net-(D201-Pad1)
- D202 pad 2: Net-(D201-Pad2) -> /a0
- D203 pad 1: GND -> Net-(D201-Pad1)
- D203 pad 2: Net-(D201-Pad2) -> /a0
- D204 pad 1: GND -> Net-(D201-Pad1)
- D204 pad 2: Net-(D201-Pad2) -> /a0
- D205 pad 1: GND -> Net-(D201-Pad1)
- D205 pad 2: Net-(D201-Pad2) -> /a0
- D206 pad 1: GND -> Net-(D201-Pad1)
- D206 pad 2: Net-(D201-Pad2) -> /a0
- D207 pad 1: GND -> Net-(D201-Pad1)
- D207 pad 2: Net-(D201-Pad2) -> /a0
- D208 pad 1: GND -> Net-(D201-Pad1)
- D208 pad 2: Net-(D201-Pad2) -> /a0
- D209 pad 1: GND -> Net-(D201-Pad1)
- D209 pad 2: Net-(D201-Pad2) -> /a0
- D210 pad 1: GND -> Net-(D201-Pad1)
- D210 pad 2: Net-(D201-Pad2) -> /a0
- D211 pad 1: GND -> Net-(D201-Pad1)
- D211 pad 2: Net-(D201-Pad2) -> /a0
- D212 pad 1: GND -> Net-(D201-Pad1)
- D212 pad 2: Net-(D201-Pad2) -> /a0
- D213 pad 1: GND -> Net-(D201-Pad1)
- D213 pad 2: Net-(D201-Pad2) -> /a0
- D214 pad 1: GND -> Net-(D201-Pad1)
- D214 pad 2: Net-(D201-Pad2) -> /a0
- D215 pad 1: GND -> Net-(D201-Pad1)
- D215 pad 2: Net-(D201-Pad2) -> /a0
- D216 pad 1: GND -> Net-(D201-Pad1)
- D216 pad 2: Net-(D201-Pad2) -> /a0
- D217 pad 1: GND -> Net-(D201-Pad1)
- D217 pad 2: Net-(D201-Pad2) -> /a0
- D218 pad 1: GND -> Net-(D201-Pad1)
- D218 pad 2: Net-(D201-Pad2) -> /a0
- D219 pad 1: GND -> Net-(D201-Pad1)
- D219 pad 2: Net-(D201-Pad2) -> /a0
- D220 pad 1: GND -> Net-(D201-Pad1)
- D220 pad 2: Net-(D201-Pad2) -> /a0
- D221 pad 1: GND -> Net-(D201-Pad1)
- D221 pad 2: Net-(D201-Pad2) -> /a0
- D222 pad 1: GND -> Net-(D201-Pad1)
- D222 pad 2: Net-(D201-Pad2) -> /a0
- D223 pad 1: GND -> Net-(D201-Pad1)
- D223 pad 2: Net-(D201-Pad2) -> /a0
- D224 pad 1: GND -> Net-(D201-Pad1)
- D224 pad 2: Net-(D201-Pad2) -> /a0
- D225 pad 1: GND -> Net-(D201-Pad1)
- D225 pad 2: Net-(D201-Pad2) -> /a0
- D226 pad 1: GND -> Net-(D201-Pad1)
- D226 pad 2: Net-(D201-Pad2) -> /a0
- D227 pad 1: GND -> Net-(D201-Pad1)
- D227 pad 2: Net-(D201-Pad2) -> /a0
- D228 pad 1: GND -> Net-(D201-Pad1)
- D228 pad 2: Net-(D201-Pad2) -> /a0
- D229 pad 1: GND -> Net-(D201-Pad1)
- D229 pad 2: Net-(D201-Pad2) -> /a0
- D230 pad 1: GND -> Net-(D201-Pad1)
- D230 pad 2: Net-(D201-Pad2) -> /a0
- D231 pad 1: GND -> Net-(D201-Pad1)
- D231 pad 2: Net-(D201-Pad2) -> /a0
- D232 pad 1: GND -> Net-(D201-Pad1)
- D232 pad 2: Net-(D201-Pad2) -> /a0
- D233 pad 1: GND -> Net-(D201-Pad1)
- D233 pad 2: Net-(D201-Pad2) -> /a0
- D234 pad 1: GND -> Net-(D234-Pad1)
- D234 pad 2: Net-(D234-Pad2) -> /a1
- D235 pad 1: GND -> Net-(D234-Pad1)
- D235 pad 2: Net-(D234-Pad2) -> /a1
- D236 pad 1: GND -> Net-(D234-Pad1)
- D236 pad 2: Net-(D234-Pad2) -> /a1
- D237 pad 1: GND -> Net-(D234-Pad1)
- D237 pad 2: Net-(D234-Pad2) -> /a1
- D238 pad 1: GND -> Net-(D234-Pad1)
- D238 pad 2: Net-(D234-Pad2) -> /a1
- D239 pad 1: GND -> Net-(D234-Pad1)
- D239 pad 2: Net-(D234-Pad2) -> /a1
- D240 pad 1: GND -> Net-(D234-Pad1)
- D240 pad 2: Net-(D234-Pad2) -> /a1
- D241 pad 1: GND -> Net-(D234-Pad1)
- D241 pad 2: Net-(D234-Pad2) -> /a1
- D242 pad 1: GND -> Net-(D234-Pad1)
- D242 pad 2: Net-(D234-Pad2) -> /a1
- D243 pad 1: GND -> Net-(D234-Pad1)
- D243 pad 2: Net-(D234-Pad2) -> /a1
- D244 pad 1: GND -> Net-(D234-Pad1)
- D244 pad 2: Net-(D234-Pad2) -> /a1
- D245 pad 1: GND -> Net-(D234-Pad1)
- D245 pad 2: Net-(D234-Pad2) -> /a1
- D246 pad 1: GND -> Net-(D234-Pad1)
- D246 pad 2: Net-(D234-Pad2) -> /a1
- D247 pad 1: GND -> Net-(D234-Pad1)
- D247 pad 2: Net-(D234-Pad2) -> /a1
- D248 pad 1: GND -> Net-(D234-Pad1)
- D248 pad 2: Net-(D234-Pad2) -> /a1
- D249 pad 1: GND -> Net-(D234-Pad1)
- D249 pad 2: Net-(D234-Pad2) -> /a1
- D250 pad 1: GND -> Net-(D234-Pad1)
- D250 pad 2: Net-(D234-Pad2) -> /a1
- D251 pad 1: GND -> Net-(D234-Pad1)
- D251 pad 2: Net-(D234-Pad2) -> /a1
- D252 pad 1: GND -> Net-(D234-Pad1)
- D252 pad 2: Net-(D234-Pad2) -> /a1
- D253 pad 1: GND -> Net-(D234-Pad1)
- D253 pad 2: Net-(D234-Pad2) -> /a1
- D254 pad 1: GND -> Net-(D234-Pad1)
- D254 pad 2: Net-(D234-Pad2) -> /a1
- D255 pad 1: GND -> Net-(D234-Pad1)
- D255 pad 2: Net-(D234-Pad2) -> /a1
- D256 pad 1: GND -> Net-(D234-Pad1)
- D256 pad 2: Net-(D234-Pad2) -> /a1
- D257 pad 1: GND -> Net-(D234-Pad1)
- D257 pad 2: Net-(D234-Pad2) -> /a1
- D258 pad 1: GND -> Net-(D234-Pad1)
- D258 pad 2: Net-(D234-Pad2) -> /a1
- D259 pad 1: GND -> Net-(D234-Pad1)
- D259 pad 2: Net-(D234-Pad2) -> /a1
- D260 pad 1: GND -> Net-(D234-Pad1)
- D260 pad 2: Net-(D234-Pad2) -> /a1
- D261 pad 1: GND -> Net-(D234-Pad1)
- D261 pad 2: Net-(D234-Pad2) -> /a1
- D262 pad 1: GND -> Net-(D234-Pad1)
- D262 pad 2: Net-(D234-Pad2) -> /a1
- D263 pad 1: GND -> Net-(D234-Pad1)
- D263 pad 2: Net-(D234-Pad2) -> /a1
- D264 pad 1: GND -> Net-(D234-Pad1)
- D264 pad 2: Net-(D234-Pad2) -> /a1
- D265 pad 1: GND -> Net-(D234-Pad1)
- D265 pad 2: Net-(D234-Pad2) -> /a1
- D266 pad 1: GND -> Net-(D234-Pad1)
- D266 pad 2: Net-(D234-Pad2) -> /a1
- D267 pad 1: GND -> Net-(D267-Pad1)
- D267 pad 2: Net-(D267-Pad2) -> /a2
- D268 pad 1: GND -> Net-(D267-Pad1)
- D268 pad 2: Net-(D267-Pad2) -> /a2
- D269 pad 1: GND -> Net-(D267-Pad1)
- D269 pad 2: Net-(D267-Pad2) -> /a2
- D270 pad 1: GND -> Net-(D267-Pad1)
- D270 pad 2: Net-(D267-Pad2) -> /a2
- D271 pad 1: GND -> Net-(D267-Pad1)
- D271 pad 2: Net-(D267-Pad2) -> /a2
- D272 pad 1: GND -> Net-(D267-Pad1)
- D272 pad 2: Net-(D267-Pad2) -> /a2
- D273 pad 1: GND -> Net-(D267-Pad1)
- D273 pad 2: Net-(D267-Pad2) -> /a2
- D274 pad 1: GND -> Net-(D267-Pad1)
- D274 pad 2: Net-(D267-Pad2) -> /a2
- D275 pad 1: GND -> Net-(D267-Pad1)
- D275 pad 2: Net-(D267-Pad2) -> /a2
- D276 pad 1: GND -> Net-(D267-Pad1)
- D276 pad 2: Net-(D267-Pad2) -> /a2
- D277 pad 1: GND -> Net-(D267-Pad1)
- D277 pad 2: Net-(D267-Pad2) -> /a2
- D278 pad 1: GND -> Net-(D267-Pad1)
- D278 pad 2: Net-(D267-Pad2) -> /a2
- D279 pad 1: GND -> Net-(D267-Pad1)
- D279 pad 2: Net-(D267-Pad2) -> /a2
- D280 pad 1: GND -> Net-(D267-Pad1)
- D280 pad 2: Net-(D267-Pad2) -> /a2
- D281 pad 1: GND -> Net-(D267-Pad1)
- D281 pad 2: Net-(D267-Pad2) -> /a2
- D282 pad 1: GND -> Net-(D267-Pad1)
- D282 pad 2: Net-(D267-Pad2) -> /a2
- D283 pad 1: GND -> Net-(D267-Pad1)
- D283 pad 2: Net-(D267-Pad2) -> /a2
- D284 pad 1: GND -> Net-(D267-Pad1)
- D284 pad 2: Net-(D267-Pad2) -> /a2
- D285 pad 1: GND -> Net-(D267-Pad1)
- D285 pad 2: Net-(D267-Pad2) -> /a2
- D286 pad 1: GND -> Net-(D267-Pad1)
- D286 pad 2: Net-(D267-Pad2) -> /a2
- D287 pad 1: GND -> Net-(D267-Pad1)
- D287 pad 2: Net-(D267-Pad2) -> /a2
- D288 pad 1: GND -> Net-(D267-Pad1)
- D288 pad 2: Net-(D267-Pad2) -> /a2
- D289 pad 1: GND -> Net-(D267-Pad1)
- D289 pad 2: Net-(D267-Pad2) -> /a2
- D290 pad 1: GND -> Net-(D267-Pad1)
- D290 pad 2: Net-(D267-Pad2) -> /a2
- D291 pad 1: GND -> Net-(D267-Pad1)
- D291 pad 2: Net-(D267-Pad2) -> /a2
- D292 pad 1: GND -> Net-(D267-Pad1)
- D292 pad 2: Net-(D267-Pad2) -> /a2
- D293 pad 1: GND -> Net-(D267-Pad1)
- D293 pad 2: Net-(D267-Pad2) -> /a2
- D294 pad 1: GND -> Net-(D267-Pad1)
- D294 pad 2: Net-(D267-Pad2) -> /a2
- D295 pad 1: GND -> Net-(D267-Pad1)
- D295 pad 2: Net-(D267-Pad2) -> /a2
- D296 pad 1: GND -> Net-(D267-Pad1)
- D296 pad 2: Net-(D267-Pad2) -> /a2
- D297 pad 1: GND -> Net-(D267-Pad1)
- D297 pad 2: Net-(D267-Pad2) -> /a2
- D298 pad 1: GND -> Net-(D267-Pad1)
- D298 pad 2: Net-(D267-Pad2) -> /a2
- D299 pad 1: GND -> Net-(D267-Pad1)
- D299 pad 2: Net-(D267-Pad2) -> /a2
- D300 pad 1: GND -> Net-(D300-Pad1)
- D300 pad 2: Net-(D300-Pad2) -> /b0
- D301 pad 1: GND -> Net-(D300-Pad1)
- D301 pad 2: Net-(D300-Pad2) -> /b0
- D302 pad 1: GND -> Net-(D300-Pad1)
- D302 pad 2: Net-(D300-Pad2) -> /b0
- D303 pad 1: GND -> Net-(D303-Pad1)
- D303 pad 2: Net-(D303-Pad2) -> /b1
- D304 pad 1: GND -> Net-(D303-Pad1)
- D304 pad 2: Net-(D303-Pad2) -> /b1
- D305 pad 1: GND -> Net-(D303-Pad1)
- D305 pad 2: Net-(D303-Pad2) -> /b1
- D306 pad 1: GND -> Net-(D306-Pad1)
- D306 pad 2: Net-(D306-Pad2) -> /b2
- D307 pad 1: GND -> Net-(D306-Pad1)
- D307 pad 2: Net-(D306-Pad2) -> /b2
- D308 pad 1: GND -> Net-(D306-Pad1)
- D308 pad 2: Net-(D306-Pad2) -> /b2
- D309 pad 1: GND -> Net-(D309-Pad1)
- D309 pad 2: Net-(D309-Pad2) -> /b3
- D310 pad 1: GND -> Net-(D309-Pad1)
- D310 pad 2: Net-(D309-Pad2) -> /b3
- D311 pad 1: GND -> Net-(D309-Pad1)
- D311 pad 2: Net-(D309-Pad2) -> /b3
- D312 pad 1: GND -> Net-(D312-Pad1)
- D312 pad 2: Net-(D312-Pad2) -> /b4
- D313 pad 1: GND -> Net-(D312-Pad1)
- D313 pad 2: Net-(D312-Pad2) -> /b4
- D314 pad 1: GND -> Net-(D312-Pad1)
- D314 pad 2: Net-(D312-Pad2) -> /b4
- D315 pad 1: GND -> Net-(D315-Pad1)
- D315 pad 2: Net-(D315-Pad2) -> /b5
- D316 pad 1: GND -> Net-(D315-Pad1)
- D316 pad 2: Net-(D315-Pad2) -> /b5
- D317 pad 1: GND -> Net-(D315-Pad1)
- D317 pad 2: Net-(D315-Pad2) -> /b5
- D318 pad 1: GND -> Net-(D318-Pad1)
- D318 pad 2: Net-(D318-Pad2) -> /b6
- D319 pad 1: GND -> Net-(D318-Pad1)
- D319 pad 2: Net-(D318-Pad2) -> /b6
- D320 pad 1: GND -> Net-(D318-Pad1)
- D320 pad 2: Net-(D318-Pad2) -> /b6
- D321 pad 1: GND -> Net-(D321-Pad1)
- D321 pad 2: Net-(D321-Pad2) -> /b7
- D322 pad 1: GND -> Net-(D321-Pad1)
- D322 pad 2: Net-(D321-Pad2) -> /b7
- D323 pad 1: GND -> Net-(D321-Pad1)
- D323 pad 2: Net-(D321-Pad2) -> /b7
- D324 pad 1: GND -> Net-(D324-Pad1)
- D324 pad 2: Net-(D324-Pad2) -> /b8
- D325 pad 1: GND -> Net-(D324-Pad1)
- D325 pad 2: Net-(D324-Pad2) -> /b8
- D326 pad 1: GND -> Net-(D324-Pad1)
- D326 pad 2: Net-(D324-Pad2) -> /b8
- D327 pad 1: GND -> Net-(D327-Pad1)
- D327 pad 2: Net-(D327-Pad2) -> /b9
- D328 pad 1: GND -> Net-(D327-Pad1)
- D328 pad 2: Net-(D327-Pad2) -> /b9
- D329 pad 1: GND -> Net-(D327-Pad1)
- D329 pad 2: Net-(D327-Pad2) -> /b9
- D330 pad 1: GND -> Net-(D330-Pad1)
- D330 pad 2: Net-(D330-Pad2) -> /b10
- D331 pad 1: GND -> Net-(D330-Pad1)
- D331 pad 2: Net-(D330-Pad2) -> /b10
- D332 pad 1: GND -> Net-(D330-Pad1)
- D332 pad 2: Net-(D330-Pad2) -> /b10
- D333 pad 1: GND -> Net-(D333-Pad1)
- D333 pad 2: Net-(D333-Pad2) -> /b11
- D334 pad 1: GND -> Net-(D333-Pad1)
- D334 pad 2: Net-(D333-Pad2) -> /b11
- D335 pad 1: GND -> Net-(D333-Pad1)
- D335 pad 2: Net-(D333-Pad2) -> /b11
- D336 pad 1: GND -> Net-(D336-Pad1)
- D336 pad 2: Net-(D336-Pad2) -> /b12
- D337 pad 1: GND -> Net-(D336-Pad1)
- D337 pad 2: Net-(D336-Pad2) -> /b12
- D338 pad 1: GND -> Net-(D336-Pad1)
- D338 pad 2: Net-(D336-Pad2) -> /b12
- D339 pad 1: GND -> Net-(D339-Pad1)
- D339 pad 2: Net-(D339-Pad2) -> /b13
- D340 pad 1: GND -> Net-(D339-Pad1)
- D340 pad 2: Net-(D339-Pad2) -> /b13
- D341 pad 1: GND -> Net-(D339-Pad1)
- D341 pad 2: Net-(D339-Pad2) -> /b13
- D342 pad 1: GND -> Net-(D342-Pad1)
- D342 pad 2: Net-(D342-Pad2) -> /b14
- D343 pad 1: GND -> Net-(D342-Pad1)
- D343 pad 2: Net-(D342-Pad2) -> /b14
- D344 pad 1: GND -> Net-(D342-Pad1)
- D344 pad 2: Net-(D342-Pad2) -> /b14
- D345 pad 1: GND -> Net-(D345-Pad1)
- D345 pad 2: Net-(D345-Pad2) -> /b15
- D346 pad 1: GND -> Net-(D345-Pad1)
- D346 pad 2: Net-(D345-Pad2) -> /b15
- D347 pad 1: GND -> Net-(D345-Pad1)
- D347 pad 2: Net-(D345-Pad2) -> /b15
- D348 pad 1: GND -> Net-(D348-Pad1)
- D348 pad 2: Net-(D348-Pad2) -> /z0
- D349 pad 1: GND -> Net-(D348-Pad1)
- D349 pad 2: Net-(D348-Pad2) -> /z0
- D350 pad 1: GND -> Net-(D348-Pad1)
- D350 pad 2: Net-(D348-Pad2) -> /z0
- D351 pad 1: GND -> Net-(D348-Pad1)
- D351 pad 2: Net-(D348-Pad2) -> /z0
- D352 pad 1: GND -> Net-(D348-Pad1)
- D352 pad 2: Net-(D348-Pad2) -> /z0
- D353 pad 1: GND -> Net-(D348-Pad1)
- D353 pad 2: Net-(D348-Pad2) -> /z0
- D354 pad 1: GND -> Net-(D348-Pad1)
- D354 pad 2: Net-(D348-Pad2) -> /z0
- D355 pad 1: GND -> Net-(D348-Pad1)
- D355 pad 2: Net-(D348-Pad2) -> /z0
- D356 pad 1: GND -> Net-(D348-Pad1)
- D356 pad 2: Net-(D348-Pad2) -> /z0
- D357 pad 1: GND -> Net-(D348-Pad1)
- D357 pad 2: Net-(D348-Pad2) -> /z0
- D358 pad 1: GND -> Net-(D348-Pad1)
- D358 pad 2: Net-(D348-Pad2) -> /z0
- D359 pad 1: GND -> Net-(D348-Pad1)
- D359 pad 2: Net-(D348-Pad2) -> /z0
- D360 pad 1: GND -> Net-(D348-Pad1)
- D360 pad 2: Net-(D348-Pad2) -> /z0
- D361 pad 1: GND -> Net-(D348-Pad1)
- D361 pad 2: Net-(D348-Pad2) -> /z0
- D362 pad 1: GND -> Net-(D348-Pad1)
- D362 pad 2: Net-(D348-Pad2) -> /z0
- D363 pad 1: GND -> Net-(D348-Pad1)
- D363 pad 2: Net-(D348-Pad2) -> /z0
- D364 pad 1: GND -> Net-(D348-Pad1)
- D364 pad 2: Net-(D348-Pad2) -> /z0
- D365 pad 1: GND -> Net-(D348-Pad1)
- D365 pad 2: Net-(D348-Pad2) -> /z0
- D366 pad 1: GND -> Net-(D348-Pad1)
- D366 pad 2: Net-(D348-Pad2) -> /z0
- D367 pad 1: GND -> Net-(D348-Pad1)
- D367 pad 2: Net-(D348-Pad2) -> /z0
- D368 pad 1: GND -> Net-(D348-Pad1)
- D368 pad 2: Net-(D348-Pad2) -> /z0
- D369 pad 1: GND -> Net-(D348-Pad1)
- D369 pad 2: Net-(D348-Pad2) -> /z0
- D370 pad 1: GND -> Net-(D370-Pad1)
- D370 pad 2: Net-(D370-Pad2) -> /z1
- D371 pad 1: GND -> Net-(D370-Pad1)
- D371 pad 2: Net-(D370-Pad2) -> /z1
- D372 pad 1: GND -> Net-(D370-Pad1)
- D372 pad 2: Net-(D370-Pad2) -> /z1
- D373 pad 1: GND -> Net-(D370-Pad1)
- D373 pad 2: Net-(D370-Pad2) -> /z1
- D374 pad 1: GND -> Net-(D370-Pad1)
- D374 pad 2: Net-(D370-Pad2) -> /z1
- D375 pad 1: GND -> Net-(D370-Pad1)
- D375 pad 2: Net-(D370-Pad2) -> /z1
- D376 pad 1: GND -> Net-(D370-Pad1)
- D376 pad 2: Net-(D370-Pad2) -> /z1
- D377 pad 1: GND -> Net-(D370-Pad1)
- D377 pad 2: Net-(D370-Pad2) -> /z1
- D378 pad 1: GND -> Net-(D370-Pad1)
- D378 pad 2: Net-(D370-Pad2) -> /z1
- D379 pad 1: GND -> Net-(D370-Pad1)
- D379 pad 2: Net-(D370-Pad2) -> /z1
- D380 pad 1: GND -> Net-(D370-Pad1)
- D380 pad 2: Net-(D370-Pad2) -> /z1
- D381 pad 1: GND -> Net-(D370-Pad1)
- D381 pad 2: Net-(D370-Pad2) -> /z1
- D382 pad 1: GND -> Net-(D370-Pad1)
- D382 pad 2: Net-(D370-Pad2) -> /z1
- D383 pad 1: GND -> Net-(D370-Pad1)
- D383 pad 2: Net-(D370-Pad2) -> /z1
- D384 pad 1: GND -> Net-(D370-Pad1)
- D384 pad 2: Net-(D370-Pad2) -> /z1
- D385 pad 1: GND -> Net-(D370-Pad1)
- D385 pad 2: Net-(D370-Pad2) -> /z1
- D386 pad 1: GND -> Net-(D370-Pad1)
- D386 pad 2: Net-(D370-Pad2) -> /z1
- D387 pad 1: GND -> Net-(D370-Pad1)
- D387 pad 2: Net-(D370-Pad2) -> /z1
- D388 pad 1: GND -> Net-(D370-Pad1)
- D388 pad 2: Net-(D370-Pad2) -> /z1
- D389 pad 1: GND -> Net-(D370-Pad1)
- D389 pad 2: Net-(D370-Pad2) -> /z1
- D390 pad 1: GND -> Net-(D370-Pad1)
- D390 pad 2: Net-(D370-Pad2) -> /z1
- D391 pad 1: GND -> Net-(D370-Pad1)
- D391 pad 2: Net-(D370-Pad2) -> /z1
- D392 pad 1: GND -> Net-(D392-Pad1)
- D392 pad 2: Net-(D392-Pad2) -> /z2
- D393 pad 1: GND -> Net-(D392-Pad1)
- D393 pad 2: Net-(D392-Pad2) -> /z2
- D394 pad 1: GND -> Net-(D392-Pad1)
- D394 pad 2: Net-(D392-Pad2) -> /z2
- D395 pad 1: GND -> Net-(D392-Pad1)
- D395 pad 2: Net-(D392-Pad2) -> /z2
- D396 pad 1: GND -> Net-(D392-Pad1)
- D396 pad 2: Net-(D392-Pad2) -> /z2
- D397 pad 1: GND -> Net-(D392-Pad1)
- D397 pad 2: Net-(D392-Pad2) -> /z2
- D398 pad 1: GND -> Net-(D392-Pad1)
- D398 pad 2: Net-(D392-Pad2) -> /z2
- D399 pad 1: GND -> Net-(D392-Pad1)
- D399 pad 2: Net-(D392-Pad2) -> /z2
- D400 pad 1: GND -> Net-(D392-Pad1)
- D400 pad 2: Net-(D392-Pad2) -> /z2
- D401 pad 1: GND -> Net-(D392-Pad1)
- D401 pad 2: Net-(D392-Pad2) -> /z2
- D402 pad 1: GND -> Net-(D392-Pad1)
- D402 pad 2: Net-(D392-Pad2) -> /z2
- D403 pad 1: GND -> Net-(D392-Pad1)
- D403 pad 2: Net-(D392-Pad2) -> /z2
- D404 pad 1: GND -> Net-(D392-Pad1)
- D404 pad 2: Net-(D392-Pad2) -> /z2
- D405 pad 1: GND -> Net-(D392-Pad1)
- D405 pad 2: Net-(D392-Pad2) -> /z2
- D406 pad 1: GND -> Net-(D392-Pad1)
- D406 pad 2: Net-(D392-Pad2) -> /z2
- D407 pad 1: GND -> Net-(D392-Pad1)
- D407 pad 2: Net-(D392-Pad2) -> /z2
- D408 pad 1: GND -> Net-(D392-Pad1)
- D408 pad 2: Net-(D392-Pad2) -> /z2
- D409 pad 1: GND -> Net-(D392-Pad1)
- D409 pad 2: Net-(D392-Pad2) -> /z2
- D410 pad 1: GND -> Net-(D392-Pad1)
- D410 pad 2: Net-(D392-Pad2) -> /z2
- D411 pad 1: GND -> Net-(D392-Pad1)
- D411 pad 2: Net-(D392-Pad2) -> /z2
- D412 pad 1: GND -> Net-(D392-Pad1)
- D412 pad 2: Net-(D392-Pad2) -> /z2
- D413 pad 1: GND -> Net-(D392-Pad1)
- D413 pad 2: Net-(D392-Pad2) -> /z2
- D414 pad 1: GND -> Net-(D414-Pad1)
- D414 pad 2: Net-(D414-Pad2) -> /z3
- D415 pad 1: GND -> Net-(D414-Pad1)
- D415 pad 2: Net-(D414-Pad2) -> /z3
- D416 pad 1: GND -> Net-(D414-Pad1)
- D416 pad 2: Net-(D414-Pad2) -> /z3
- D417 pad 1: GND -> Net-(D414-Pad1)
- D417 pad 2: Net-(D414-Pad2) -> /z3
- D418 pad 1: GND -> Net-(D414-Pad1)
- D418 pad 2: Net-(D414-Pad2) -> /z3
- D419 pad 1: GND -> Net-(D414-Pad1)
- D419 pad 2: Net-(D414-Pad2) -> /z3
- D420 pad 1: GND -> Net-(D414-Pad1)
- D420 pad 2: Net-(D414-Pad2) -> /z3
- D421 pad 1: GND -> Net-(D414-Pad1)
- D421 pad 2: Net-(D414-Pad2) -> /z3
- D422 pad 1: GND -> Net-(D414-Pad1)
- D422 pad 2: Net-(D414-Pad2) -> /z3
- D423 pad 1: GND -> Net-(D414-Pad1)
- D423 pad 2: Net-(D414-Pad2) -> /z3
- D424 pad 1: GND -> Net-(D414-Pad1)
- D424 pad 2: Net-(D414-Pad2) -> /z3
- D425 pad 1: GND -> Net-(D414-Pad1)
- D425 pad 2: Net-(D414-Pad2) -> /z3
- D426 pad 1: GND -> Net-(D414-Pad1)
- D426 pad 2: Net-(D414-Pad2) -> /z3
- D427 pad 1: GND -> Net-(D414-Pad1)
- D427 pad 2: Net-(D414-Pad2) -> /z3
- D428 pad 1: GND -> Net-(D414-Pad1)
- D428 pad 2: Net-(D414-Pad2) -> /z3
- D429 pad 1: GND -> Net-(D414-Pad1)
- D429 pad 2: Net-(D414-Pad2) -> /z3
- D430 pad 1: GND -> Net-(D414-Pad1)
- D430 pad 2: Net-(D414-Pad2) -> /z3
- D431 pad 1: GND -> Net-(D414-Pad1)
- D431 pad 2: Net-(D414-Pad2) -> /z3
- D432 pad 1: GND -> Net-(D414-Pad1)
- D432 pad 2: Net-(D414-Pad2) -> /z3
- D433 pad 1: GND -> Net-(D414-Pad1)
- D433 pad 2: Net-(D414-Pad2) -> /z3
- D434 pad 1: GND -> Net-(D414-Pad1)
- D434 pad 2: Net-(D414-Pad2) -> /z3
- D435 pad 1: GND -> Net-(D435-Pad1)
- D435 pad 2: Net-(D435-Pad2) -> /z4
- D436 pad 1: GND -> Net-(D435-Pad1)
- D436 pad 2: Net-(D435-Pad2) -> /z4
- D437 pad 1: GND -> Net-(D435-Pad1)
- D437 pad 2: Net-(D435-Pad2) -> /z4
- D438 pad 1: GND -> Net-(D435-Pad1)
- D438 pad 2: Net-(D435-Pad2) -> /z4
- D439 pad 1: GND -> Net-(D435-Pad1)
- D439 pad 2: Net-(D435-Pad2) -> /z4
- D440 pad 1: GND -> Net-(D435-Pad1)
- D440 pad 2: Net-(D435-Pad2) -> /z4
- D441 pad 1: GND -> Net-(D435-Pad1)
- D441 pad 2: Net-(D435-Pad2) -> /z4
- D442 pad 1: GND -> Net-(D435-Pad1)
- D442 pad 2: Net-(D435-Pad2) -> /z4
- D443 pad 1: GND -> Net-(D435-Pad1)
- D443 pad 2: Net-(D435-Pad2) -> /z4
- D444 pad 1: GND -> Net-(D435-Pad1)
- D444 pad 2: Net-(D435-Pad2) -> /z4
- D445 pad 1: GND -> Net-(D435-Pad1)
- D445 pad 2: Net-(D435-Pad2) -> /z4
- D446 pad 1: GND -> Net-(D435-Pad1)
- D446 pad 2: Net-(D435-Pad2) -> /z4
- D447 pad 1: GND -> Net-(D435-Pad1)
- D447 pad 2: Net-(D435-Pad2) -> /z4
- D448 pad 1: GND -> Net-(D435-Pad1)
- D448 pad 2: Net-(D435-Pad2) -> /z4
- D449 pad 1: GND -> Net-(D435-Pad1)
- D449 pad 2: Net-(D435-Pad2) -> /z4
- D450 pad 1: GND -> Net-(D435-Pad1)
- D450 pad 2: Net-(D435-Pad2) -> /z4
- D451 pad 1: GND -> Net-(D435-Pad1)
- D451 pad 2: Net-(D435-Pad2) -> /z4
- D452 pad 1: GND -> Net-(D435-Pad1)
- D452 pad 2: Net-(D435-Pad2) -> /z4
- D453 pad 1: GND -> Net-(D435-Pad1)
- D453 pad 2: Net-(D435-Pad2) -> /z4
- D454 pad 1: GND -> Net-(D435-Pad1)
- D454 pad 2: Net-(D435-Pad2) -> /z4
- D455 pad 1: GND -> Net-(D435-Pad1)
- D455 pad 2: Net-(D435-Pad2) -> /z4
- D456 pad 1: GND -> Net-(D456-Pad1)
- D456 pad 2: Net-(D456-Pad2) -> /z5
- D457 pad 1: GND -> Net-(D456-Pad1)
- D457 pad 2: Net-(D456-Pad2) -> /z5
- D458 pad 1: GND -> Net-(D456-Pad1)
- D458 pad 2: Net-(D456-Pad2) -> /z5
- D459 pad 1: GND -> Net-(D456-Pad1)
- D459 pad 2: Net-(D456-Pad2) -> /z5
- D460 pad 1: GND -> Net-(D456-Pad1)
- D460 pad 2: Net-(D456-Pad2) -> /z5
- D461 pad 1: GND -> Net-(D456-Pad1)
- D461 pad 2: Net-(D456-Pad2) -> /z5
- D462 pad 1: GND -> Net-(D456-Pad1)
- D462 pad 2: Net-(D456-Pad2) -> /z5
- D463 pad 1: GND -> Net-(D456-Pad1)
- D463 pad 2: Net-(D456-Pad2) -> /z5
- D464 pad 1: GND -> Net-(D456-Pad1)
- D464 pad 2: Net-(D456-Pad2) -> /z5
- D465 pad 1: GND -> Net-(D456-Pad1)
- D465 pad 2: Net-(D456-Pad2) -> /z5
- D466 pad 1: GND -> Net-(D456-Pad1)
- D466 pad 2: Net-(D456-Pad2) -> /z5
- D467 pad 1: GND -> Net-(D456-Pad1)
- D467 pad 2: Net-(D456-Pad2) -> /z5
- D468 pad 1: GND -> Net-(D456-Pad1)
- D468 pad 2: Net-(D456-Pad2) -> /z5
- D469 pad 1: GND -> Net-(D456-Pad1)
- D469 pad 2: Net-(D456-Pad2) -> /z5
- D470 pad 1: GND -> Net-(D456-Pad1)
- D470 pad 2: Net-(D456-Pad2) -> /z5
- D471 pad 1: GND -> Net-(D456-Pad1)
- D471 pad 2: Net-(D456-Pad2) -> /z5
- D472 pad 1: GND -> Net-(D456-Pad1)
- D472 pad 2: Net-(D456-Pad2) -> /z5
- D473 pad 1: GND -> Net-(D456-Pad1)
- D473 pad 2: Net-(D456-Pad2) -> /z5
- D474 pad 1: GND -> Net-(D456-Pad1)
- D474 pad 2: Net-(D456-Pad2) -> /z5
- D475 pad 1: GND -> Net-(D456-Pad1)
- D475 pad 2: Net-(D456-Pad2) -> /z5
- D476 pad 1: GND -> Net-(D456-Pad1)
- D476 pad 2: Net-(D456-Pad2) -> /z5
- D477 pad 1: GND -> Net-(D477-Pad1)
- D477 pad 2: Net-(D477-Pad2) -> /z6
- D478 pad 1: GND -> Net-(D477-Pad1)
- D478 pad 2: Net-(D477-Pad2) -> /z6
- D479 pad 1: GND -> Net-(D477-Pad1)
- D479 pad 2: Net-(D477-Pad2) -> /z6
- D480 pad 1: GND -> Net-(D477-Pad1)
- D480 pad 2: Net-(D477-Pad2) -> /z6
- D481 pad 1: GND -> Net-(D477-Pad1)
- D481 pad 2: Net-(D477-Pad2) -> /z6
- D482 pad 1: GND -> Net-(D477-Pad1)
- D482 pad 2: Net-(D477-Pad2) -> /z6
- D483 pad 1: GND -> Net-(D477-Pad1)
- D483 pad 2: Net-(D477-Pad2) -> /z6
- D484 pad 1: GND -> Net-(D477-Pad1)
- D484 pad 2: Net-(D477-Pad2) -> /z6
- D485 pad 1: GND -> Net-(D477-Pad1)
- D485 pad 2: Net-(D477-Pad2) -> /z6
- D486 pad 1: GND -> Net-(D477-Pad1)
- D486 pad 2: Net-(D477-Pad2) -> /z6
- D487 pad 1: GND -> Net-(D477-Pad1)
- D487 pad 2: Net-(D477-Pad2) -> /z6
- D488 pad 1: GND -> Net-(D477-Pad1)
- D488 pad 2: Net-(D477-Pad2) -> /z6
- D489 pad 1: GND -> Net-(D477-Pad1)
- D489 pad 2: Net-(D477-Pad2) -> /z6
- D490 pad 1: GND -> Net-(D477-Pad1)
- D490 pad 2: Net-(D477-Pad2) -> /z6
- D491 pad 1: GND -> Net-(D477-Pad1)
- D491 pad 2: Net-(D477-Pad2) -> /z6
- D492 pad 1: GND -> Net-(D477-Pad1)
- D492 pad 2: Net-(D477-Pad2) -> /z6
- D493 pad 1: GND -> Net-(D477-Pad1)
- D493 pad 2: Net-(D477-Pad2) -> /z6
- D494 pad 1: GND -> Net-(D477-Pad1)
- D494 pad 2: Net-(D477-Pad2) -> /z6
- D495 pad 1: GND -> Net-(D477-Pad1)
- D495 pad 2: Net-(D477-Pad2) -> /z6
- D496 pad 1: GND -> Net-(D477-Pad1)
- D496 pad 2: Net-(D477-Pad2) -> /z6
- D497 pad 1: GND -> Net-(D477-Pad1)
- D497 pad 2: Net-(D477-Pad2) -> /z6
- D498 pad 1: GND -> Net-(D498-Pad1)
- D498 pad 2: Net-(D498-Pad2) -> /z7
- D499 pad 1: GND -> Net-(D498-Pad1)
- D499 pad 2: Net-(D498-Pad2) -> /z7
- D500 pad 1: GND -> Net-(D498-Pad1)
- D500 pad 2: Net-(D498-Pad2) -> /z7
- D501 pad 1: GND -> Net-(D498-Pad1)
- D501 pad 2: Net-(D498-Pad2) -> /z7
- D502 pad 1: GND -> Net-(D498-Pad1)
- D502 pad 2: Net-(D498-Pad2) -> /z7
- D503 pad 1: GND -> Net-(D498-Pad1)
- D503 pad 2: Net-(D498-Pad2) -> /z7
- D504 pad 1: GND -> Net-(D498-Pad1)
- D504 pad 2: Net-(D498-Pad2) -> /z7
- D505 pad 1: GND -> Net-(D498-Pad1)
- D505 pad 2: Net-(D498-Pad2) -> /z7
- D506 pad 1: GND -> Net-(D498-Pad1)
- D506 pad 2: Net-(D498-Pad2) -> /z7
- D507 pad 1: GND -> Net-(D498-Pad1)
- D507 pad 2: Net-(D498-Pad2) -> /z7
- D508 pad 1: GND -> Net-(D498-Pad1)
- D508 pad 2: Net-(D498-Pad2) -> /z7
- D509 pad 1: GND -> Net-(D498-Pad1)
- D509 pad 2: Net-(D498-Pad2) -> /z7
- D510 pad 1: GND -> Net-(D498-Pad1)
- D510 pad 2: Net-(D498-Pad2) -> /z7
- D511 pad 1: GND -> Net-(D498-Pad1)
- D511 pad 2: Net-(D498-Pad2) -> /z7
- D512 pad 1: GND -> Net-(D498-Pad1)
- D512 pad 2: Net-(D498-Pad2) -> /z7
- D513 pad 1: GND -> Net-(D498-Pad1)
- D513 pad 2: Net-(D498-Pad2) -> /z7
- D514 pad 1: GND -> Net-(D498-Pad1)
- D514 pad 2: Net-(D498-Pad2) -> /z7
- D515 pad 1: GND -> Net-(D498-Pad1)
- D515 pad 2: Net-(D498-Pad2) -> /z7
- D516 pad 1: GND -> Net-(D498-Pad1)
- D516 pad 2: Net-(D498-Pad2) -> /z7
- D517 pad 1: GND -> Net-(D498-Pad1)
- D517 pad 2: Net-(D498-Pad2) -> /z7
- D518 pad 1: GND -> Net-(D498-Pad1)
- D518 pad 2: Net-(D498-Pad2) -> /z7
- D519 pad 1: GND -> Net-(D519-Pad1)
- D519 pad 2: Net-(D519-Pad2) -> /o0
- D520 pad 1: GND -> Net-(D519-Pad1)
- D520 pad 2: Net-(D519-Pad2) -> /o0
- D521 pad 1: GND -> Net-(D519-Pad1)
- D521 pad 2: Net-(D519-Pad2) -> /o0
- D522 pad 1: GND -> Net-(D519-Pad1)
- D522 pad 2: Net-(D519-Pad2) -> /o0
- D523 pad 1: GND -> Net-(D519-Pad1)
- D523 pad 2: Net-(D519-Pad2) -> /o0
- D524 pad 1: GND -> Net-(D519-Pad1)
- D524 pad 2: Net-(D519-Pad2) -> /o0
- D525 pad 1: GND -> Net-(D519-Pad1)
- D525 pad 2: Net-(D519-Pad2) -> /o0
- D526 pad 1: GND -> Net-(D519-Pad1)
- D526 pad 2: Net-(D519-Pad2) -> /o0
- D527 pad 1: GND -> Net-(D519-Pad1)
- D527 pad 2: Net-(D519-Pad2) -> /o0
- D528 pad 1: GND -> Net-(D519-Pad1)
- D528 pad 2: Net-(D519-Pad2) -> /o0
- D529 pad 1: GND -> Net-(D519-Pad1)
- D529 pad 2: Net-(D519-Pad2) -> /o0
- D530 pad 1: GND -> Net-(D519-Pad1)
- D530 pad 2: Net-(D519-Pad2) -> /o0
- D531 pad 1: GND -> Net-(D519-Pad1)
- D531 pad 2: Net-(D519-Pad2) -> /o0
- D532 pad 1: GND -> Net-(D519-Pad1)
- D532 pad 2: Net-(D519-Pad2) -> /o0
- D533 pad 1: GND -> Net-(D519-Pad1)
- D533 pad 2: Net-(D519-Pad2) -> /o0
- D534 pad 1: GND -> Net-(D519-Pad1)
- D534 pad 2: Net-(D519-Pad2) -> /o0
- D535 pad 1: GND -> Net-(D535-Pad1)
- D535 pad 2: Net-(D535-Pad2) -> /o1
- D536 pad 1: GND -> Net-(D535-Pad1)
- D536 pad 2: Net-(D535-Pad2) -> /o1
- D537 pad 1: GND -> Net-(D535-Pad1)
- D537 pad 2: Net-(D535-Pad2) -> /o1
- D538 pad 1: GND -> Net-(D535-Pad1)
- D538 pad 2: Net-(D535-Pad2) -> /o1
- D539 pad 1: GND -> Net-(D535-Pad1)
- D539 pad 2: Net-(D535-Pad2) -> /o1
- D540 pad 1: GND -> Net-(D535-Pad1)
- D540 pad 2: Net-(D535-Pad2) -> /o1
- D541 pad 1: GND -> Net-(D535-Pad1)
- D541 pad 2: Net-(D535-Pad2) -> /o1
- D542 pad 1: GND -> Net-(D535-Pad1)
- D542 pad 2: Net-(D535-Pad2) -> /o1
- D543 pad 1: GND -> Net-(D535-Pad1)
- D543 pad 2: Net-(D535-Pad2) -> /o1
- D544 pad 1: GND -> Net-(D535-Pad1)
- D544 pad 2: Net-(D535-Pad2) -> /o1
- D545 pad 1: GND -> Net-(D535-Pad1)
- D545 pad 2: Net-(D535-Pad2) -> /o1
- D546 pad 1: GND -> Net-(D535-Pad1)
- D546 pad 2: Net-(D535-Pad2) -> /o1
- D547 pad 1: GND -> Net-(D535-Pad1)
- D547 pad 2: Net-(D535-Pad2) -> /o1
- D548 pad 1: GND -> Net-(D535-Pad1)
- D548 pad 2: Net-(D535-Pad2) -> /o1
- D549 pad 1: GND -> Net-(D535-Pad1)
- D549 pad 2: Net-(D535-Pad2) -> /o1
- D550 pad 1: GND -> Net-(D535-Pad1)
- D550 pad 2: Net-(D535-Pad2) -> /o1
- D551 pad 1: GND -> Net-(D551-Pad1)
- D551 pad 2: Net-(D551-Pad2) -> /o2
- D552 pad 1: GND -> Net-(D551-Pad1)
- D552 pad 2: Net-(D551-Pad2) -> /o2
- D553 pad 1: GND -> Net-(D551-Pad1)
- D553 pad 2: Net-(D551-Pad2) -> /o2
- D554 pad 1: GND -> Net-(D551-Pad1)
- D554 pad 2: Net-(D551-Pad2) -> /o2
- D555 pad 1: GND -> Net-(D551-Pad1)
- D555 pad 2: Net-(D551-Pad2) -> /o2
- D556 pad 1: GND -> Net-(D551-Pad1)
- D556 pad 2: Net-(D551-Pad2) -> /o2
- D557 pad 1: GND -> Net-(D551-Pad1)
- D557 pad 2: Net-(D551-Pad2) -> /o2
- D558 pad 1: GND -> Net-(D551-Pad1)
- D558 pad 2: Net-(D551-Pad2) -> /o2
- D559 pad 1: GND -> Net-(D551-Pad1)
- D559 pad 2: Net-(D551-Pad2) -> /o2
- D560 pad 1: GND -> Net-(D551-Pad1)
- D560 pad 2: Net-(D551-Pad2) -> /o2
- D561 pad 1: GND -> Net-(D551-Pad1)
- D561 pad 2: Net-(D551-Pad2) -> /o2
- D562 pad 1: GND -> Net-(D551-Pad1)
- D562 pad 2: Net-(D551-Pad2) -> /o2
- D563 pad 1: GND -> Net-(D551-Pad1)
- D563 pad 2: Net-(D551-Pad2) -> /o2
- D564 pad 1: GND -> Net-(D551-Pad1)
- D564 pad 2: Net-(D551-Pad2) -> /o2
- D565 pad 1: GND -> Net-(D551-Pad1)
- D565 pad 2: Net-(D551-Pad2) -> /o2
- D566 pad 1: GND -> Net-(D551-Pad1)
- D566 pad 2: Net-(D551-Pad2) -> /o2
- D567 pad 1: GND -> Net-(D567-Pad1)
- D567 pad 2: Net-(D567-Pad2) -> /o3
- D568 pad 1: GND -> Net-(D567-Pad1)
- D568 pad 2: Net-(D567-Pad2) -> /o3
- D569 pad 1: GND -> Net-(D567-Pad1)
- D569 pad 2: Net-(D567-Pad2) -> /o3
- D570 pad 1: GND -> Net-(D567-Pad1)
- D570 pad 2: Net-(D567-Pad2) -> /o3
- D571 pad 1: GND -> Net-(D567-Pad1)
- D571 pad 2: Net-(D567-Pad2) -> /o3
- D572 pad 1: GND -> Net-(D567-Pad1)
- D572 pad 2: Net-(D567-Pad2) -> /o3
- D573 pad 1: GND -> Net-(D567-Pad1)
- D573 pad 2: Net-(D567-Pad2) -> /o3
- D574 pad 1: GND -> Net-(D567-Pad1)
- D574 pad 2: Net-(D567-Pad2) -> /o3
- D575 pad 1: GND -> Net-(D567-Pad1)
- D575 pad 2: Net-(D567-Pad2) -> /o3
- D576 pad 1: GND -> Net-(D567-Pad1)
- D576 pad 2: Net-(D567-Pad2) -> /o3
- D577 pad 1: GND -> Net-(D567-Pad1)
- D577 pad 2: Net-(D567-Pad2) -> /o3
- D578 pad 1: GND -> Net-(D567-Pad1)
- D578 pad 2: Net-(D567-Pad2) -> /o3
- D579 pad 1: GND -> Net-(D567-Pad1)
- D579 pad 2: Net-(D567-Pad2) -> /o3
- D580 pad 1: GND -> Net-(D567-Pad1)
- D580 pad 2: Net-(D567-Pad2) -> /o3
- D581 pad 1: GND -> Net-(D567-Pad1)
- D581 pad 2: Net-(D567-Pad2) -> /o3
- D582 pad 1: GND -> Net-(D582-Pad1)
- D582 pad 2: Net-(D582-Pad2) -> /o4
- D583 pad 1: GND -> Net-(D582-Pad1)
- D583 pad 2: Net-(D582-Pad2) -> /o4
- D584 pad 1: GND -> Net-(D582-Pad1)
- D584 pad 2: Net-(D582-Pad2) -> /o4
- D585 pad 1: GND -> Net-(D582-Pad1)
- D585 pad 2: Net-(D582-Pad2) -> /o4
- D586 pad 1: GND -> Net-(D582-Pad1)
- D586 pad 2: Net-(D582-Pad2) -> /o4
- D587 pad 1: GND -> Net-(D582-Pad1)
- D587 pad 2: Net-(D582-Pad2) -> /o4
- D588 pad 1: GND -> Net-(D582-Pad1)
- D588 pad 2: Net-(D582-Pad2) -> /o4
- D589 pad 1: GND -> Net-(D582-Pad1)
- D589 pad 2: Net-(D582-Pad2) -> /o4
- D590 pad 1: GND -> Net-(D582-Pad1)
- D590 pad 2: Net-(D582-Pad2) -> /o4
- D591 pad 1: GND -> Net-(D582-Pad1)
- D591 pad 2: Net-(D582-Pad2) -> /o4
- D592 pad 1: GND -> Net-(D582-Pad1)
- D592 pad 2: Net-(D582-Pad2) -> /o4
- D593 pad 1: GND -> Net-(D582-Pad1)
- D593 pad 2: Net-(D582-Pad2) -> /o4
- D594 pad 1: GND -> Net-(D582-Pad1)
- D594 pad 2: Net-(D582-Pad2) -> /o4
- D595 pad 1: GND -> Net-(D582-Pad1)
- D595 pad 2: Net-(D582-Pad2) -> /o4
- D596 pad 1: GND -> Net-(D582-Pad1)
- D596 pad 2: Net-(D582-Pad2) -> /o4
- D597 pad 1: GND -> Net-(D597-Pad1)
- D597 pad 2: Net-(D597-Pad2) -> /o5
- D598 pad 1: GND -> Net-(D597-Pad1)
- D598 pad 2: Net-(D597-Pad2) -> /o5
- D599 pad 1: GND -> Net-(D597-Pad1)
- D599 pad 2: Net-(D597-Pad2) -> /o5
- D600 pad 1: GND -> Net-(D597-Pad1)
- D600 pad 2: Net-(D597-Pad2) -> /o5
- D601 pad 1: GND -> Net-(D597-Pad1)
- D601 pad 2: Net-(D597-Pad2) -> /o5
- D602 pad 1: GND -> Net-(D597-Pad1)
- D602 pad 2: Net-(D597-Pad2) -> /o5
- D603 pad 1: GND -> Net-(D597-Pad1)
- D603 pad 2: Net-(D597-Pad2) -> /o5
- D604 pad 1: GND -> Net-(D597-Pad1)
- D604 pad 2: Net-(D597-Pad2) -> /o5
- D605 pad 1: GND -> Net-(D597-Pad1)
- D605 pad 2: Net-(D597-Pad2) -> /o5
- D606 pad 1: GND -> Net-(D597-Pad1)
- D606 pad 2: Net-(D597-Pad2) -> /o5
- D607 pad 1: GND -> Net-(D597-Pad1)
- D607 pad 2: Net-(D597-Pad2) -> /o5
- D608 pad 1: GND -> Net-(D597-Pad1)
- D608 pad 2: Net-(D597-Pad2) -> /o5
- D609 pad 1: GND -> Net-(D597-Pad1)
- D609 pad 2: Net-(D597-Pad2) -> /o5
- D610 pad 1: GND -> Net-(D597-Pad1)
- D610 pad 2: Net-(D597-Pad2) -> /o5
- D611 pad 1: GND -> Net-(D597-Pad1)
- D611 pad 2: Net-(D597-Pad2) -> /o5
- D612 pad 1: GND -> Net-(D612-Pad1)
- D612 pad 2: Net-(D612-Pad2) -> /o6
- D613 pad 1: GND -> Net-(D612-Pad1)
- D613 pad 2: Net-(D612-Pad2) -> /o6
- D614 pad 1: GND -> Net-(D612-Pad1)
- D614 pad 2: Net-(D612-Pad2) -> /o6
- D615 pad 1: GND -> Net-(D612-Pad1)
- D615 pad 2: Net-(D612-Pad2) -> /o6
- D616 pad 1: GND -> Net-(D612-Pad1)
- D616 pad 2: Net-(D612-Pad2) -> /o6
- D617 pad 1: GND -> Net-(D612-Pad1)
- D617 pad 2: Net-(D612-Pad2) -> /o6
- D618 pad 1: GND -> Net-(D612-Pad1)
- D618 pad 2: Net-(D612-Pad2) -> /o6
- D619 pad 1: GND -> Net-(D612-Pad1)
- D619 pad 2: Net-(D612-Pad2) -> /o6
- D620 pad 1: GND -> Net-(D612-Pad1)
- D620 pad 2: Net-(D612-Pad2) -> /o6
- D621 pad 1: GND -> Net-(D612-Pad1)
- D621 pad 2: Net-(D612-Pad2) -> /o6
- D622 pad 1: GND -> Net-(D612-Pad1)
- D622 pad 2: Net-(D612-Pad2) -> /o6
- D623 pad 1: GND -> Net-(D612-Pad1)
- D623 pad 2: Net-(D612-Pad2) -> /o6
- D624 pad 1: GND -> Net-(D612-Pad1)
- D624 pad 2: Net-(D612-Pad2) -> /o6
- D625 pad 1: GND -> Net-(D612-Pad1)
- D625 pad 2: Net-(D612-Pad2) -> /o6
- D626 pad 1: GND -> Net-(D612-Pad1)
- D626 pad 2: Net-(D612-Pad2) -> /o6
- D627 pad 1: GND -> Net-(D627-Pad1)
- D627 pad 2: Net-(D627-Pad2) -> /o7
- D628 pad 1: GND -> Net-(D627-Pad1)
- D629 pad 1: GND -> Net-(D627-Pad1)
- D630 pad 1: GND -> Net-(D627-Pad1)
- D631 pad 1: GND -> Net-(D627-Pad1)
- D632 pad 1: GND -> Net-(D627-Pad1)
- D633 pad 1: GND -> Net-(D627-Pad1)
- D634 pad 1: GND -> Net-(D627-Pad1)
- D635 pad 1: GND -> Net-(D627-Pad1)
- D636 pad 1: GND -> Net-(D627-Pad1)
- D637 pad 1: GND -> Net-(D627-Pad1)
- D638 pad 1: GND -> Net-(D627-Pad1)
- D639 pad 1: GND -> Net-(D627-Pad1)
- D640 pad 1: GND -> Net-(D627-Pad1)
- D641 pad 1: GND -> Net-(D627-Pad1)
- R201 pad 1: Net-(D201-Pad2) -> GND
- R201 pad 2: /a0 -> Net-(D201-Pad1)
- R202 pad 1: Net-(D234-Pad2) -> GND
- R202 pad 2: /a1 -> Net-(D234-Pad1)
- R203 pad 1: Net-(D267-Pad2) -> GND
- R203 pad 2: /a2 -> Net-(D267-Pad1)
- R204 pad 1: Net-(D300-Pad2) -> GND
- R204 pad 2: /b0 -> Net-(D300-Pad1)
- R205 pad 1: Net-(D303-Pad2) -> GND
- R205 pad 2: /b1 -> Net-(D303-Pad1)
- R206 pad 1: Net-(D306-Pad2) -> GND
- R206 pad 2: /b2 -> Net-(D306-Pad1)
- R207 pad 1: Net-(D309-Pad2) -> GND
- R207 pad 2: /b3 -> Net-(D309-Pad1)
- R208 pad 1: Net-(D312-Pad2) -> GND
- R208 pad 2: /b4 -> Net-(D312-Pad1)
- R209 pad 1: Net-(D315-Pad2) -> GND
- R209 pad 2: /b5 -> Net-(D315-Pad1)
- R210 pad 1: Net-(D318-Pad2) -> GND
- R210 pad 2: /b6 -> Net-(D318-Pad1)
- R211 pad 1: Net-(D321-Pad2) -> GND
- R211 pad 2: /b7 -> Net-(D321-Pad1)
- R212 pad 1: Net-(D324-Pad2) -> GND
- R212 pad 2: /b8 -> Net-(D324-Pad1)
- R213 pad 1: Net-(D327-Pad2) -> GND
- R213 pad 2: /b9 -> Net-(D327-Pad1)
- R214 pad 1: Net-(D330-Pad2) -> GND
- R214 pad 2: /b10 -> Net-(D330-Pad1)
- R215 pad 1: Net-(D333-Pad2) -> GND
- R215 pad 2: /b11 -> Net-(D333-Pad1)
- R216 pad 1: Net-(D336-Pad2) -> GND
- R216 pad 2: /b12 -> Net-(D336-Pad1)
- R217 pad 1: Net-(D339-Pad2) -> GND
- R217 pad 2: /b13 -> Net-(D339-Pad1)
- R218 pad 1: Net-(D342-Pad2) -> GND
- R218 pad 2: /b14 -> Net-(D342-Pad1)
- R219 pad 1: Net-(D345-Pad2) -> GND
- R219 pad 2: /b15 -> Net-(D345-Pad1)
- R220 pad 1: Net-(D348-Pad2) -> GND
- R220 pad 2: /z0 -> Net-(D348-Pad1)
- R221 pad 1: Net-(D370-Pad2) -> GND
- R221 pad 2: /z1 -> Net-(D370-Pad1)
- R222 pad 1: Net-(D392-Pad2) -> GND
- R222 pad 2: /z2 -> Net-(D392-Pad1)
- R223 pad 1: Net-(D414-Pad2) -> GND
- R223 pad 2: /z3 -> Net-(D414-Pad1)
- R224 pad 1: Net-(D435-Pad2) -> GND
- R224 pad 2: /z4 -> Net-(D435-Pad1)
- R225 pad 1: Net-(D456-Pad2) -> GND
- R225 pad 2: /z5 -> Net-(D456-Pad1)
- R226 pad 1: Net-(D477-Pad2) -> GND
- R226 pad 2: /z6 -> Net-(D477-Pad1)
- R227 pad 1: Net-(D498-Pad2) -> GND
- R227 pad 2: /z7 -> Net-(D498-Pad1)
- R228 pad 1: Net-(D519-Pad2) -> GND
- R228 pad 2: /o0 -> Net-(D519-Pad1)
- R229 pad 1: Net-(D535-Pad2) -> GND
- R229 pad 2: /o1 -> Net-(D535-Pad1)
- R230 pad 1: Net-(D551-Pad2) -> GND
- R230 pad 2: /o2 -> Net-(D551-Pad1)
- R231 pad 1: Net-(D567-Pad2) -> GND
- R231 pad 2: /o3 -> Net-(D567-Pad1)
- R232 pad 1: Net-(D582-Pad2) -> GND
- R232 pad 2: /o4 -> Net-(D582-Pad1)
- R233 pad 1: Net-(D597-Pad2) -> GND
- R233 pad 2: /o5 -> Net-(D597-Pad1)
- R234 pad 1: Net-(D612-Pad2) -> GND
- R234 pad 2: /o6 -> Net-(D612-Pad1)
- R235 pad 1: Net-(D627-Pad2) -> GND
- R235 pad 2: /o7 -> Net-(D627-Pad1)

Commit message: Work on laying out the LED matrix
Parts:
- moved D241 240.5 mm to (99.1, 24.1), turned to 90 degrees
- moved D243 240.0 mm to (99.1, 31.8), turned to 90 degrees
- moved D313 238.3 mm to (95.2, 39.4), turned to 90 degrees
- moved D244 234.5 mm to (99.1, 35.6), turned to 90 degrees
- moved D240 230.4 mm to (99.1, 20.3), turned to 90 degrees
- moved D259 229.8 mm to (87.6, 27.9), turned to 90 degrees
- moved D245 224.4 mm to (99.1, 39.4), turned to 90 degrees
- moved D248 222.8 mm to (91.4, 43.2), turned to 90 degrees
- moved D263 222.5 mm to (91.4, 31.8), turned to 90 degrees
- moved D266 222.4 mm to (91.4, 35.6), turned to 90 degrees
- moved D235 221.7 mm to (80.0, 20.3), turned to 90 degrees
- moved D250 220.8 mm to (83.8, 43.2), turned to 90 degrees
- moved D264 220.0 mm to (83.8, 35.6), turned to 90 degrees
- moved D246 219.6 mm to (99.1, 43.2), turned to 90 degrees
- moved D260 217.5 mm to (91.4, 27.9), turned to 90 degrees
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
Commit message: Work on laying out the LED matrix
Parts:
- moved D319 156.2 mm to (87.6, 39.4)
- moved D371 151.3 mm to (72.4, 24.1)
- moved D394 146.8 mm to (72.4, 31.8)
- moved D435 143.8 mm to (68.6, 20.3)
- moved D348 140.4 mm to (49.5, 20.3)
- moved D349 139.3 mm to (64.8, 24.1)
- moved D392 138.8 mm to (61.0, 20.3)
- moved D351 137.9 mm to (61.0, 39.4)
- moved D370 136.6 mm to (57.1, 20.3)
- moved D567 136.1 mm to (68.6, 24.1)
- moved D456 134.3 mm to (72.4, 20.3)
- moved D372 133.9 mm to (61.0, 31.8)
- moved D414 132.9 mm to (64.8, 20.3)
- moved D436 132.8 mm to (64.8, 27.9)
- moved D628 129.4 mm to (68.6, 39.4)
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Connections:
- D628 pad 2: Net-(D628-Pad2) -> /o7
- D629 pad 2: Net-(D628-Pad2) -> /o7
- D630 pad 2: Net-(D628-Pad2) -> /o7
- D631 pad 2: Net-(D628-Pad2) -> /o7
- D632 pad 2: Net-(D628-Pad2) -> /o7
- D633 pad 2: Net-(D628-Pad2) -> /o7
- D634 pad 2: Net-(D628-Pad2) -> /o7
- D635 pad 2: Net-(D628-Pad2) -> /o7
- D636 pad 2: Net-(D628-Pad2) -> /o7
- D637 pad 2: Net-(D628-Pad2) -> /o7
- D638 pad 2: Net-(D628-Pad2) -> /o7
- D639 pad 2: Net-(D628-Pad2) -> /o7
- D640 pad 2: Net-(D628-Pad2) -> /o7
- D641 pad 2: Net-(D628-Pad2) -> /o7
Routing:
- net /a0: track 96.9 -> 110.3 mm
- net Net-(U105-Pad13): track 14.5 -> 24.7 mm
- net Net-(U105-Pad12): track 10.2 -> 20.3 mm
