File: midnight-sun-2019/midnight-sun-2019.kicad_pcb (KiCad board)
At the start: 4 copper layers, 223.5 x 156.2 mm, 553 parts, among them J1 Conn_02x02_Odd_Even, J2 USB_B_Micro, SW1 SW_SPDT, SW2 SW_SPDT, SW3 SW_SPDT, U1 74HC14, U10 74HC14, U11 74HC86, U12 74HC86, U13 74HC86, U14 74HC86, U15 74HC14, U16 74HC14, U2 74HC595, U3 74HC595, U4 74HC595, U5 74HC86, U6 74HC86, U7 74HC86, U8 74HC86, U9 74HC14

Commit message: Add GND and VCC connections to ICs...
Connections:
- U1 pad 14: (no net) -> VCC
- U1 pad 7: (no net) -> GND
- U10 pad 14: (no net) -> VCC
- U10 pad 7: (no net) -> GND
- U11 pad 14: (no net) -> VCC
- U11 pad 7: (no net) -> GND
- U12 pad 14: (no net) -> VCC
- U12 pad 7: (no net) -> GND
- U13 pad 14: (no net) -> VCC
- U13 pad 7: (no net) -> GND
- U14 pad 14: (no net) -> VCC
- U14 pad 7: (no net) -> GND
- U15 pad 14: (no net) -> VCC
- U15 pad 7: (no net) -> GND
- U16 pad 14: (no net) -> VCC
- U16 pad 7: (no net) -> GND
- U5 pad 14: (no net) -> VCC
- U5 pad 7: (no net) -> GND
- U6 pad 14: (no net) -> VCC
- U6 pad 7: (no net) -> GND
- U7 pad 14: (no net) -> VCC
- U7 pad 7: (no net) -> GND
- U8 pad 14: (no net) -> VCC
- U8 pad 7: (no net) -> GND
- U9 pad 14: (no net) -> VCC
- U9 pad 7: (no net) -> GND
Routing:
- net /z4: track 89.4 -> 90.1 mm, vias 0 -> 2

Commit message: Update PCB routes to agree with new schematic
Parts:
- added C2: 10 uF, Capacitor_THT:CP_Radial_D5.0mm_P2.00mm, F.Cu at (185.4, 29.2)
- added R4: 10k, Resistor_THT:R_Axial_DIN0207_L6.3mm_D2.5mm_P7.62mm_Horizontal, F.Cu at (185.4, 38.1)
- R1: value 10k -> 1k
- moved U1 17.0 mm to (223.5, 45.7), turned to 0 degrees
- moved R1 7.62 mm to (185.4, 33.0), turned to 180 degrees
- moved SW1 4.55 mm to (171.4, 33.0)
- renumbered C2 to C3, C3 to C4, R9 to R10, R10 to R11, R11 to R12, R12 to R13, R13 to R14, R14 to R15, R15 to R16, R16 to R17, R17 to R18, R18 to R19, R19 to R20, R20 to R21, R21 to R22, R22 to R23, R23 to R24, R24 to R25, R25 to R26, R26 to R27, R27 to R28, R28 to R29, R29 to R30, R30 to R31, R31 to R32, R32 to R33, R33 to R34, R34 to R35, R35 to R36, R36 to R37, R37 to R38, R38 to R39, R39 to R40, R40 to R41, R41 to R42, R42 to R43, R43 to R44, R44 to R45, R45 to R46, R46 to R47, R47 to R48, R48 to R49, R4 to R5, R49 to R50, R50 to R51, R51 to R52, R52 to R53, R53 to R54, R54 to R55, R55 to R56, R56 to R57, R57 to R58, R58 to R59, R5 to R6, R59 to R60, R60 to R61, R6 to R7, R7 to R8, R8 to R9
Connections:
- C3 pad 1: Net-(C2-Pad1) -> Net-(C3-Pad1)
- C4 pad 1: Net-(C3-Pad1) -> Net-(C4-Pad1)
- J2 pad 2: Net-(J2-Pad2) -> (no net)
- J2 pad 3: Net-(J2-Pad3) -> (no net)
- J2 pad 4: Net-(J2-Pad4) -> (no net)
- J2 pad 6: Net-(J2-Pad6) -> (no net)
- R1 pad 1: /usr -> Net-(C2-Pad1)
- R1 pad 2: GND -> Net-(R1-Pad2)
- R2 pad 1: Net-(C2-Pad1) -> Net-(C3-Pad1)
- R3 pad 1: Net-(C3-Pad1) -> Net-(C4-Pad1)
- SW1 pad 2: /usr -> Net-(R1-Pad2)
- U1 pad 1: Net-(C2-Pad1) -> (no net)
- U1 pad 10: Net-(U1-Pad10) -> /rst
- U1 pad 11: Net-(U1-Pad11) -> Net-(C4-Pad1)
- U1 pad 12: Net-(U1-Pad12) -> /clk
- U1 pad 13: Net-(U1-Pad13) -> Net-(C3-Pad1)
- U1 pad 2: /clk -> (no net)
- U1 pad 3: Net-(C3-Pad1) -> Net-(C2-Pad1)
- U1 pad 4: /rst -> /usr
- U1 pad 5: Net-(U1-Pad5) -> (no net)
- U1 pad 6: Net-(D4-Pad2) -> (no net)
- U1 pad 8: Net-(U1-Pad8) -> Net-(D4-Pad2)
- U10 pad 10: Net-(U10-Pad10) -> (no net)
- U10 pad 11: Net-(U10-Pad11) -> (no net)
- U10 pad 12: Net-(U10-Pad12) -> (no net)
- U10 pad 13: Net-(U10-Pad13) -> (no net)
- U10 pad 8: Net-(U10-Pad8) -> (no net)
- U10 pad 9: Net-(U10-Pad9) -> (no net)
- U15 pad 10: Net-(U15-Pad10) -> (no net)
- U15 pad 11: Net-(U15-Pad11) -> (no net)
- U15 pad 12: Net-(U15-Pad12) -> (no net)
- U15 pad 13: Net-(U15-Pad13) -> (no net)
- U2 pad 2: Net-(U2-Pad2) -> (no net)
- U2 pad 3: Net-(U2-Pad3) -> (no net)
- U2 pad 4: Net-(U2-Pad4) -> (no net)
- U2 pad 5: Net-(U2-Pad5) -> (no net)
- U2 pad 9: Net-(U2-Pad9) -> (no net)
- U4 pad 9: Net-(U4-Pad9) -> (no net)
- U5 pad 3: Net-(U1-Pad5) -> Net-(U1-Pad9)
Routing:
- net Net-(C2-Pad1): track 141.1 -> 57.5 mm
- net Net-(U1-Pad5): track 62.2 -> 0.00 mm, vias 4 -> 0
- net Net-(U1-Pad9): track 0.00 -> 54.6 mm, vias 0 -> 4
- net /usr: track 145.6 -> 179.3 mm, vias 0 -> 2
- net Net-(C4-Pad1): track 0.00 -> 30.1 mm, vias 0 -> 2
- net Net-(D4-Pad2): track 36.5 -> 23.8 mm
- net Net-(R1-Pad2): track 0.00 -> 11.4 mm
- net Net-(C3-Pad1): track 40.6 -> 49.3 mm, vias 2 -> 0

Commit message: Rotate U16 footprint 180 degrees
Parts:
- moved U16 17.0 mm to (149.9, 147.3), turned to 0 degrees
Connections:
- U16 pad 1: Net-(U14-Pad8) -> (no net)
- U16 pad 10: (no net) -> /z5
- U16 pad 11: (no net) -> Net-(U14-Pad6)
- U16 pad 12: (no net) -> /z4
- U16 pad 13: (no net) -> Net-(U14-Pad3)
- U16 pad 2: /z6 -> (no net)
- U16 pad 3: Net-(U14-Pad6) -> (no net)
- U16 pad 4: /z5 -> (no net)
- U16 pad 5: Net-(U14-Pad3) -> Net-(U14-Pad11)
- U16 pad 6: /z4 -> /z7
- U16 pad 8: /z7 -> /z6
- U16 pad 9: Net-(U14-Pad11) -> Net-(U14-Pad8)
Routing:
- net /z7: track 64.6 -> 51.3 mm
- net Net-(U14-Pad11): track 70.0 -> 64.9 mm
- net /z4: track 90.1 -> 93.0 mm
- net /z5: track 90.2 -> 93.2 mm
- net /z6: track 63.9 -> 61.4 mm
- net Net-(U14-Pad6): track 16.3 -> 17.3 mm
- net Net-(U14-Pad8): track 32.1 -> 33.1 mm
- net Net-(U14-Pad3): track 15.2 -> 16.3 mm
