File: midnight-sun-2019/led-matrix.sch (KiCad schematic (older format))
At the start: 826 parts

Commit message: Clean up circuit draft
Parts:
- removed R202, R203, R204, R205, R206, R207, R208, R209, R210, R211, R212, R213, R214, R215, R216, R217, R218, R219, R220, R221, R222, R223, R224, R225, R226, R227, R228, R229, R230, R231, R232, R233, R235, R236, R237, R238, R239, R240, R241, R242, R243, R244, R245, R246, R247, R248, R249, R250, R251, R252, R253, R254, R255, R256, R257, R258, R259, R260, R261, R262, R263, R264, R265, R266, R268, R269, R270, R271, R272, R273, R274, R275, R276, R277, R278, R279, R280, R281, R282, R283, R284, R285, R286, R287, R288, R289, R290, R291, R292, R293, R294, R295, R296, R297, R298, R299, R301, R302, R304, R305, R307, R308, R310, R311, R313, R314, R316, R317, R319, R320, R322, R323, R325, R326, R327, R328, R329, R330, R331, R332, R333, R334, R335, R336, R337, R338, R339, R340, R341, R342, R343, R344, R346, R347, R348, R349, R350, R351, R352, R353, R354, R355, R356, R357, R358, R359, R360, R361, R362, R363, R364, R366, R367, R368, R369, R370, R371, R372, R373, R374, R375, R376, R377, R378, R379, R380, R381, R382, R383, R384, R386, R387, R388, R389, R390, R391, R392, R393, R394, R395, R396, R397, R398, R399, R400, R401, R402, R403, R404, R406, R407, R408, R409, R410, R411, R412, R413, R414, R415, R416, R417, R418, R419, R420, R421, R422, R423, R424, R426, R427, R428, R429, R430, R431, R432, R433, R434, R435, R436, R437, R438, R439, R440, R441, R442, R443, R444, R446, R447, R448, R449, R450, R451, R452, R453, R454, R455, R456, R457, R458, R459, R460, R461, R462, R463, R464, R466, R467, R468, R469, R470, R471, R472, R473, R474, R475, R476, R477, R478, R479, R480, R481, R482, R483, R484, R486, R487, R488, R489, R490, R491, R492, R493, R494, R495, R496, R497, R498, R499, R500, R501, R503, R504, R505, R506, R507, R508, R509, R510, R511, R512, R513, R514, R515, R516, R517, R519, R520, R521, R522, R523, R524, R525, R526, R527, R528, R529, R530, R531, R532, R533, R535, R536, R537, R538, R539, R540, R541, R542, R543, R544, R545, R546, R547, R548, R549, R551, R552, R553, R554, R555, R556, R557, R558, R559, R560, R561, R562, R563, R564, R565, R567, R568, R569, R570, R571, R572, R573, R574, R575, R576, R577, R578, R579, R580, R581, R583, R584, R585, R586, R587, R588, R589, R590, R591, R592, R593, R594, R595, R596, R597, R599, R600, R601, R602, R603, R604, R605, R606, R607, R608, R609, R610, R611, R612, R613: R, symbol Device:R
- renumbered R234 to R202, R267 to R203, R300 to R204, R303 to R205, R306 to R206, R309 to R207, R312 to R208, R315 to R209, R318 to R210, R321 to R211, R324 to R212, R345 to R213, R365 to R214, R385 to R215, R405 to R216, R425 to R217, R445 to R218, R465 to R219, R485 to R220, R502 to R221, R518 to R222, R534 to R223, R550 to R224, R566 to R225, R582 to R226, R598 to R227
Connections:
- net at D612.2 (A): now also D599.2 (A), D600.2 (A), D601.2 (A), D602.2 (A), D603.2 (A), D604.2 (A), D605.2 (A), D606.2 (A), D607.2 (A), D608.2 (A), D609.2 (A), D610.2 (A)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
- net at D596.2 (A): now also D582.2 (A), D583.2 (A), D584.2 (A), D585.2 (A), D586.2 (A), D587.2 (A), D588.2 (A), D589.2 (A), D590.2 (A), D591.2 (A), D592.2 (A), D593.2 (A)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
- net at D580.2 (A): now also D566.2 (A), D567.2 (A), D568.2 (A), D569.2 (A), D570.2 (A), D571.2 (A), D572.2 (A), D573.2 (A), D574.2 (A), D575.2 (A), D576.2 (A), D577.2 (A)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
- net at D564.2 (A): now also D550.2 (A), D551.2 (A), D552.2 (A), D553.2 (A), D554.2 (A), D555.2 (A), D556.2 (A), D557.2 (A), D558.2 (A), D559.2 (A), D560.2 (A), D561.2 (A)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
- net at D548.2 (A): now also D534.2 (A), D535.2 (A), D536.2 (A), D537.2 (A), D538.2 (A), D539.2 (A), D540.2 (A), D541.2 (A), D542.2 (A), D543.2 (A), D544.2 (A), D545.2 (A)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
- net at D532.2 (A): now also D518.2 (A), D519.2 (A), D520.2 (A), D521.2 (A), D522.2 (A), D523.2 (A), D524.2 (A), D525.2 (A), D526.2 (A), D527.2 (A), D528.2 (A), D529.2 (A)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
- net at D516.2 (A): now also D502.2 (A), D503.2 (A), D504.2 (A), D505.2 (A), D506.2 (A), D507.2 (A), D508.2 (A), D509.2 (A), D510.2 (A), D511.2 (A), D512.2 (A), D513.2 (A)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
- net at D501.2 (A): now also D485.2 (A), D486.2 (A), D487.2 (A), D488.2 (A), D489.2 (A), D490.2 (A), D491.2 (A), D492.2 (A), D493.2 (A), D494.2 (A), D495.2 (A), D496.2 (A)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
- net at D484.2 (A): now also D465.2 (A), D466.2 (A), D467.2 (A), D468.2 (A), D469.2 (A), D470.2 (A), D471.2 (A), D472.2 (A), D473.2 (A), D474.2 (A), D475.2 (A), D476.2 (A)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
- net at D464.2 (A): now also D445.2 (A), D446.2 (A), D447.2 (A), D448.2 (A), D449.2 (A), D450.2 (A), D451.2 (A), D452.2 (A), D453.2 (A), D454.2 (A), D455.2 (A), D456.2 (A)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
- net at D444.2 (A): now also D425.2 (A), D426.2 (A), D427.2 (A), D428.2 (A), D429.2 (A), D430.2 (A), D431.2 (A), D432.2 (A), D433.2 (A), D434.2 (A), D435.2 (A), D436.2 (A)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
- net at D424.2 (A): now also D405.2 (A), D406.2 (A), D407.2 (A), D408.2 (A), D409.2 (A), D410.2 (A), D411.2 (A), D412.2 (A), D413.2 (A), D414.2 (A), D415.2 (A), D416.2 (A)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
- net at D404.2 (A): now also D385.2 (A), D386.2 (A), D387.2 (A), D388.2 (A), D389.2 (A), D390.2 (A), D391.2 (A), D392.2 (A), D393.2 (A), D394.2 (A), D395.2 (A), D396.2 (A)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
- net at D384.2 (A): now also D365.2 (A), D366.2 (A), D367.2 (A), D368.2 (A), D369.2 (A), D370.2 (A), D371.2 (A), D372.2 (A), D373.2 (A), D374.2 (A), D375.2 (A), D376.2 (A)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
- net at D364.2 (A): now also D345.2 (A), D346.2 (A), D347.2 (A), D348.2 (A), D349.2 (A), D350.2 (A), D351.2 (A), D352.2 (A), D353.2 (A), D354.2 (A), D355.2 (A), D356.2 (A)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
- net at D344.2 (A): now also D324.2 (A), D325.2 (A), D326.2 (A), D327.2 (A), D328.2 (A), D329.2 (A), D330.2 (A), D331.2 (A), D332.2 (A), D333.2 (A), D334.2 (A), D335.2 (A)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
- net at D312.2 (A), R208.1: now also D313.2 (A), D314.2 (A)
- net at D315.2 (A), R209.1: now also D316.2 (A), D317.2 (A)
- net at D318.2 (A), R210.1: now also D319.2 (A), D320.2 (A)
- net at D321.2 (A), R211.1: now also D322.2 (A), D323.2 (A)
- net at D300.2 (A), R204.1: now also D301.2 (A), D302.2 (A)
- net at D303.2 (A), R205.1: now also D304.2 (A), D305.2 (A)
- net at D306.2 (A), R206.1: now also D307.2 (A), D308.2 (A)
- net at D309.2 (A), R207.1: now also D310.2 (A), D311.2 (A)
- net at D299.2 (A): now also D267.2 (A), D268.2 (A), D269.2 (A), D270.2 (A), D271.2 (A), D272.2 (A), D273.2 (A), D274.2 (A), D275.2 (A), D276.2 (A), D277.2 (A), D278.2 (A)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
- net at D266.2 (A): now also D234.2 (A), D235.2 (A), D236.2 (A), D237.2 (A), D238.2 (A), D239.2 (A), D240.2 (A), D241.2 (A), D242.2 (A), D243.2 (A), D244.2 (A), D245.2 (A)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
- net at D233.2 (A): now also D201.2 (A), D202.2 (A), D203.2 (A), D204.2 (A), D205.2 (A), D206.2 (A), D207.2 (A), D208.2 (A), D209.2 (A), D210.2 (A), D211.2 (A), D212.2 (A)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

Commit message: WIP: schematic
Parts:
- D201, D202, D203, D204, D205, D206, D207, D208, D209, D210, D211, D212, D213, D214, D215, D216, D217, D218, D219, D220, D221, D222, D223, D224, D225, D226, D227, D228, D229, D230, D231, D232, D233, D234, D235, D236, D237, D238, D239, D240, D241, D242, D243, D244, D245, D246, D247, D248, D249, D250, D251, D252, D253, D254, D255, D256, D257, D258, D259, D260, D261, D262, D263, D264, D265, D266, D267, D268, D269, D270, D271, D272, D273, D274, D275, D276, D277, D278, D279, D280, D281, D282, D283, D284, D285, D286, D287, D288, D289, D290, D291, D292, D293, D294, D295, D296, D297, D298, D299, D300, D301, D302, D303, D304, D305, D306, D307, D308, D309, D310, D311, D312, D313, D314, D315, D316, D317, D318, D319, D320, D321, D322, D323, D324, D325, D326, D327, D328, D329, D330, D331, D332, D333, D334, D335, D336, D337, D338, D339, D340, D341, D342, D343, D344, D345, D346, D347, D348, D349, D350, D351, D352, D353, D354, D355, D356, D357, D358, D359, D360, D361, D362, D363, D364, D365, D366, D367, D368, D369, D370, D371, D372, D373, D374, D375, D376, D377, D378, D379, D380, D381, D382, D383, D384, D385, D386, D387, D388, D389, D390, D391, D392, D393, D394, D395, D396, D397, D398, D399, D400, D401, D402, D403, D404, D405, D406, D407, D408, D409, D410, D411, D412, D413, D414, D415, D416, D417, D418, D419, D420, D421, D422, D423, D424, D425, D426, D427, D428, D429, D430, D431, D432, D433, D434, D435, D436, D437, D438, D439, D440, D441, D442, D443, D444, D445, D446, D447, D448, D449, D450, D451, D452, D453, D454, D455, D456, D457, D458, D459, D460, D461, D462, D463, D464, D465, D466, D467, D468, D469, D470, D471, D472, D473, D474, D475, D476, D477, D478, D479, D480, D481, D482, D483, D484, D485, D486, D487, D488, D489, D490, D491, D492, D493, D494, D495, D496, D497, D498, D499, D500, D501, D502, D503, D504, D505, D506, D507, D508, D509, D510, D511, D512, D513, D514, D515, D516, D517, D518, D519, D520, D521, D522, D523, D524, D525, D526, D527, D528, D529, D530, D531, D532, D533, D534, D535, D536, D537, D538, D539, D540, D541, D542, D543, D544, D545, D546, D547, D548, D549, D550, D551, D552, D553, D554, D555, D556, D557, D558, D559, D560, D561, D562, D563, D564, D565, D566, D567, D568, D569, D570, D571, D572, D573, D574, D575, D576, D577, D578, D579, D580, D581, D582, D583, D584, D585, D586, D587, D588, D589, D590, D591, D592, D593, D594, D595, D596, D597, D598, D599, D600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: footprint (none) -> LED_SMD:LED_0805_2012Metric_Castellated
- R201, R202, R203, R204, R205, R206, R207, R208, R209, R210, R211, R212, R213, R214, R215, R216, R217, R218, R219, R220, R221, R222, R223, R224, R225, R226, R227: footprint (none) -> Resistor_SMD:R_0805_2012Metric_Pad1.15x1.40mm_HandSolder

Commit message: Wire up all the logic
Parts:
- added D324, D325, D326, D327, D328, D329, D330, D331, D332, D333, D334, D335, D336, D337, D338, D339, D340, D341, D342, D343, D344, D345, D346, D347: LED, LED_SMD:LED_0805_2012Metric_Castellated, symbol Device:LED
- added R212, R213, R214, R215, R216, R217, R218, R219: R, Resistor_SMD:R_0805_2012Metric_Pad1.15x1.40mm_HandSolder, symbol Device:R
- renumbered D324 to D348, D325 to D349, D326 to D350, D327 to D351, D328 to D352, D329 to D353, D330 to D354, D331 to D355, D332 to D356, D333 to D357, D334 to D358, D335 to D359, D336 to D360, D337 to D361, D338 to D362, D339 to D363, D340 to D364, D341 to D365, D342 to D366, D343 to D367, D344 to D368, D345 to D369, D346 to D370, D347 to D371, D348 to D372, D349 to D373, D350 to D374, D351 to D375, D352 to D376, D353 to D377, D354 to D378, D355 to D379, D356 to D380, D357 to D381, D358 to D382, D359 to D383, D360 to D384, D361 to D385, D362 to D386, D363 to D387, D364 to D388, D365 to D389, D366 to D390, D367 to D391, D368 to D392, D369 to D393, D370 to D394, D371 to D395, D372 to D396, D373 to D397, D374 to D398, D375 to D399, D376 to D400, D377 to D401, D378 to D402, D379 to D403, D380 to D404, D381 to D405, D382 to D406, D383 to D407, D384 to D408, D385 to D409, D386 to D410, D387 to D411, D388 to D412, D389 to D413, D390 to D414, D391 to D415, D392 to D416, D393 to D417, D394 to D418, D395 to D419, D396 to D420, D397 to D421, D398 to D422, D399 to D423, D400 to D424, D401 to D425, D402 to D426, D403 to D427, D404 to D428, D405 to D429, D406 to D430, D407 to D431, D408 to D432, D409 to D433, D410 to D434, D411 to D435, D412 to D436, D413 to D437, D414 to D438, D415 to D439, D416 to D440, D417 to D441, D418 to D442, D419 to D443, D420 to D444, D421 to D445, D422 to D446, D423 to D447, D424 to D448, D425 to D449, D426 to D450, D427 to D451, D428 to D452, D429 to D453, D430 to D454, D431 to D455, D432 to D456, D433 to D457, D434 to D458, D435 to D459, D436 to D460, D437 to D461, D438 to D462, D439 to D463, D440 to D464, D441 to D465, D442 to D466, D443 to D467, D444 to D468, D445 to D469, D446 to D470, D447 to D471, D448 to D472, D449 to D473, D450 to D474, D451 to D475, D452 to D476, D453 to D477, D454 to D478, D455 to D479, D456 to D480, D457 to D481, D458 to D482, D459 to D483, D460 to D484, D461 to D485, D462 to D486, D463 to D487, D464 to D488, D465 to D489, D466 to D490, D467 to D491, D468 to D492, D469 to D493, D470 to D494, D471 to D495, D472 to D496, D473 to D497, D474 to D498, D475 to D499, D476 to D500, D477 to D501, D478 to D502, D479 to D503, D480 to D504, D481 to D505, D482 to D506, D483 to D507, D484 to D508, D485 to D509, D486 to D510, D487 to D511, D488 to D512, D489 to D513, D490 to D514, D491 to D515, D492 to D516, D493 to D517, D494 to D518, D495 to D519, D496 to D520, D497 to D521, D498 to D522, D499 to D523, D500 to D524, D501 to D525, D502 to D526, D503 to D527, D504 to D528, D505 to D529, D506 to D530, D507 to D531, D508 to D532, D509 to D533, D510 to D534, D511 to D535, D512 to D536, D513 to D537, D514 to D538, D515 to D539, D516 to D540, D517 to D541, D518 to D542, D519 to D543, D520 to D544, D521 to D545, D522 to D546, D523 to D547, D524 to D548, D525 to D549, D526 to D550, D527 to D551, D528 to D552, D529 to D553, D530 to D554, D531 to D555, D532 to D556, D533 to D557, D534 to D558, D535 to D559, D536 to D560, D537 to D561, D538 to D562, D539 to D563, D540 to D564, D541 to D565, D542 to D566, D543 to D567, D544 to D568, D545 to D569, D546 to D570, D547 to D571, D548 to D572, D549 to D573, D550 to D574, D551 to D575, D552 to D576, D553 to D577, D554 to D578, D555 to D579, D556 to D580, D557 to D581, D558 to D582, D559 to D583, D560 to D584, D561 to D585, D562 to D586, D563 to D587, D564 to D588, D565 to D589, D566 to D590, D567 to D591, D568 to D592, D569 to D593, D570 to D594, D571 to D595, D572 to D596, D573 to D597, D574 to D598, D575 to D599, D576 to D600, D577 to D601, D578 to D602, D579 to D603, D580 to D604, D581 to D605, D582 to D606, D583 to D607, D584 to D608, D585 to D609, D586 to D610, D587 to D611, D588 to D612, D589 to D613, D590 to D614, D591 to D615, D592 to D616, D593 to D617, D594 to D618, D595 to D619, D596 to D620, D597 to D621, D598 to D622, D599 to D623, D600 to D624, D601 to D625, D602 to D626, D603 to D627, D604 to D628, D605 to D629, D606 to D630, D607 to D631, D608 to D632, D609 to D633, D610 to D634, D611 to D635, D612 to D636, D613 to D637, R212 to R220, R213 to R221, R214 to R222, R215 to R223, R216 to R224, R217 to R225, R218 to R226, R219 to R227, R220 to R228, R221 to R229, R222 to R230, R223 to R231, R224 to R232, R225 to R233, R226 to R234, R227 to R235
Connections:
- net GND: now also D324.1 (K), D325.1 (K), D326.1 (K), D327.1 (K), D328.1 (K), D329.1 (K), D330.1 (K), D331.1 (K), D332.1 (K), D333.1 (K), D334.1 (K), D335.1 (K), D336.1 (K), D337.1 (K), D338.1 (K), D339.1 (K), D340.1 (K), D341.1 (K), D342.1 (K), D343.1 (K), D344.1 (K), D345.1 (K), D346.1 (K), D347.1 (K)
- new net: D336.2 (A), D337.2 (A), D338.2 (A), R216.1
- new net: D339.2 (A), D340.2 (A), D341.2 (A), R217.1
- new net: D342.2 (A), D343.2 (A), D344.2 (A), R218.1
- new net: D345.2 (A), D346.2 (A), D347.2 (A), R219.1
- new net: D324.2 (A), D325.2 (A), D326.2 (A), R212.1
- new net: D327.2 (A), D328.2 (A), D329.2 (A), R213.1
- new net: D330.2 (A), D331.2 (A), D332.2 (A), R214.1
- new net: D333.2 (A), D334.2 (A), D335.2 (A), R215.1
- new net b10: R214.2
- new net b11: R215.2
- new net b12: R216.2
- new net b13: R217.2
- new net b14: R218.2
- new net b15: R219.2
- new net b8: R212.2
- new net b9: R213.2

Commit message: Update QR code to real flag
Parts:
- removed D525, D573, D589, D605, D621, D637: LED, LED_SMD:LED_0805_2012Metric_Castellated, symbol Device:LED
- added D369, D390, D391, D412, D413, D434, D455, D476, D497, D518: LED, LED_SMD:LED_0805_2012Metric_Castellated, symbol Device:LED
- renumbered D369 to D370, D370 to D371, D371 to D372, D372 to D373, D373 to D374, D374 to D375, D375 to D376, D376 to D377, D377 to D378, D378 to D379, D379 to D380, D380 to D381, D381 to D382, D382 to D383, D383 to D384, D384 to D385, D385 to D386, D386 to D387, D387 to D388, D388 to D389, D389 to D392, D390 to D393, D391 to D394, D392 to D395, D393 to D396, D394 to D397, D395 to D398, D396 to D399, D397 to D400, D398 to D401, D399 to D402, D400 to D403, D401 to D404, D402 to D405, D403 to D406, D404 to D407, D405 to D408, D406 to D409, D407 to D410, D408 to D411, D409 to D414, D410 to D415, D411 to D416, D412 to D417, D413 to D418, D414 to D419, D415 to D420, D416 to D421, D417 to D422, D418 to D423, D419 to D424, D420 to D425, D421 to D426, D422 to D427, D423 to D428, D424 to D429, D425 to D430, D426 to D431, D427 to D432, D428 to D433, D429 to D435, D430 to D436, D431 to D437, D432 to D438, D433 to D439, D434 to D440, D435 to D441, D436 to D442, D437 to D443, D438 to D444, D439 to D445, D440 to D446, D441 to D447, D442 to D448, D443 to D449, D444 to D450, D445 to D451, D446 to D452, D447 to D453, D448 to D454, D449 to D456, D450 to D457, D451 to D458, D452 to D459, D453 to D460, D454 to D461, D455 to D462, D456 to D463, D457 to D464, D458 to D465, D459 to D466, D460 to D467, D461 to D468, D462 to D469, D463 to D470, D464 to D471, D465 to D472, D466 to D473, D467 to D474, D468 to D475, D469 to D477, D470 to D478, D471 to D479, D472 to D480, D473 to D481, D474 to D482, D475 to D483, D476 to D484, D477 to D485, D478 to D486, D479 to D487, D480 to D488, D481 to D489, D482 to D490, D483 to D491, D484 to D492, D485 to D493, D486 to D494, D487 to D495, D488 to D496, D489 to D498, D490 to D499, D491 to D500, D492 to D501, D493 to D502, D494 to D503, D495 to D504, D496 to D505, D497 to D506, D498 to D507, D499 to D508, D500 to D509, D501 to D510, D502 to D511, D503 to D512, D504 to D513, D505 to D514, D506 to D515, D507 to D516, D508 to D517, D509 to D519, D510 to D520, D511 to D521, D512 to D522, D513 to D523, D514 to D524, D515 to D525, D516 to D526, D517 to D527, D518 to D528, D519 to D529, D520 to D530, D521 to D531, D522 to D532, D523 to D533, D524 to D534, D526 to D535, D527 to D536, D528 to D537, D529 to D538, D530 to D539, D531 to D540, D532 to D541, D533 to D542, D534 to D543, D535 to D544, D536 to D545, D537 to D546, D538 to D547, D539 to D548, D540 to D549, D541 to D550, D542 to D551, D543 to D552, D544 to D553, D545 to D554, D546 to D555, D547 to D556, D548 to D557, D549 to D558, D550 to D559, D551 to D560, D552 to D561, D553 to D562, D554 to D563, D555 to D564, D556 to D565, D557 to D566, D558 to D567, D559 to D568, D560 to D569, D561 to D570, D562 to D571, D563 to D572, D564 to D573, D565 to D574, D566 to D575, D567 to D576, D568 to D577, D569 to D578, D570 to D579, D571 to D580, D572 to D581, D574 to D582, D575 to D583, D576 to D584, D577 to D585, D578 to D586, D579 to D587, D580 to D588, D581 to D589, D582 to D590, D583 to D591, D584 to D592, D585 to D593, D586 to D594, D587 to D595, D588 to D596, D590 to D597, D591 to D598, D592 to D599, D593 to D600, D594 to D601, D595 to D602, D596 to D603, D597 to D604, D598 to D605, D599 to D606, D600 to D607, D601 to D608, D602 to D609, D603 to D610, D604 to D611, D606 to D612, D607 to D613, D608 to D614, D609 to D615, D610 to D616, D611 to D617, D612 to D618, D613 to D619, D614 to D620, D615 to D621, D616 to D622, D617 to D623, D618 to D624, D619 to D625, D620 to D626, D622 to D627, D623 to D628, D624 to D629, D625 to D630, D626 to D631, D627 to D632, D628 to D633, D629 to D634, D630 to D635, D631 to D636, D632 to D637, D633 to D638, D634 to D639, D635 to D640, D636 to D641
Connections:
- net GND: now also D369.1 (K), D390.1 (K), D391.1 (K), D412.1 (K), D413.1 (K), D434.1 (K), D455.1 (K), D476.1 (K), D497.1 (K), D518.1 (K)
- net at D498.2 (A), D499.2 (A), D500.2 (A)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: now also D518.2 (A)
- net at D477.2 (A), D478.2 (A), D479.2 (A)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: now also D497.2 (A)
- net at D456.2 (A), D457.2 (A), D458.2 (A)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: now also D476.2 (A)
- net at D435.2 (A), D436.2 (A), D437.2 (A)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: now also D455.2 (A)
- net at D414.2 (A), D415.2 (A), D416.2 (A)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: now also D434.2 (A)
- net at D392.2 (A), D393.2 (A), D394.2 (A)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: now also D412.2 (A), D413.2 (A)
- net at D370.2 (A), D371.2 (A), D372.2 (A)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: now also D390.2 (A), D391.2 (A)
- net at D348.2 (A), D349.2 (A), D350.2 (A)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: now also D369.2 (A)

Commit message: Swap positions of LEDs and Rs in matrix
Connections:
- net GND: now also R201.1, R202.1, R203.1, R204.1, R205.1, R206.1, R207.1, R208.1, R209.1, R210.1, R211.1, R212.1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; no longer D201.1 (K), D202.1 (K), D203.1 (K), D204.1 (K), D205.1 (K), D206.1 (K), D207.1 (K), D208.1 (K), D209.1 (K), D210.1 (K), D211.1 (K), D212.1 (K)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
- net a0: now also D201.2 (A), D202.2 (A), D203.2 (A), D204.2 (A), D205.2 (A), D206.2 (A), D207.2 (A), D208.2 (A), D209.2 (A), D210.2 (A), D211.2 (A), D212.2 (A)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; no longer R201.2
- net a1: now also D234.2 (A), D235.2 (A), D236.2 (A), D237.2 (A), D238.2 (A), D239.2 (A), D240.2 (A), D241.2 (A), D242.2 (A), D243.2 (A), D244.2 (A), D245.2 (A)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; no longer R202.2
- net a2: now also D267.2 (A), D268.2 (A), D269.2 (A), D270.2 (A), D271.2 (A), D272.2 (A), D273.2 (A), D274.2 (A), D275.2 (A), D276.2 (A), D277.2 (A), D278.2 (A)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; no longer R203.2
- net b0: now also D300.2 (A), D301.2 (A), D302.2 (A); no longer R204.2
- net b1: now also D303.2 (A), D304.2 (A), D305.2 (A); no longer R205.2
- net b10: now also D330.2 (A), D331.2 (A), D332.2 (A); no longer R214.2
- net b11: now also D333.2 (A), D334.2 (A), D335.2 (A); no longer R215.2
- net b12: now also D336.2 (A), D337.2 (A), D338.2 (A); no longer R216.2
- net b13: now also D339.2 (A), D340.2 (A), D341.2 (A); no longer R217.2
- net b14: now also D342.2 (A), D343.2 (A), D344.2 (A); no longer R218.2
- net b15: now also D345.2 (A), D346.2 (A), D347.2 (A); no longer R219.2
- net b2: now also D306.2 (A), D307.2 (A), D308.2 (A); no longer R206.2
- net b3: now also D309.2 (A), D310.2 (A), D311.2 (A); no longer R207.2
- net b4: now also D312.2 (A), D313.2 (A), D314.2 (A); no longer R208.2
- net b5: now also D315.2 (A), D316.2 (A), D317.2 (A); no longer R209.2
- net b6: now also D318.2 (A), D319.2 (A), D320.2 (A); no longer R210.2
- net b7: now also D321.2 (A), D322.2 (A), D323.2 (A); no longer R211.2
- net b8: now also D324.2 (A), D325.2 (A), D326.2 (A); no longer R212.2
- net b9: now also D327.2 (A), D328.2 (A), D329.2 (A); no longer R213.2
- net o0: now also D519.2 (A), D520.2 (A), D521.2 (A), D522.2 (A), D523.2 (A), D524.2 (A), D525.2 (A), D526.2 (A), D527.2 (A), D528.2 (A), D529.2 (A), D530.2 (A)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; no longer R228.2
- net o1: now also D535.2 (A), D536.2 (A), D537.2 (A), D538.2 (A), D539.2 (A), D540.2 (A), D541.2 (A), D542.2 (A), D543.2 (A), D544.2 (A), D545.2 (A), D546.2 (A)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; no longer R229.2
- net o2: now also D551.2 (A), D552.2 (A), D553.2 (A), D554.2 (A), D555.2 (A), D556.2 (A), D557.2 (A), D558.2 (A), D559.2 (A), D560.2 (A), D561.2 (A), D562.2 (A)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; no longer R230.2
- net o3: now also D567.2 (A), D568.2 (A), D569.2 (A), D570.2 (A), D571.2 (A), D572.2 (A), D573.2 (A), D574.2 (A), D575.2 (A), D576.2 (A), D577.2 (A), D578.2 (A)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; no longer R231.2
- net o4: now also D582.2 (A), D583.2 (A), D584.2 (A), D585.2 (A), D586.2 (A), D587.2 (A), D588.2 (A), D589.2 (A), D590.2 (A), D591.2 (A), D592.2 (A), D593.2 (A)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; no longer R232.2
- net o5: now also D597.2 (A), D598.2 (A), D599.2 (A), D600.2 (A), D601.2 (A), D602.2 (A), D603.2 (A), D604.2 (A), D605.2 (A), D606.2 (A), D607.2 (A), D608.2 (A)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; no longer R233.2
- net o6: now also D612.2 (A), D613.2 (A), D614.2 (A), D615.2 (A), D616.2 (A), D617.2 (A), D618.2 (A), D619.2 (A), D620.2 (A), D621.2 (A), D622.2 (A), D623.2 (A)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; no longer R234.2
- net o7: now also D627.2 (A); no longer R235.2
- net z0: now also D348.2 (A), D349.2 (A), D350.2 (A), D351.2 (A), D352.2 (A), D353.2 (A), D354.2 (A), D355.2 (A), D356.2 (A), D357.2 (A), D358.2 (A), D359.2 (A)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; no longer R220.2
- net z1: now also D370.2 (A), D371.2 (A), D372.2 (A), D373.2 (A), D374.2 (A), D375.2 (A), D376.2 (A), D377.2 (A), D378.2 (A), D379.2 (A), D380.2 (A), D381.2 (A)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; no longer R221.2
- net z2: now also D392.2 (A), D393.2 (A), D394.2 (A), D395.2 (A), D396.2 (A), D397.2 (A), D398.2 (A), D399.2 (A), D400.2 (A), D401.2 (A), D402.2 (A), D403.2 (A)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; no longer R222.2
- net z3: now also D414.2 (A), D415.2 (A), D416.2 (A), D417.2 (A), D418.2 (A), D419.2 (A), D420.2 (A), D421.2 (A), D422.2 (A), D423.2 (A), D424.2 (A), D425.2 (A)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; no longer R223.2
- net z4: now also D435.2 (A), D436.2 (A), D437.2 (A), D438.2 (A), D439.2 (A), D440.2 (A), D441.2 (A), D442.2 (A), D443.2 (A), D444.2 (A), D445.2 (A), D446.2 (A)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; no longer R224.2
- net z5: now also D456.2 (A), D457.2 (A), D458.2 (A), D459.2 (A), D460.2 (A), D461.2 (A), D462.2 (A), D463.2 (A), D464.2 (A), D465.2 (A), D466.2 (A), D467.2 (A)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; no longer R225.2
- net z6: now also D477.2 (A), D478.2 (A), D479.2 (A), D480.2 (A), D481.2 (A), D482.2 (A), D483.2 (A), D484.2 (A), D485.2 (A), D486.2 (A), D487.2 (A), D488.2 (A)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; no longer R226.2
- net z7: now also D498.2 (A), D499.2 (A), D500.2 (A), D501.2 (A), D502.2 (A), D503.2 (A), D504.2 (A), D505.2 (A), D506.2 (A), D507.2 (A), D508.2 (A), D509.2 (A)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; no longer R227.2
- new net: D336.1 (K), D337.1 (K), D338.1 (K), R216.2
- new net: D339.1 (K), D340.1 (K), D341.1 (K), R217.2
- new net: D342.1 (K), D343.1 (K), D344.1 (K), R218.2
- new net: D345.1 (K), D346.1 (K), D347.1 (K), R219.2
- new net: D324.1 (K), D325.1 (K), D326.1 (K), R212.2
- new net: D327.1 (K), D328.1 (K), D329.1 (K), R213.2
- new net: D330.1 (K), D331.1 (K), D332.1 (K), R214.2
- new net: D333.1 (K), D334.1 (K), D335.1 (K), R215.2
- new net: D348.1 (K), D349.1 (K), D350.1 (K), D351.1 (K), D352.1 (K), D353.1 (K), D354.1 (K), D355.1 (K), D356.1 (K), D357.1 (K), D358.1 (K), D359.1 (K)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
- new net: D370.1 (K), D371.1 (K), D372.1 (K), D373.1 (K), D374.1 (K), D375.1 (K), D376.1 (K), D377.1 (K), D378.1 (K), D379.1 (K), D380.1 (K), D381.1 (K)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
- new net: D392.1 (K), D393.1 (K), D394.1 (K), D395.1 (K), D396.1 (K), D397.1 (K), D398.1 (K), D399.1 (K), D400.1 (K), D401.1 (K), D402.1 (K), D403.1 (K)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
- new net: D414.1 (K), D415.1 (K), D416.1 (K), D417.1 (K), D418.1 (K), D419.1 (K), D420.1 (K), D421.1 (K), D422.1 (K), D423.1 (K), D424.1 (K), D425.1 (K)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
- new net: D435.1 (K), D436.1 (K), D437.1 (K), D438.1 (K), D439.1 (K), D440.1 (K), D441.1 (K), D442.1 (K), D443.1 (K), D444.1 (K), D445.1 (K), D446.1 (K)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
- new net: D627.1 (K), D628.1 (K), D629.1 (K), D630.1 (K), D631.1 (K), D632.1 (K), D633.1 (K), D634.1 (K), D635.1 (K), D636.1 (K), D637.1 (K), D638.1 (K)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
- new net: D612.1 (K), D613.1 (K), D614.1 (K), D615.1 (K), D616.1 (K), D617.1 (K), D618.1 (K), D619.1 (K), D620.1 (K), D621.1 (K), D622.1 (K), D623.1 (K)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
- new net: D597.1 (K), D598.1 (K), D599.1 (K), D600.1 (K), D601.1 (K), D602.1 (K), D603.1 (K), D604.1 (K), D605.1 (K), D606.1 (K), D607.1 (K), D608.1 (K)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
- new net: D582.1 (K), D583.1 (K), D584.1 (K), D585.1 (K), D586.1 (K), D587.1 (K), D588.1 (K), D589.1 (K), D590.1 (K), D591.1 (K), D592.1 (K), D593.1 (K)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
- new net: D567.1 (K), D568.1 (K), D569.1 (K), D570.1 (K), D571.1 (K), D572.1 (K), D573.1 (K), D574.1 (K), D575.1 (K), D576.1 (K), D577.1 (K), D578.1 (K)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
- new net: D551.1 (K), D552.1 (K), D553.1 (K), D554.1 (K), D555.1 (K), D556.1 (K), D557.1 (K), D558.1 (K), D559.1 (K), D560.1 (K), D561.1 (K), D562.1 (K)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
- new net: D535.1 (K), D536.1 (K), D537.1 (K), D538.1 (K), D539.1 (K), D540.1 (K), D541.1 (K), D542.1 (K), D543.1 (K), D544.1 (K), D545.1 (K), D546.1 (K)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
- new net: D519.1 (K), D520.1 (K), D521.1 (K), D522.1 (K), D523.1 (K), D524.1 (K), D525.1 (K), D526.1 (K), D527.1 (K), D528.1 (K), D529.1 (K), D530.1 (K)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
- new net: D498.1 (K), D499.1 (K), D500.1 (K), D501.1 (K), D502.1 (K), D503.1 (K), D504.1 (K), D505.1 (K), D506.1 (K), D507.1 (K), D508.1 (K), D509.1 (K)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
- new net: D477.1 (K), D478.1 (K), D479.1 (K), D480.1 (K), D481.1 (K), D482.1 (K), D483.1 (K), D484.1 (K), D485.1 (K), D486.1 (K), D487.1 (K), D488.1 (K)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
- new net: D456.1 (K), D457.1 (K), D458.1 (K), D459.1 (K), D460.1 (K), D461.1 (K), D462.1 (K), D463.1 (K), D464.1 (K), D465.1 (K), D466.1 (K), D467.1 (K)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
- new net: D312.1 (K), D313.1 (K), D314.1 (K), R208.2
- new net: D315.1 (K), D316.1 (K), D317.1 (K), R209.2
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Other:
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
Commit message: Work on laying out the LED matrix
Connections:
- net o7: now also D628.2 (A), D629.2 (A), D630.2 (A), D631.2 (A), D632.2 (A), D633.2 (A), D634.2 (A), D635.2 (A), D636.2 (A), D637.2 (A), D638.2 (A), D639.2 (A), D640.2 (A), D641.2 (A)
Changed lines of the file:
@@
 Wire Wire Line
 	6850 6800 6850 6900
-Wire Wire Line
-	6850 7900 6850 7950
 Connection ~ 6850 7950
 Wire Wire Line
@@
 Connection ~ 7150 5500
 Connection ~ 7150 7850
+Wire Wire Line
+	6850 7850 6850 7950
+Connection ~ 6850 7850
 $EndSCHEMATC

Commit message: Swap positions of LEDs and Rs in matrix
Connections:
- net GND: now also D201.1 (K), D202.1 (K), D203.1 (K), D204.1 (K), D205.1 (K), D206.1 (K), D207.1 (K), D208.1 (K), D209.1 (K), D210.1 (K), D211.1 (K), D212.1 (K)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; no longer R201.1, R202.1, R203.1, R204.1, R205.1, R206.1, R207.1, R208.1, R209.1, R210.1, R211.1, R212.1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
- net a0: now also R201.2; no longer D201.2 (A), D202.2 (A), D203.2 (A), D204.2 (A), D205.2 (A), D206.2 (A), D207.2 (A), D208.2 (A), D209.2 (A), D210.2 (A), D211.2 (A), D212.2 (A)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
- net a1: now also R202.2; no longer D234.2 (A), D235.2 (A), D236.2 (A), D237.2 (A), D238.2 (A), D239.2 (A), D240.2 (A), D241.2 (A), D242.2 (A), D243.2 (A), D244.2 (A), D245.2 (A)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
- net a2: now also R203.2; no longer D267.2 (A), D268.2 (A), D269.2 (A), D270.2 (A), D271.2 (A), D272.2 (A), D273.2 (A), D274.2 (A), D275.2 (A), D276.2 (A), D277.2 (A), D278.2 (A)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
- net b0: now also R204.2; no longer D300.2 (A), D301.2 (A), D302.2 (A)
- net b1: now also R205.2; no longer D303.2 (A), D304.2 (A), D305.2 (A)
- net b10: now also R214.2; no longer D330.2 (A), D331.2 (A), D332.2 (A)
- net b11: now also R215.2; no longer D333.2 (A), D334.2 (A), D335.2 (A)
- net b12: now also R216.2; no longer D336.2 (A), D337.2 (A), D338.2 (A)
- net b13: now also R217.2; no longer D339.2 (A), D340.2 (A), D341.2 (A)
- net b14: now also R218.2; no longer D342.2 (A), D343.2 (A), D344.2 (A)
- net b15: now also R219.2; no longer D345.2 (A), D346.2 (A), D347.2 (A)
- net b2: now also R206.2; no longer D306.2 (A), D307.2 (A), D308.2 (A)
- net b3: now also R207.2; no longer D309.2 (A), D310.2 (A), D311.2 (A)
- net b4: now also R208.2; no longer D312.2 (A), D313.2 (A), D314.2 (A)
- net b5: now also R209.2; no longer D315.2 (A), D316.2 (A), D317.2 (A)
- net b6: now also R210.2; no longer D318.2 (A), D319.2 (A), D320.2 (A)
- net b7: now also R211.2; no longer D321.2 (A), D322.2 (A), D323.2 (A)
- net b8: now also R212.2; no longer D324.2 (A), D325.2 (A), D326.2 (A)
- net b9: now also R213.2; no longer D327.2 (A), D328.2 (A), D329.2 (A)
- net o0: now also R228.2; no longer D519.2 (A), D520.2 (A), D521.2 (A), D522.2 (A), D523.2 (A), D524.2 (A), D525.2 (A), D526.2 (A), D527.2 (A), D528.2 (A), D529.2 (A), D530.2 (A)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
- net o1: now also R229.2; no longer D535.2 (A), D536.2 (A), D537.2 (A), D538.2 (A), D539.2 (A), D540.2 (A), D541.2 (A), D542.2 (A), D543.2 (A), D544.2 (A), D545.2 (A), D546.2 (A)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
- net o2: now also R230.2; no longer D551.2 (A), D552.2 (A), D553.2 (A), D554.2 (A), D555.2 (A), D556.2 (A), D557.2 (A), D558.2 (A), D559.2 (A), D560.2 (A), D561.2 (A), D562.2 (A)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
- net o3: now also R231.2; no longer D567.2 (A), D568.2 (A), D569.2 (A), D570.2 (A), D571.2 (A), D572.2 (A), D573.2 (A), D574.2 (A), D575.2 (A), D576.2 (A), D577.2 (A), D578.2 (A)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
- net o4: now also R232.2; no longer D582.2 (A), D583.2 (A), D584.2 (A), D585.2 (A), D586.2 (A), D587.2 (A), D588.2 (A), D589.2 (A), D590.2 (A), D591.2 (A), D592.2 (A), D593.2 (A)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
- net o5: now also R233.2; no longer D597.2 (A), D598.2 (A), D599.2 (A), D600.2 (A), D601.2 (A), D602.2 (A), D603.2 (A), D604.2 (A), D605.2 (A), D606.2 (A), D607.2 (A), D608.2 (A)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
- net o6: now also R234.2; no longer D612.2 (A), D613.2 (A), D614.2 (A), D615.2 (A), D616.2 (A), D617.2 (A), D618.2 (A), D619.2 (A), D620.2 (A), D621.2 (A), D622.2 (A), D623.2 (A)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
- net o7: now also R235.2; no longer D627.2 (A), D628.2 (A), D629.2 (A), D630.2 (A), D631.2 (A), D632.2 (A), D633.2 (A), D634.2 (A), D635.2 (A), D636.2 (A), D637.2 (A), D638.2 (A)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
- net z0: now also R220.2; no longer D348.2 (A), D349.2 (A), D350.2 (A), D351.2 (A), D352.2 (A), D353.2 (A), D354.2 (A), D355.2 (A), D356.2 (A), D357.2 (A), D358.2 (A), D359.2 (A)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
- net z1: now also R221.2; no longer D370.2 (A), D371.2 (A), D372.2 (A), D373.2 (A), D374.2 (A), D375.2 (A), D376.2 (A), D377.2 (A), D378.2 (A), D379.2 (A), D380.2 (A), D381.2 (A)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
- net z2: now also R222.2; no longer D392.2 (A), D393.2 (A), D394.2 (A), D395.2 (A), D396.2 (A), D397.2 (A), D398.2 (A), D399.2 (A), D400.2 (A), D401.2 (A), D402.2 (A), D403.2 (A)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
- net z3: now also R223.2; no longer D414.2 (A), D415.2 (A), D416.2 (A), D417.2 (A), D418.2 (A), D419.2 (A), D420.2 (A), D421.2 (A), D422.2 (A), D423.2 (A), D424.2 (A), D425.2 (A)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
- net z4: now also R224.2; no longer D435.2 (A), D436.2 (A), D437.2 (A), D438.2 (A), D439.2 (A), D440.2 (A), D441.2 (A), D442.2 (A), D443.2 (A), D444.2 (A), D445.2 (A), D446.2 (A)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
- net z5: now also R225.2; no longer D456.2 (A), D457.2 (A), D458.2 (A), D459.2 (A), D460.2 (A), D461.2 (A), D462.2 (A), D463.2 (A), D464.2 (A), D465.2 (A), D466.2 (A), D467.2 (A)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
- net z6: now also R226.2; no longer D477.2 (A), D478.2 (A), D479.2 (A), D480.2 (A), D481.2 (A), D482.2 (A), D483.2 (A), D484.2 (A), D485.2 (A), D486.2 (A), D487.2 (A), D488.2 (A)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
- net z7: now also R227.2; no longer D498.2 (A), D499.2 (A), D500.2 (A), D501.2 (A), D502.2 (A), D503.2 (A), D504.2 (A), D505.2 (A), D506.2 (A), D507.2 (A), D508.2 (A), D509.2 (A)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
- new net: D336.2 (A), D337.2 (A), D338.2 (A), R216.1
- new net: D339.2 (A), D340.2 (A), D341.2 (A), R217.1
- new net: D342.2 (A), D343.2 (A), D344.2 (A), R218.1
- new net: D345.2 (A), D346.2 (A), D347.2 (A), R219.1
- new net: D324.2 (A), D325.2 (A), D326.2 (A), R212.1
- new net: D327.2 (A), D328.2 (A), D329.2 (A), R213.1
- new net: D330.2 (A), D331.2 (A), D332.2 (A), R214.1
- new net: D333.2 (A), D334.2 (A), D335.2 (A), R215.1
- new net: D348.2 (A), D349.2 (A), D350.2 (A), D351.2 (A), D352.2 (A), D353.2 (A), D354.2 (A), D355.2 (A), D356.2 (A), D357.2 (A), D358.2 (A), D359.2 (A)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
- new net: D370.2 (A), D371.2 (A), D372.2 (A), D373.2 (A), D374.2 (A), D375.2 (A), D376.2 (A), D377.2 (A), D378.2 (A), D379.2 (A), D380.2 (A), D381.2 (A)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
- new net: D392.2 (A), D393.2 (A), D394.2 (A), D395.2 (A), D396.2 (A), D397.2 (A), D398.2 (A), D399.2 (A), D400.2 (A), D401.2 (A), D402.2 (A), D403.2 (A)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
- new net: D414.2 (A), D415.2 (A), D416.2 (A), D417.2 (A), D418.2 (A), D419.2 (A), D420.2 (A), D421.2 (A), D422.2 (A), D423.2 (A), D424.2 (A), D425.2 (A)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
- new net: D435.2 (A), D436.2 (A), D437.2 (A), D438.2 (A), D439.2 (A), D440.2 (A), D441.2 (A), D442.2 (A), D443.2 (A), D444.2 (A), D445.2 (A), D446.2 (A)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
- new net: D627.2 (A), D628.2 (A), D629.2 (A), D630.2 (A), D631.2 (A), D632.2 (A), D633.2 (A), D634.2 (A), D635.2 (A), D636.2 (A), D637.2 (A), D638.2 (A)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
- new net: D612.2 (A), D613.2 (A), D614.2 (A), D615.2 (A), D616.2 (A), D617.2 (A), D618.2 (A), D619.2 (A), D620.2 (A), D621.2 (A), D622.2 (A), D623.2 (A)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
- new net: D597.2 (A), D598.2 (A), D599.2 (A), D600.2 (A), D601.2 (A), D602.2 (A), D603.2 (A), D604.2 (A), D605.2 (A), D606.2 (A), D607.2 (A), D608.2 (A)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
- new net: D582.2 (A), D583.2 (A), D584.2 (A), D585.2 (A), D586.2 (A), D587.2 (A), D588.2 (A), D589.2 (A), D590.2 (A), D591.2 (A), D592.2 (A), D593.2 (A)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
- new net: D567.2 (A), D568.2 (A), D569.2 (A), D570.2 (A), D571.2 (A), D572.2 (A), D573.2 (A), D574.2 (A), D575.2 (A), D576.2 (A), D577.2 (A), D578.2 (A)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
- new net: D551.2 (A), D552.2 (A), D553.2 (A), D554.2 (A), D555.2 (A), D556.2 (A), D557.2 (A), D558.2 (A), D559.2 (A), D560.2 (A), D561.2 (A), D562.2 (A)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
- new net: D535.2 (A), D536.2 (A), D537.2 (A), D538.2 (A), D539.2 (A), D540.2 (A), D541.2 (A), D542.2 (A), D543.2 (A), D544.2 (A), D545.2 (A), D546.2 (A)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
- new net: D519.2 (A), D520.2 (A), D521.2 (A), D522.2 (A), D523.2 (A), D524.2 (A), D525.2 (A), D526.2 (A), D527.2 (A), D528.2 (A), D529.2 (A), D530.2 (A)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
- new net: D498.2 (A), D499.2 (A), D500.2 (A), D501.2 (A), D502.2 (A), D503.2 (A), D504.2 (A), D505.2 (A), D506.2 (A), D507.2 (A), D508.2 (A), D509.2 (A)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
- new net: D477.2 (A), D478.2 (A), D479.2 (A), D480.2 (A), D481.2 (A), D482.2 (A), D483.2 (A), D484.2 (A), D485.2 (A), D486.2 (A), D487.2 (A), D488.2 (A)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
- new net: D456.2 (A), D457.2 (A), D458.2 (A), D459.2 (A), D460.2 (A), D461.2 (A), D462.2 (A), D463.2 (A), D464.2 (A), D465.2 (A), D466.2 (A), D467.2 (A)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
Other:
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
Commit message: Add GND wires to LED matrix
Changed lines of the file:
@@
 Connection ~ 2550 1400
 Connection ~ 2550 800
-Connection ~ 1050 800
 Wire Wire Line
 	950  800  1050 800
@@
 Wire Wire Line
 	1050 1000 1050 1100
-Connection ~ 1050 1000
-Wire Wire Line
-	1050 900  1050 1000
-Connection ~ 1050 900
-Wire Wire Line
-	1050 800  1050 900
-Wire Wire Line
-	1350 800  1350 900
-Connection ~ 1350 900
 $Comp
 L Device:LED D?
@@
 	-1   0    0    1
 $EndComp
-$Comp
-L Device:LED D?
-U 1 1 61C56D7B
-P 1200 800
-AR Path="/61C56D7B" Ref="D?"  Part="1"
-AR Path="/61AF721F/61C56D7B" Ref="D201"  Part="1"
-F 0 "D201" H 1193 545 50  0000 C CNN
-F 1 "LED" H 1193 636 50  0000 C CNN
-F 2 "LED_SMD:LED_0805_2012Metric_Castellated" H 1200 800 50  0001 C CNN
-F 3 "~" H 1200 800 50  0001 C CNN
-	1    1200 800
-	-1   0    0    1
-$EndComp
 Connection ~ 1350 1100
 Wire Wire Line
@@
 	-1   0    0    1
 $EndComp
-Wire Wire Line
-	1350 900  1350 1000
-Connection ~ 1350 1000
-$Comp
-L Device:LED D?
-U 1 1 61C56D5A
-P 1200 1000
-AR Path="/61C56D5A" Ref="D?"  Part="1"
-AR Path="/61AF721F/61C56D5A" Ref="D203"  Part="1"
-F 0 "D203" H 1193 745 50  0000 C CNN
-F 1 "LED" H 1193 836 50  0000 C CNN
-F 2 "LED_SMD:LED_0805_2012Metric_Castellated" H 1200 1000 50  0001 C CNN
-F 3 "~" H 1200 1000 50  0001 C CNN
-	1    1200 1000
-	-1   0    0    1
-$EndComp
 Connection ~ 1350 1300
 Wire Wire Line
@@
 	-1   0    0    1
 $EndComp
-Connection ~ 1350 800
 Connection ~ 1050 4350
 Connection ~ 1350 4350
@@
 Connection ~ 7450 5500
 Connection ~ 7450 7850
+$Comp
+L Device:LED D?
+U 1 1 61C56D5A
+P 1200 1000
+AR Path="/61C56D5A" Ref="D?"  Part="1"
+AR Path="/61AF721F/61C56D5A" Ref="D203"  Part="1"
+F 0 "D203" H 1193 745 50  0000 C CNN
+F 1 "LED" H 1193 836 50  0000 C CNN
+F 2 "LED_SMD:LED_0805_2012Metric_Castellated" H 1200 1000 50  0001 C CNN
+F 3 "~" H 1200 1000 50  0001 C CNN
+	1    1200 1000
+	-1   0    0    1
+$EndComp
+$Comp
+L Device:LED D?
+U 1 1 61C56D7B
+P 1200 800
+AR Path="/61C56D7B" Ref="D?"  Part="1"
+AR Path="/61AF721F/61C56D7B" Ref="D201"  Part="1"
+F 0 "D201" H 1193 545 50  0000 C CNN
+F 1 "LED" H 1193 636 50  0000 C CNN
+F 2 "LED_SMD:LED_0805_2012Metric_Castellated" H 1200 800 50  0001 C CNN
+F 3 "~" H 1200 800 50  0001 C CNN
+	1    1200 800
+	-1   0    0    1
+$EndComp
+Wire Wire Line
+	1050 800  1050 900
+Connection ~ 1050 800
+Wire Wire Line
+	1050 900  1050 1000
+Connection ~ 1050 900
+Connection ~ 1050 1000
+Wire Wire Line
+	1350 1000 1350 900
+Connection ~ 1350 1000
+Wire Wire Line
+	1350 900  1350 800
+Connection ~ 1350 900
+Connection ~ 1350 800
 $EndSCHEMATC
