File: midnight-sun-2019/midnight-sun-2019.sch (KiCad schematic (older format))
At the start: 66 parts, among them J101 Conn_01x02, J102 USB_A, SW101 SW_SPDT, SW102 SW_Push, SW103 SW_Push, U101 74HC14, U102 74HC595, U103 74HC595, U104 74HC595, U105 74HC86, U106 74HC86, U107 74HC86, U108 74HC86, U109 74HC14, U110 74HC14, U111 74HC86, U112 74HC86, U113 74HC14, U114 74HC86, U115 74HC86

Commit message: Clean up circuit draft
Parts:
- U101: footprint Package_DIP:DIP-14_W7.62mm_Socket -> (none)
Connections:
- net labels added: usr
- net labels removed: f2, f3, f4, f5, u
- wire segments 135 -> 179
- no-connect marks 19 -> 17
Other:
- moved on the sheet: C101, C102, D102, D103, R101, R103, R106, R107, SW102, U101C, U106E, U107E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

Commit message: WIP: schematic
Parts:
- removed J102: USB_A, electrokit:USB_Micro-B_Electrokit_anr41011019, symbol Connector:USB_A
- added J102: USB_B_Micro, electrokit:USB_Micro-B_Electrokit_anr41011019, symbol Connector:USB_B_Micro
- added R101: R, Resistor_THT:R_Axial_DIN0207_L6.3mm_D2.5mm_P7.62mm_Horizontal, symbol Device:R
- C101, C102: footprint (none) -> Capacitor_THT:CP_Radial_D5.0mm_P2.00mm
- D101, D102, D103, D104, D105, D106, D107, D108, D109, D110, D111, D112, D113, D114, D115, D116, D117, D118, D119, D120: footprint (none) -> LED_SMD:LED_0805_2012Metric_Castellated
- R102: renamed from R101; footprint (none) -> Resistor_THT:R_Axial_DIN0207_L6.3mm_D2.5mm_P7.62mm_Horizontal
- R103: renamed from R102; footprint (none) -> Resistor_THT:R_Axial_DIN0207_L6.3mm_D2.5mm_P7.62mm_Horizontal
- R104: renamed from R103; footprint (none) -> Resistor_THT:R_Axial_DIN0207_L6.3mm_D2.5mm_P7.62mm_Horizontal
- R105: renamed from R104; footprint (none) -> Resistor_THT:R_Axial_DIN0207_L6.3mm_D2.5mm_P7.62mm_Horizontal
- R106: renamed from R105; footprint (none) -> Resistor_SMD:R_0805_2012Metric_Pad1.15x1.40mm_HandSolder
- R107: renamed from R106; footprint (none) -> Resistor_SMD:R_0805_2012Metric_Pad1.15x1.40mm_HandSolder
- R108: renamed from R107; footprint (none) -> Resistor_SMD:R_0805_2012Metric_Pad1.15x1.40mm_HandSolder
- R109: renamed from R108; footprint (none) -> Resistor_SMD:R_0805_2012Metric_Pad1.15x1.40mm_HandSolder
- R110: renamed from R109; footprint (none) -> Resistor_SMD:R_0805_2012Metric_Pad1.15x1.40mm_HandSolder
- R111: renamed from R110; footprint (none) -> Resistor_SMD:R_0805_2012Metric_Pad1.15x1.40mm_HandSolder
- R112: renamed from R111; footprint (none) -> Resistor_SMD:R_0805_2012Metric_Pad1.15x1.40mm_HandSolder
- R113: renamed from R112; footprint (none) -> Resistor_SMD:R_0805_2012Metric_Pad1.15x1.40mm_HandSolder
- R114: renamed from R113; footprint (none) -> Resistor_SMD:R_0805_2012Metric_Pad1.15x1.40mm_HandSolder
- R115: renamed from R114; footprint (none) -> Resistor_SMD:R_0805_2012Metric_Pad1.15x1.40mm_HandSolder
- R116: renamed from R115; footprint (none) -> Resistor_SMD:R_0805_2012Metric_Pad1.15x1.40mm_HandSolder
- R117: renamed from R116; footprint (none) -> Resistor_SMD:R_0805_2012Metric_Pad1.15x1.40mm_HandSolder
- R118: renamed from R117; footprint (none) -> Resistor_SMD:R_0805_2012Metric_Pad1.15x1.40mm_HandSolder
- R119: renamed from R118; footprint (none) -> Resistor_SMD:R_0805_2012Metric_Pad1.15x1.40mm_HandSolder
- R120: renamed from R119; footprint (none) -> Resistor_SMD:R_0805_2012Metric_Pad1.15x1.40mm_HandSolder
- R121: renamed from R120; footprint (none) -> Resistor_SMD:R_0805_2012Metric_Pad1.15x1.40mm_HandSolder
- R122: renamed from R121; footprint (none) -> Resistor_SMD:R_0805_2012Metric_Pad1.15x1.40mm_HandSolder
- R123: renamed from R122; footprint (none) -> Resistor_SMD:R_0805_2012Metric_Pad1.15x1.40mm_HandSolder
- R124: renamed from R123; footprint (none) -> Resistor_SMD:R_0805_2012Metric_Pad1.15x1.40mm_HandSolder
- R125: renamed from R124; footprint (none) -> Resistor_SMD:R_0805_2012Metric_Pad1.15x1.40mm_HandSolder
- SW101: footprint (none) -> Button_Switch_THT:SW_CuK_JS202011CQN_DPDT_Straight
- SW102, SW103: footprint (none) -> Button_Switch_THT:SW_DIP_SPSTx03_Slide_9.78x9.8mm_W7.62mm_P2.54mm
- U101, U105, U106, U107, U108, U109, U110, U111, U112, U113, U114, U115: footprint (none) -> Package_DIP:DIP-14_W7.62mm_Socket
Connections:
- no-connect marks 17 -> 18
Other:
- moved on the sheet: D101, D102, D103, D104, D105, D106, D107, D108, D109, D110, D111, D112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

Commit message: Wire up all the logic
Parts:
- removed SW102, SW103: SW_Push, Button_Switch_THT:SW_DIP_SPSTx03_Slide_9.78x9.8mm_W7.62mm_P2.54mm, symbol Switch:SW_Push
- removed unit 7 of U101
- removed unit 5 of U105
- removed unit 5 of U106
- removed unit 5 of U107
- removed unit 5 of U108
- removed unit 7 of U109
- removed unit 7 of U110
- removed unit 5 of U111
- removed unit 5 of U112
- removed unit 7 of U113
- removed unit 5 of U114
- removed unit 5 of U115
- added C103: 10 uF, Capacitor_THT:CP_Radial_D5.0mm_P2.00mm, symbol Device:C
- added J102: Conn_01x02, Connector_PinHeader_2.54mm:PinHeader_1x02_P2.54mm_Vertical, symbol Connector_Generic:Conn_01x02
- added SW102, SW103: SW_SPDT, electrokit:SW_PUSH_DPDT_CW_Industries_GPBS850L, symbol Switch:SW_SPDT
- added U116: 74HC14, Package_DIP:DIP-14_W7.62mm_Socket, symbol 74xx:74HC14
- C101: value C -> 100 nF; footprint Capacitor_THT:CP_Radial_D5.0mm_P2.00mm -> Capacitor_THT:C_Disc_D7.5mm_W2.5mm_P5.00mm
- C102: value C -> 10 uF
- D101, D103: footprint LED_SMD:LED_0805_2012Metric_Castellated -> LED_THT:LED_D5.0mm
- D102: footprint LED_SMD:LED_0805_2012Metric_Castellated -> LED_THT:LED_D5.0mm_Clear
- R101, R104, R105: value R -> 10k
- R102, R103: value R -> 1k
- SW101: footprint Button_Switch_THT:SW_CuK_JS202011CQN_DPDT_Straight -> electrokit:SW_SPDT_MTS-102-A2
- renumbered J102 to J103, U114 to U111, U115 to U112, U111 to U113, U112 to U114, U113 to U115
Connections:
- net GND: now also C102.2, C103.2, J102.1 (Pin_1), SW102.1 (A), SW103.1 (A); no longer C102.1
- net VCC: now also C101.2, J102.2 (Pin_2), SW102.3 (C), SW103.3 (C)
- net z0: now also U115.6; no longer U110.8
- net z1: now also U115.4; no longer U110.10
- net z3: now also U115.8; no longer U115.4
- net z4: now also U116.6; no longer U115.6
- net z5: now also U116.4; no longer U115.8
- net z6: now also U116.2; no longer U115.10
- net z7: now also U116.8; no longer U115.12
- net at R103.2, R105.2: now also SW103.2 (B)
- net at R102.2, R104.2: now also SW102.2 (B)
- net at R102.1, U101.1: now also C102.1; no longer C101.2
- net at R103.1, U101.3: now also C103.1; no longer C102.2
- net at U114.6: now also U116.3; no longer U115.9
- net at U114.8: now also U116.1; no longer U115.11
- net at U114.11: now also U116.9; no longer U115.13
- net at U113.3: now also U115.5; no longer U110.9
- net at U113.6: now also U115.3; no longer U110.11
- net at U113.11: now also U115.9; no longer U115.3
- net at U114.3: now also U116.5; no longer U115.5
- no-connect marks 18 -> 26
Other:
- moved on the sheet: D113, D114, D115, D116, D117, D118, D119, D120, J103, R118, R119, R120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

Commit message: Finish wiring everything up
Parts:
- removed J101: Conn_01x02, Connector_PinSocket_2.54mm:PinSocket_1x02_P2.54mm_Vertical, symbol Connector_Generic:Conn_01x02
- removed J102: Conn_01x02, Connector_PinHeader_2.54mm:PinHeader_1x02_P2.54mm_Vertical, symbol Connector_Generic:Conn_01x02
- added J101: Conn_02x02_Odd_Even, Connector_PinHeader_2.54mm:PinHeader_2x02_P2.54mm_Vertical, symbol Connector_Generic:Conn_02x02_Odd_Even
- renumbered J103 to J102
Connections:
- net GND: now also J101.3 (Pin_3), J101.4 (Pin_4)
- net VCC: now also J101.1 (Pin_1), J101.2 (Pin_2)
Changed lines of the file:
@@
 Text Label 3250 2000 2    50   ~ 0
 rst
-$Comp
-L Connector_Generic:Conn_01x02 J101
-U 1 1 5CEEE3A8
-P 750 950
-F 0 "J101" H 668 625 50  0000 C CNN
-F 1 "Conn_01x02" H 668 716 50  0000 C CNN
-F 2 "Connector_PinSocket_2.54mm:PinSocket_1x02_P2.54mm_Vertical" H 750 950 50  0001 C CNN
-F 3 "~" H 750 950 50  0001 C CNN
-	1    750  950
-	-1   0    0    1
-$EndComp
 Text Label 4050 3900 0    50   ~ 0
 x0
@@
 NoConn ~ 4050 2200
 $Comp
-L power:GND #PWR0104
+L power:GND #PWR0114
 U 1 1 5CEEF634
-P 950 950
-F 0 "#PWR0104" H 950 700 50  0001 C CNN
-F 1 "GND" V 955 822 50  0000 R CNN
-F 2 "" H 950 950 50  0001 C CNN
-F 3 "" H 950 950 50  0001 C CNN
-	1    950  950
+P 1250 900
+F 0 "#PWR0114" H 1250 650 50  0001 C CNN
+F 1 "GND" V 1255 772 50  0000 R CNN
+F 2 "" H 1250 900 50  0001 C CNN
+F 3 "" H 1250 900 50  0001 C CNN
+	1    1250 900
 	0    -1   -1   0
 $EndComp
@@
 NoConn ~ 1700 1550
 $Comp
-L Connector:USB_B_Micro J103
+L Connector:USB_B_Micro J102
 U 1 1 76EFDB97
 P 1400 1550
-F 0 "J103" H 1457 2017 50  0000 C CNN
+F 0 "J102" H 1457 2017 50  0000 C CNN
 F 1 "USB_B_Micro" H 1457 1926 50  0000 C CNN
 F 2 "electrokit:USB_Micro-B_Electrokit_anr41011019" H 1550 1500 50  0001 C CNN
@@
 $EndComp
 $Comp
-L power:VCC #PWR0103
+L power:VCC #PWR0113
 U 1 1 76F38640
-P 950 850
-F 0 "#PWR0103" H 950 700 50  0001 C CNN
-F 1 "VCC" V 967 978 50  0000 L CNN
-F 2 "" H 950 850 50  0001 C CNN
-F 3 "" H 950 850 50  0001 C CNN
-	1    950  850
+P 1250 800
+F 0 "#PWR0113" H 1250 650 50  0001 C CNN
+F 1 "VCC" V 1267 928 50  0000 L CNN
+F 2 "" H 1250 800 50  0001 C CNN
+F 3 "" H 1250 800 50  0001 C CNN
+	1    1250 800
 	0    1    1    0
 $EndComp
@@
 $EndComp
 $Comp
-L power:GND #PWR0113
+L power:GND #PWR0115
 U 1 1 76FDF255
 P 1350 2600
-F 0 "#PWR0113" H 1350 2350 50  0001 C CNN
+F 0 "#PWR0115" H 1350 2350 50  0001 C CNN
 F 1 "GND" H 1355 2427 50  0000 C CNN
 F 2 "" H 1350 2600 50  0001 C CNN
@@
 $EndComp
 $Comp
-L power:GND #PWR0102
+L power:GND #PWR0104
 U 1 1 5CBF3918
 P 750 1650
-F 0 "#PWR0102" H 750 1400 50  0001 C CNN
+F 0 "#PWR0104" H 750 1400 50  0001 C CNN
 F 1 "GND" H 755 1477 50  0000 C CNN
 F 2 "" H 750 1650 50  0001 C CNN
@@
 $EndComp
 $Comp
-L power:VCC #PWR0101
+L power:VCC #PWR0103
 U 1 1 5CBE8005
 P 750 1350
-F 0 "#PWR0101" H 750 1200 50  0001 C CNN
+F 0 "#PWR0103" H 750 1200 50  0001 C CNN
 F 1 "VCC" H 767 1523 50  0000 C CNN
 F 2 "" H 750 1350 50  0001 C CNN
@@
 $EndComp
 $Comp
-L power:GND #PWR0114
+L power:GND #PWR0116
 U 1 1 5CC60BF0
 P 1400 1950
-F 0 "#PWR0114" H 1400 1700 50  0001 C CNN
+F 0 "#PWR0116" H 1400 1700 50  0001 C CNN
 F 1 "GND" H 1405 1777 50  0000 C CNN
 F 2 "" H 1400 1950 50  0001 C CNN
@@
 b15
 $Comp
-L Connector_Generic:Conn_01x02 J102
-U 1 1 5FC8D734
-P 1350 950
-F 0 "J102" H 1268 625 50  0000 C CNN
-F 1 "Conn_01x02" H 1268 716 50  0000 C CNN
-F 2 "Connector_PinHeader_2.54mm:PinHeader_1x02_P2.54mm_Vertical" H 1350 950 50  0001 C CNN
-F 3 "~" H 1350 950 50  0001 C CNN
-	1    1350 950
-	-1   0    0    1
-$EndComp
-$Comp
-L power:GND #PWR0116
-U 1 1 5FC8D73A
-P 1550 950
-F 0 "#PWR0116" H 1550 700 50  0001 C CNN
-F 1 "GND" V 1555 822 50  0000 R CNN
-F 2 "" H 1550 950 50  0001 C CNN
-F 3 "" H 1550 950 50  0001 C CNN
-	1    1550 950
+L Connector_Generic:Conn_02x02_Odd_Even J101
+U 1 1 5F1504BD
+P 950 800
+F 0 "J101" H 1000 1017 50  0000 C CNN
+F 1 "Conn_02x02_Odd_Even" H 1000 926 50  0000 C CNN
+F 2 "Connector_PinHeader_2.54mm:PinHeader_2x02_P2.54mm_Vertical" H 950 800 50  0001 C CNN
+F 3 "~" H 950 800 50  0001 C CNN
+	1    950  800
+	1    0    0    -1
+$EndComp
+$Comp
+L power:GND #PWR0102
+U 1 1 5F16ECDF
+P 750 900
+F 0 "#PWR0102" H 750 650 50  0001 C CNN
+F 1 "GND" V 755 772 50  0000 R CNN
+F 2 "" H 750 900 50  0001 C CNN
+F 3 "" H 750 900 50  0001 C CNN
+	1    750  900
+	0    1    1    0
+$EndComp
+$Comp
+L power:VCC #PWR0101
+U 1 1 5F171491
+P 750 800
+F 0 "#PWR0101" H 750 650 50  0001 C CNN
+F 1 "VCC" V 768 927 50  0000 L CNN
+F 2 "" H 750 800 50  0001 C CNN
+F 3 "" H 750 800 50  0001 C CNN
+	1    750  800
 	0    -1   -1   0
 $EndComp
-$Comp
-L power:VCC #PWR0115
-U 1 1 5FC8D740
-P 1550 850
-F 0 "#PWR0115" H 1550 700 50  0001 C CNN
-F 1 "VCC" V 1567 978 50  0000 L CNN
-F 2 "" H 1550 850 50  0001 C CNN
-F 3 "" H 1550 850 50  0001 C CNN
-	1    1550 850
-	0    1    1    0
-$EndComp
-Wire Wire Line
+Wire Wire Line

Commit message: Add battery holders
Parts:
- added BT101, BT103: Battery_Cell, electrokit:BatteryHolder_CR2016_CR2025_CR2032_22mm, symbol Device:Battery_Cell
Connections:
- net GND: now also BT101.2 (-)
- net VCC: now also BT103.1 (+)
- new net: BT101.1 (+), BT103.2 (-)
Changed lines of the file:
@@
 $EndComp
 $Comp
-L power:GND #PWR0124
+L power:GND #PWR0126
 U 1 1 5CC0CF82
 P 3250 2300
-F 0 "#PWR0124" H 3250 2050 50  0001 C CNN
+F 0 "#PWR0126" H 3250 2050 50  0001 C CNN
 F 1 "GND" V 3255 2172 50  0000 R CNN
 F 2 "" H 3250 2300 50  0001 C CNN
@@
 clk
 $Comp
-L power:VCC #PWR0127
+L power:VCC #PWR0129
 U 1 1 5CC0F9A9
 P 3650 1500
-F 0 "#PWR0127" H 3650 1350 50  0001 C CNN
+F 0 "#PWR0129" H 3650 1350 50  0001 C CNN
 F 1 "VCC" V 3667 1628 50  0000 L CNN
 F 2 "" H 3650 1500 50  0001 C CNN
@@
 NoConn ~ 4050 2600
 $Comp
-L power:GND #PWR0126
+L power:GND #PWR0128
 U 1 1 5CC1B6EE
 P 3250 6150
-F 0 "#PWR0126" H 3250 5900 50  0001 C CNN
+F 0 "#PWR0128" H 3250 5900 50  0001 C CNN
 F 1 "GND" V 3255 6022 50  0000 R CNN
 F 2 "" H 3250 6150 50  0001 C CNN
@@
 clk
 $Comp
-L power:VCC #PWR0131
+L power:VCC #PWR0133
 U 1 1 5CC1B702
 P 3650 5350
-F 0 "#PWR0131" H 3650 5200 50  0001 C CNN
+F 0 "#PWR0133" H 3650 5200 50  0001 C CNN
 F 1 "VCC" V 3667 5478 50  0000 L CNN
 F 2 "" H 3650 5350 50  0001 C CNN
@@
 clk
 $Comp
-L power:GND #PWR0130
+L power:GND #PWR0132
 U 1 1 5CC1C9E9
 P 3650 5000
-F 0 "#PWR0130" H 3650 4750 50  0001 C CNN
+F 0 "#PWR0132" H 3650 4750 50  0001 C CNN
 F 1 "GND" V 3655 4872 50  0000 R CNN
 F 2 "" H 3650 5000 50  0001 C CNN
@@
 $EndComp
 $Comp
-L power:VCC #PWR0129
+L power:VCC #PWR0131
 U 1 1 5CC1C9EF
 P 3650 3700
-F 0 "#PWR0129" H 3650 3550 50  0001 C CNN
+F 0 "#PWR0131" H 3650 3550 50  0001 C CNN
 F 1 "VCC" V 3667 3828 50  0000 L CNN
 F 2 "" H 3650 3700 50  0001 C CNN
@@
 	3250 3450 3250 3900
 $Comp
-L power:GND #PWR0123
+L power:GND #PWR0124
 U 1 1 5CD027AA
 P 2650 1700
-F 0 "#PWR0123" H 2650 1450 50  0001 C CNN
+F 0 "#PWR0124" H 2650 1450 50  0001 C CNN
 F 1 "GND" V 2655 1572 50  0000 R CNN
 F 2 "" H 2650 1700 50  0001 C CNN
@@
 $EndComp
 $Comp
-L power:GND #PWR0133
+L power:GND #PWR0135
 U 1 1 5CD20D5E
 P 5450 4150
-F 0 "#PWR0133" H 5450 3900 50  0001 C CNN
+F 0 "#PWR0135" H 5450 3900 50  0001 C CNN
 F 1 "GND" V 5455 4022 50  0000 R CNN
 F 2 "" H 5450 4150 50  0001 C CNN
@@
 $EndComp
 $Comp
-L power:GND #PWR0134
+L power:GND #PWR0136
 U 1 1 5CD20D70
 P 5450 4550
-F 0 "#PWR0134" H 5450 4300 50  0001 C CNN
+F 0 "#PWR0136" H 5450 4300 50  0001 C CNN
 F 1 "GND" V 5455 4422 50  0000 R CNN
 F 2 "" H 5450 4550 50  0001 C CNN
@@
 $EndComp
 $Comp
-L power:GND #PWR0135
+L power:GND #PWR0137
 U 1 1 5CD20D82
 P 5450 4950
-F 0 "#PWR0135" H 5450 4700 50  0001 C CNN
+F 0 "#PWR0137" H 5450 4700 50  0001 C CNN
 F 1 "GND" V 5455 4822 50  0000 R CNN
 F 2 "" H 5450 4950 50  0001 C CNN
@@
 $EndComp
 $Comp
-L power:GND #PWR0136
+L power:GND #PWR0138
 U 1 1 5CD20D94
 P 5450 5350
-F 0 "#PWR0136" H 5450 5100 50  0001 C CNN
+F 0 "#PWR0138" H 5450 5100 50  0001 C CNN
 F 1 "GND" V 5455 5222 50  0000 R CNN
 F 2 "" H 5450 5350 50  0001 C CNN
@@
 $EndComp
 $Comp
-L power:GND #PWR0120
+L power:GND #PWR0121
 U 1 1 5DF27255
 P 2550 2600
-F 0 "#PWR0120" H 2550 2350 50  0001 C CNN
+F 0 "#PWR0121" H 2550 2350 50  0001 C CNN
 F 1 "GND" V 2555 2472 50  0000 R CNN
 F 2 "" H 2550 2600 50  0001 C CNN
@@
 $EndComp
 $Comp
-L power:GND #PWR0137
+L power:GND #PWR0139
 U 1 1 76A8EDEC
 P 5450 5750
-F 0 "#PWR0137" H 5450 5500 50  0001 C CNN
+F 0 "#PWR0139" H 5450 5500 50  0001 C CNN
 F 1 "GND" V 5455 5622 50  0000 R CNN
 F 2 "" H 5450 5750 50  0001 C CNN
@@
 $EndComp
 $Comp
-L power:GND #PWR0138
+L power:GND #PWR0140
 U 1 1 76A8EDF2
 P 5450 6150
-F 0 "#PWR0138" H 5450 5900 50  0001 C CNN
+F 0 "#PWR0140" H 5450 5900 50  0001 C CNN
 F 1 "GND" V 5455 6022 50  0000 R CNN
 F 2 "" H 5450 6150 50  0001 C CNN
@@
 $EndComp
 $Comp
-L power:GND #PWR0139
+L power:GND #PWR0141
 U 1 1 76A8EDF8
 P 5450 6550
-F 0 "#PWR0139" H 5450 6300 50  0001 C CNN
+F 0 "#PWR0141" H 5450 6300 50  0001 C CNN
 F 1 "GND" V 5455 6422 50  0000 R CNN
 F 2 "" H 5450 6550 50  0001 C CNN
@@
 $EndComp
 $Comp
-L power:GND #PWR0140
+L power:GND #PWR0142
 U 1 1 76A8EDFE
 P 5450 6950
-F 0 "#PWR0140" H 5450 6700 50  0001 C CNN
+F 0 "#PWR0142" H 5450 6700 50  0001 C CNN
 F 1 "GND" V 5455 6822 50  0000 R CNN
 F 2 "" H 5450 6950 50  0001 C CNN
@@
 $EndComp
 $Comp
-L power:GND #PWR0141
+L power:GND #PWR0143
 U 1 1 76B2DE98
 P 5450 7350
-F 0 "#PWR0141" H 5450 7100 50  0001 C CNN
+F 0 "#PWR0143" H 5450 7100 50  0001 C CNN
 F 1 "GND" V 5455 7222 50  0000 R CNN
 F 2 "" H 5450 7350 50  0001 C CNN
@@
 $EndComp
 $Comp
-L power:GND #PWR0142
+L power:GND #PWR0144
 U 1 1 76B2DE9E
 P 5450 7750
-F 0 "#PWR0142" H 5450 7500 50  0001 C CNN
+F 0 "#PWR0144" H 5450 7500 50  0001 C CNN
 F 1 "GND" V 5455 7622 50  0000 R CNN
 F 2 "" H 5450 7750 50  0001 C CNN
@@
 $EndComp
 $Comp
-L power:GND #PWR0143
+L power:GND #PWR0145
 U 1 1 76B2DEA4
 P 5450 8150
-F 0 "#PWR0143" H 5450 7900 50  0001 C CNN
+F 0 "#PWR0145" H 5450 7900 50  0001 C CNN
 F 1 "GND" V 5455 8022 50  0000 R CNN
 F 2 "" H 5450 8150 50  0001 C CNN
@@
 $EndComp
 $Comp
-L power:GND #PWR0144
+L power:GND #PWR0146
 U 1 1 76B2DEAA
 P 5450 8550
-F 0 "#PWR0144" H 5450 8300 50  0001 C CNN
+F 0 "#PWR0146" H 5450 8300 50  0001 C CNN
 F 1 "GND" V 5455 8422 50  0000 R CNN
 F 2 "" H 5450 8550 50  0001 C CNN
@@
 $EndComp
 $Comp
-L power:GND #PWR0145
+L power:GND #PWR0147
 U 1 1 76B2DEE0
 P 5450 8950
-F 0 "#PWR0145" H 5450 8700 50  0001 C CNN
+F 0 "#PWR0147" H 5450 8700 50  0001 C CNN
 F 1 "GND" V 5455 8822 50  0000 R CNN
 F 2 "" H 5450 8950 50  0001 C CNN
@@
 $EndComp
 $Comp
-L power:GND #PWR0146
+L power:GND #PWR0148
 U 1 1 76B2DEE6
 P 5450 9350
-F 0 "#PWR0146" H 5450 9100 50  0001 C CNN
+F 0 "#PWR0148" H 5450 9100 50  0001 C CNN
 F 1 "GND" V 5455 9222 50  0000 R CNN
 F 2 "" H 5450 9350 50  0001 C CNN
@@
 $EndComp
 $Comp
-L power:GND #PWR0147
+L power:GND #PWR0149
 U 1 1 76B2DEEC
 P 5450 9750
-F 0 "#PWR0147" H 5450 9500 50  0001 C CNN
+F 0 "#PWR0149" H 5450 9500 50  0001 C CNN
 F 1 "GND" V 5455 9622 50  0000 R CNN
 F 2 "" H 5450 9750 50  0001 C CNN
@@
 $EndComp
 $Comp
-L power:GND #PWR0148
+L power:GND #PWR0150
 U 1 1 76B2DEF2
 P 5450 10150
-F 0 "#PWR0148" H 5450 9900 50  0001 C CNN
+F 0 "#PWR0150" H 5450 9900 50  0001 C CNN
 F 1 "GND" V 5455 10022 50  0000 R CNN
 F 2 "" H 5450 10150 50  0001 C CNN
@@
 $EndComp
 $Comp
-L power:GND #PWR0132
+L power:GND #PWR0134
 U 1 1 5CC95636
 P 3650 6650
-F 0 "#PWR0132" H 3650 6400 50  0001 C CNN
+F 0 "#PWR0134" H 3650 6400 50  0001 C CNN
 F 1 "GND" H 3655 6477 50  0000 C CNN
 F 2 "" H 3650 6650 50  0001 C CNN
@@
 Connection ~ 3250 1700
 $Comp
-L power:GND #PWR0128
+L power:GND #PWR0130
 U 1 1 5CCDCBB3
 P 3650 2800
-F 0 "#PWR0128" H 3650 2550 50  0001 C CNN
+F 0 "#PWR0130" H 3650 2550 50  0001 C CNN
 F 1 "GND" H 3655 2627 50  0000 C CNN
 F 2 "" H 3650 2800 50  0001 C CNN
@@
 $EndComp
 $Comp
-L power:GND #PWR0125
+L power:GND #PWR0127
 U 1 1 5CCE0EF9
 P 3250 4500
-F 0 "#PWR0125" H 3250 4250 50  0001 C CNN
+F 0 "#PWR0127" H 3250 4250 50  0001 C CNN
 F 1 "GND" H 3255 4327 50  0000 C CNN
 F 2 "" H 3250 4500 50  0001 C CNN
@@
 $EndComp
 $Comp
-L power:GND #PWR0122
+L power:GND #PWR0123
 U 1 1 5CEC139D
 P 2550 5100
-F 0 "#PWR0122" H 2550 4850 50  0001 C CNN
+F 0 "#PWR0123" H 2550 4850 50  0001 C CNN
 F 1 "GND" V 2555 4972 50  0000 R CNN
 F 2 "" H 2550 5100 50  0001 C CNN
@@
 Connection ~ 1950 4100
 $Comp
-L power:GND #PWR0121
+L power:GND #PWR0122
 U 1 1 5CEBD2B8
 P 2550 3800
-F 0 "#PWR0121" H 2550 3550 50  0001 C CNN
+F 0 "#PWR0122" H 2550 3550 50  0001 C CNN
 F 1 "GND" V 2555 3672 50  0000 R CNN
 F 2 "" H 2550 3800 50  0001 C CNN
@@
 	0    -1   -1   0
 $EndComp
+$Comp
+L power:VCC #PWR0125
+U 1 1 5CF5D8FC
+P 2450 850
+F 0 "#PWR0125" H 2450 700 50  0001 C CNN
+F 1 "VCC" V 2467 978 50  0000 L CNN
+F 2 "" H 2450 850 50  0001 C CNN
+F 3 "" H 2450 850 50  0001 C CNN
+	1    2450 850
+	0    1    1    0
+$EndComp
+$Comp
+L power:GND #PWR0120
+U 1 1 5CF60359
+P 1850 850
+F 0 "#PWR0120" H 1850 600 50  0001 C CNN
+F 1 "GND" V 1855 722 50  0000 R CNN
+F 2 "" H 1850 850 50  0001 C CNN
+F 3 "" H 1850 850 50  0001 C CNN
+	1    1850 850
+	0    1    1    0
+$EndComp
+$Comp
+L Device:Battery_Cell BT101
+U 1 1 5CF621CA
+P 1950 850
+F 0 "BT101" V 1695 900 50  0000 C CNN
+F 1 "Battery_Cell" V 1786 900 50  0000 C CNN
+F 2 "electrokit:BatteryHolder_CR2016_CR2025_CR2032_22mm" V 1950 910 50  0001 C CNN
+F 3 "~" V 1950 910 50  0001 C CNN
+	1    1950 850
+	0    1    1    0
+$EndComp
+$Comp
+L Device:Battery_Cell BT103
+U 1 1 5CF653D3
+P 2250 850
+F 0 "BT103" V 1995 900 50  0000 C CNN
+F 1 "Battery_Cell" V 2086 900 50  0000 C CNN
+F 2 "electrokit:BatteryHolder_CR2016_CR2025_CR2032_22mm" V 2250 910 50  0001 C CNN
+F 3 "~" V 2250 910 50  0001 C CNN
+	1    2250 850
+	0    1    1    0
+$EndComp
 Wire Wire Line
 	6450 9800 7300 9800
@@
 	4300 3800 4300 6150
 Wire Bus Line
+	7050 6400 7050 11100
+Wire Bus Line
 	9800 2650 9800 5650
 Wire Bus Line
@@
 Wire Bus Line
 	4600 3800 4600 10050
-Wire Bus Line
-	7050 6400 7050 11100
 $EndSCHEMATC

Commit message: Re-annotate components
Parts:
- renumbered BT101 to BT1, BT103 to BT2, C101 to C1, C102 to C2, C103 to C3, D101 to D1, D110 to D10, D111 to D11, D112 to D12, D113 to D13, D114 to D14, D115 to D15, D116 to D16, D117 to D17, D118 to D18, D119 to D19, D102 to D2, D120 to D20, D103 to D3, D104 to D4, D105 to D5, D106 to D6, D107 to D7, D108 to D8, D109 to D9, J101 to J1, J102 to J2, R101 to R1, R110 to R10, R111 to R11, R112 to R12, R113 to R13, R114 to R14, R115 to R15, R116 to R16, R117 to R17, R118 to R18, R119 to R19, R102 to R2, R120 to R20, R121 to R21, R122 to R22, R123 to R23, R124 to R24, R125 to R25, R103 to R3, R104 to R4, R105 to R5, R106 to R6, R107 to R7, R108 to R8, R109 to R9, SW101 to SW1, SW102 to SW2, SW103 to SW3, U101 to U1, U110 to U10, U111 to U11, U112 to U12, U113 to U13, U114 to U14, U115 to U15, U116 to U16, U102 to U2, U103 to U3, U104 to U4, U105 to U5, U106 to U6, U107 to U7, U108 to U8, U109 to U9

Commit message: More finishing touches
Parts:
- D10, D11, D12, D13, D14, D15, D16, D17, D18, D19, D20, D4, D5, D6, D7, D8, D9: footprint LED_SMD:LED_0805_2012Metric_Castellated -> electrokit:LED_0805_2012Metric_Castellated_no_silkscreen
- R10, R11, R12, R13, R14, R15, R16, R17, R18, R19, R20, R21, R22, R23, R24, R25, R6, R7, R8, R9: footprint Resistor_SMD:R_0805_2012Metric_Pad1.15x1.40mm_HandSolder -> electrokit:R_0805_2012Metric_Pad1.15x1.40mm_HandSolder_no_silkscreen
