File: midnight-sun-2019/midnight-sun-2019.sch (KiCad schematic (older format))
At the start: 71 parts, among them J1 Conn_02x02_Odd_Even, J2 USB_B_Micro, SW1 SW_SPDT, SW2 SW_SPDT, SW3 SW_SPDT, U1 74HC14, U10 74HC14, U11 74HC86, U12 74HC86, U13 74HC86, U14 74HC86, U15 74HC14, U16 74HC14, U2 74HC595, U3 74HC595, U4 74HC595, U5 74HC86, U6 74HC86, U7 74HC86, U8 74HC86, U9 74HC14

Commit message: Add GND and VCC connections to ICs...
Parts:
- added unit 7 of U1
- added unit 7 of U10
- added unit 5 of U11
- added unit 5 of U12
- added unit 5 of U13
- added unit 5 of U14
- added unit 7 of U15
- added unit 7 of U16
- added unit 5 of U5
- added unit 5 of U6
- added unit 5 of U7
- added unit 5 of U8
- added unit 7 of U9
Connections:
- net GND: now also U1.7 (GND), U10.7 (GND), U11.7 (GND), U12.7 (GND), U13.7 (GND), U14.7 (GND), U15.7 (GND), U16.7 (GND), U5.7 (GND), U6.7 (GND), U7.7 (GND), U8.7 (GND), U9.7 (GND)
- net VCC: now also U1.14 (VCC), U10.14 (VCC), U11.14 (VCC), U12.14 (VCC), U13.14 (VCC), U14.14 (VCC), U15.14 (VCC), U16.14 (VCC), U5.14 (VCC), U6.14 (VCC), U7.14 (VCC), U8.14 (VCC), U9.14 (VCC)

Commit message: Add debounce to SW1
Parts:
- removed R1: 10k, Resistor_THT:R_Axial_DIN0207_L6.3mm_D2.5mm_P7.62mm_Horizontal, symbol Device:R
- removed SW1: SW_SPDT, electrokit:SW_SPDT_MTS-102-A2, symbol Switch:SW_SPDT
- added C?: 10 uF, Capacitor_THT:CP_Radial_D5.0mm_P2.00mm, symbol Device:C
- added R?: 10k, Resistor_THT:R_Axial_DIN0207_L6.3mm_D2.5mm_P7.62mm_Horizontal, symbol Device:R
- added R?: 1k, Resistor_THT:R_Axial_DIN0207_L6.3mm_D2.5mm_P7.62mm_Horizontal, symbol Device:R
- added SW?: SW_SPDT, electrokit:SW_PUSH_DPDT_CW_Industries_GPBS850L, symbol Switch:SW_SPDT
Connections:
- net GND: now also C?.2, SW?.1 (A)
- net VCC: now also R?.1, SW?.3 (C)
- net clk: now also U1.4; no longer U1.2
- net rst: now also U1.6; no longer U1.4
- net usr: now also U1.2
- net at U5.3: now also U1.9; no longer U1.5
- net at D4.2 (A), U2.14 (SER): now also U1.8; no longer U1.6
- net at C2.1, R2.1: now also U1.3; no longer U1.1
- net at C3.1, R3.1: now also U1.5; no longer U1.3
- new net: R?.2, R?.2, SW?.2 (B)
- new net: C?.1, R?.1, U1.1
- no-connect marks 26 -> 24
Other:
- moved on the sheet: BT1, BT2, J2, U1A, U1B, U1C, U1D

Commit message: Update PCB routes to agree with new schematic
Parts:
- SW1: renamed from SW?; footprint electrokit:SW_PUSH_DPDT_CW_Industries_GPBS850L -> electrokit:SW_SPDT_MTS-102-A2
- U1, U10, U11, U12, U13, U14, U15, U16, U5, U6, U7, U8, U9: footprint (none) -> Package_DIP:DIP-14_W7.62mm_Socket
- gave numbers to parts that had none: 3
- renumbered C2 to C3, C3 to C4, R9 to R10, R10 to R11, R11 to R12, R12 to R13, R13 to R14, R14 to R15, R15 to R16, R16 to R17, R17 to R18, R18 to R19, R19 to R20, R20 to R21, R21 to R22, R22 to R23, R23 to R24, R24 to R25, R25 to R26, R4 to R5, R5 to R6, R6 to R7, R7 to R8, R8 to R9
Connections:
- net clk: now also U1.12; no longer U1.4
- net rst: now also U1.10; no longer U1.6
- net usr: now also U1.4; no longer U1.2
- net at C3.1, R2.1: now also U1.13; no longer U1.3
- net at C4.1, R3.1: now also U1.11; no longer U1.5
- net at C2.1, R1.1: now also U1.3; no longer U1.1
Other:
- moved on the sheet: U1A, U1B, U1C, U1E, U1F

Commit message: Rotate U16 footprint 180 degrees
Parts:
- added unit 5 of U16
- added unit 6 of U16
Connections:
- net z4: now also U16.12; no longer U16.6
- net z5: now also U16.10; no longer U16.4
- net z6: now also U16.8; no longer U16.2
- net z7: now also U16.6; no longer U16.8
- net at U14.6: now also U16.11; no longer U16.3
- net at U14.8: now also U16.9; no longer U16.1
- net at U14.11: now also U16.5; no longer U16.9
- net at U14.3: now also U16.13; no longer U16.5
- no-connect marks 24 -> 28
Other:
- moved on the sheet: U10D, U10E, U10F, U15E, U15F, U16A, U16B, U16C, U16D
Changed lines of the file:
@@
 	4600 2850 4600 2950
 Wire Wire Line
-	5200 3050 5200 3250
-Wire Wire Line
 	3250 3450 3250 3900
 $Comp
@@
 L 74xx:74HC14 U10
 U 4 1 5CFEC926
-P 9550 10450
-F 0 "U10" H 9550 10767 50  0000 C CNN
-F 1 "74HC14" H 9550 10676 50  0000 C CNN
-F 2 "Package_DIP:DIP-14_W7.62mm_Socket" H 9550 10450 50  0001 C CNN
-F 3 "http://www.ti.com/lit/gpn/sn74HC14" H 9550 10450 50  0001 C CNN
-	4    9550 10450
+P 9250 10400
+F 0 "U10" H 9250 10717 50  0000 C CNN
+F 1 "74HC14" H 9250 10626 50  0000 C CNN
+F 2 "Package_DIP:DIP-14_W7.62mm_Socket" H 9250 10400 50  0001 C CNN
+F 3 "http://www.ti.com/lit/gpn/sn74HC14" H 9250 10400 50  0001 C CNN
+	4    9250 10400
 	1    0    0    -1
 $EndComp
@@
 L 74xx:74HC14 U10
 U 5 1 5CFEC92C
-P 9550 10950
-F 0 "U10" H 9550 11267 50  0000 C CNN
-F 1 "74HC14" H 9550 11176 50  0000 C CNN
-F 2 "Package_DIP:DIP-14_W7.62mm_Socket" H 9550 10950 50  0001 C CNN
-F 3 "http://www.ti.com/lit/gpn/sn74HC14" H 9550 10950 50  0001 C CNN
-	5    9550 10950
+P 9250 10900
+F 0 "U10" H 9250 11217 50  0000 C CNN
+F 1 "74HC14" H 9250 11126 50  0000 C CNN
+F 2 "Package_DIP:DIP-14_W7.62mm_Socket" H 9250 10900 50  0001 C CNN
+F 3 "http://www.ti.com/lit/gpn/sn74HC14" H 9250 10900 50  0001 C CNN
+	5    9250 10900
 	1    0    0    -1
 $EndComp
@@
 L 74xx:74HC14 U15
 U 5 1 5CFF1027
-P 11100 10450
-F 0 "U15" H 11100 10767 50  0000 C CNN
-F 1 "74HC14" H 11100 10676 50  0000 C CNN
-F 2 "Package_DIP:DIP-14_W7.62mm_Socket" H 11100 10450 50  0001 C CNN
-F 3 "http://www.ti.com/lit/gpn/sn74HC14" H 11100 10450 50  0001 C CNN
-	5    11100 10450
+P 10800 10400
+F 0 "U15" H 10800 10717 50  0000 C CNN
+F 1 "74HC14" H 10800 10626 50  0000 C CNN
+F 2 "Package_DIP:DIP-14_W7.62mm_Socket" H 10800 10400 50  0001 C CNN
+F 3 "http://www.ti.com/lit/gpn/sn74HC14" H 10800 10400 50  0001 C CNN
+	5    10800 10400
 	1    0    0    -1
 $EndComp
@@
 L 74xx:74HC14 U15
 U 6 1 5DEEF6B3
-P 11100 10950
-F 0 "U15" H 11100 11267 50  0000 C CNN
-F 1 "74HC14" H 11100 11176 50  0000 C CNN
-F 2 "Package_DIP:DIP-14_W7.62mm_Socket" H 11100 10950 50  0001 C CNN
-F 3 "http://www.ti.com/lit/gpn/sn74HC14" H 11100 10950 50  0001 C CNN
-	6    11100 10950
+P 10800 10900
+F 0 "U15" H 10800 11217 50  0000 C CNN
+F 1 "74HC14" H 10800 11126 50  0000 C CNN
+F 2 "Package_DIP:DIP-14_W7.62mm_Socket" H 10800 10900 50  0001 C CNN
+F 3 "http://www.ti.com/lit/gpn/sn74HC14" H 10800 10900 50  0001 C CNN
+	6    10800 10900
 	1    0    0    -1
 $EndComp
@@
 L 74xx:74HC14 U10
 U 6 1 5E202D30
-P 10300 10950
-F 0 "U10" H 10300 11267 50  0000 C CNN
-F 1 "74HC14" H 10300 11176 50  0000 C CNN
-F 2 "Package_DIP:DIP-14_W7.62mm_Socket" H 10300 10950 50  0001 C CNN
-F 3 "http://www.ti.com/lit/gpn/sn74HC14" H 10300 10950 50  0001 C CNN
-	6    10300 10950
-	1    0    0    -1
-$EndComp
-NoConn ~ 9250 10450
-NoConn ~ 9250 10950
-NoConn ~ 9850 10950
-NoConn ~ 9850 10450
-NoConn ~ 10000 10950
-NoConn ~ 10600 10950
-$Comp
-L 74xx:74HC14 U16
-U 1 1 5E2E0C30
-P 11100 9300
-F 0 "U16" H 11100 9617 50  0000 C CNN
-F 1 "74HC14" H 11100 9526 50  0000 C CNN
-F 2 "Package_DIP:DIP-14_W7.62mm_Socket" H 11100 9300 50  0001 C CNN
-F 3 "http://www.ti.com/lit/gpn/sn74HC14" H 11100 9300 50  0001 C CNN
-	1    11100 9300
+P 10000 10900
+F 0 "U10" H 10000 11217 50  0000 C CNN
+F 1 "74HC14" H 10000 11126 50  0000 C CNN
+F 2 "Package_DIP:DIP-14_W7.62mm_Socket" H 10000 10900 50  0001 C CNN
+F 3 "http://www.ti.com/lit/gpn/sn74HC14" H 10000 10900 50  0001 C CNN
+	6    10000 10900
 	1    0    0    -1
 $EndComp
+NoConn ~ 8950 10400
+NoConn ~ 8950 10900
+NoConn ~ 9550 10900
+NoConn ~ 9550 10400
+NoConn ~ 9700 10900
+NoConn ~ 10300 10900
 $Comp
 L 74xx:74HC14 U16
 U 2 1 5E2E1550
-P 11100 8800
-F 0 "U16" H 11100 9117 50  0000 C CNN
-F 1 "74HC14" H 11100 9026 50  0000 C CNN
-F 2 "Package_DIP:DIP-14_W7.62mm_Socket" H 11100 8800 50  0001 C CNN
-F 3 "http://www.ti.com/lit/gpn/sn74HC14" H 11100 8800 50  0001 C CNN
-	2    11100 8800
+P 12250 8800
+F 0 "U16" H 12250 9117 50  0000 C CNN
+F 1 "74HC14" H 12250 9026 50  0000 C CNN
+F 2 "Package_DIP:DIP-14_W7.62mm_Socket" H 12250 8800 50  0001 C CNN
+F 3 "http://www.ti.com/lit/gpn/sn74HC14" H 12250 8800 50  0001 C CNN
+	2    12250 8800
 	1    0    0    -1
 $EndComp
@@
 L 74xx:74HC14 U16
 U 3 1 5E409A75
-P 11100 8300
-F 0 "U16" H 11100 8617 50  0000 C CNN
-F 1 "74HC14" H 11100 8526 50  0000 C CNN
-F 2 "Package_DIP:DIP-14_W7.62mm_Socket" H 11100 8300 50  0001 C CNN
-F 3 "http://www.ti.com/lit/gpn/sn74HC14" H 11100 8300 50  0001 C CNN
-	3    11100 8300
-	1    0    0    -1
-$EndComp
-$Comp
-L 74xx:74HC14 U16
-U 4 1 5E40AA6C
 P 11100 9800
 F 0 "U16" H 11100 10117 50  0000 C CNN
@@
 F 2 "Package_DIP:DIP-14_W7.62mm_Socket" H 11100 9800 50  0001 C CNN
 F 3 "http://www.ti.com/lit/gpn/sn74HC14" H 11100 9800 50  0001 C CNN
-	4    11100 9800
+	3    11100 9800
 	1    0    0    -1
 $EndComp
-NoConn ~ 10800 10450
-NoConn ~ 10800 10950
-NoConn ~ 11400 10950
-NoConn ~ 11400 10450
+$Comp
+L 74xx:74HC14 U16
+U 4 1 5E40AA6C
+P 11100 9300
+F 0 "U16" H 11100 9617 50  0000 C CNN
+F 1 "74HC14" H 11100 9526 50  0000 C CNN
+F 2 "Package_DIP:DIP-14_W7.62mm_Socket" H 11100 9300 50  0001 C CNN
+F 3 "http://www.ti.com/lit/gpn/sn74HC14" H 11100 9300 50  0001 C CNN
+	4    11100 9300
+	1    0    0    -1
+$EndComp
+NoConn ~ 10500 10400
+NoConn ~ 10500 10900
+NoConn ~ 11100 10900
+NoConn ~ 11100 10400
 Entry Wire Line
 	10950 3650 11050 3750
@@
 $EndComp
 Connection ~ 1350 2900
+$Comp
+L 74xx:74HC14 U16
+U 1 1 5E2E0C30
+P 12250 8350
+F 0 "U16" H 12250 8667 50  0000 C CNN
+F 1 "74HC14" H 12250 8576 50  0000 C CNN
+F 2 "Package_DIP:DIP-14_W7.62mm_Socket" H 12250 8350 50  0001 C CNN
+F 3 "http://www.ti.com/lit/gpn/sn74HC14" H 12250 8350 50  0001 C CNN
+	1    12250 8350
+	1    0    0    -1
+$EndComp
+$Comp
+L 74xx:74HC14 U16
+U 5 1 5D03EF2F
+P 11100 8800
+F 0 "U16" H 11100 9117 50  0000 C CNN
+F 1 "74HC14" H 11100 9026 50  0000 C CNN
+F 2 "" H 11100 8800 50  0001 C CNN
+F 3 "http://www.ti.com/lit/gpn/sn74HC14" H 11100 8800 50  0001 C CNN
+	5    11100 8800
+	1    0    0    -1
+$EndComp
+$Comp
+L 74xx:74HC14 U16
+U 6 1 5D041566
+P 11100 8300
+F 0 "U16" H 11100 8617 50  0000 C CNN
+F 1 "74HC14" H 11100 8526 50  0000 C CNN
+F 2 "" H 11100 8300 50  0001 C CNN
+F 3 "http://www.ti.com/lit/gpn/sn74HC14" H 11100 8300 50  0001 C CNN
+	6    11100 8300
+	1    0    0    -1
+$EndComp
+NoConn ~ 11950 8350
+Wire Wire Line
+	5200 3050 5200 3450
+NoConn ~ 11950 8800
+NoConn ~ 12550 8800
+NoConn ~ 12550 8350
 Wire Wire Line
 	6450 9800 7300 9800
@@
 Wire Bus Line
 	4600 3800 4600 10050
-Connection ~ 5200 3250
-Wire Wire Line
-	5200 3250 5200 3450
 $EndSCHEMATC

Commit message: Rotate U15 footprint 180 degrees
Connections:
- net z0: now also U15.12; no longer U15.6
- net z1: now also U15.10; no longer U15.4
- net z2: now also U15.8; no longer U15.2
- net z3: now also U15.6; no longer U15.8
- net at U13.3: now also U15.13; no longer U15.5
- net at U13.6: now also U15.11; no longer U15.3
- net at U13.8: now also U15.9; no longer U15.1
- net at U13.11: now also U15.5; no longer U15.9
Other:
- moved on the sheet: U15A, U15B, U15C, U15D, U15E, U15F
Changed lines of the file:
@@
 L 74xx:74HC14 U15
 U 1 1 5CFF100F
+P 10800 10900
+F 0 "U15" H 10800 11217 50  0000 C CNN
+F 1 "74HC14" H 10800 11126 50  0000 C CNN
+F 2 "Package_DIP:DIP-14_W7.62mm_Socket" H 10800 10900 50  0001 C CNN
+F 3 "http://www.ti.com/lit/gpn/sn74HC14" H 10800 10900 50  0001 C CNN
+	1    10800 10900
+	1    0    0    -1
+$EndComp
+$Comp
+L 74xx:74HC14 U15
+U 4 1 5CFF1021
 P 11100 7300
 F 0 "U15" H 11100 7617 50  0000 C CNN
@@
 F 2 "Package_DIP:DIP-14_W7.62mm_Socket" H 11100 7300 50  0001 C CNN
 F 3 "http://www.ti.com/lit/gpn/sn74HC14" H 11100 7300 50  0001 C CNN
-	1    11100 7300
+	4    11100 7300
 	1    0    0    -1
 $EndComp
 $Comp
 L 74xx:74HC14 U15
-U 2 1 5CFF1015
+U 5 1 5CFF1027
 P 11100 6800
 F 0 "U15" H 11100 7117 50  0000 C CNN
@@
 F 2 "Package_DIP:DIP-14_W7.62mm_Socket" H 11100 6800 50  0001 C CNN
 F 3 "http://www.ti.com/lit/gpn/sn74HC14" H 11100 6800 50  0001 C CNN
-	2    11100 6800
-	1    0    0    -1
-$EndComp
-$Comp
-L 74xx:74HC14 U15
-U 3 1 5CFF101B
-P 11100 6300
-F 0 "U15" H 11100 6617 50  0000 C CNN
-F 1 "74HC14" H 11100 6526 50  0000 C CNN
-F 2 "Package_DIP:DIP-14_W7.62mm_Socket" H 11100 6300 50  0001 C CNN
-F 3 "http://www.ti.com/lit/gpn/sn74HC14" H 11100 6300 50  0001 C CNN
-	3    11100 6300
-	1    0    0    -1
-$EndComp
-$Comp
-L 74xx:74HC14 U15
-U 4 1 5CFF1021
-P 11100 7800
-F 0 "U15" H 11100 8117 50  0000 C CNN
-F 1 "74HC14" H 11100 8026 50  0000 C CNN
-F 2 "Package_DIP:DIP-14_W7.62mm_Socket" H 11100 7800 50  0001 C CNN
-F 3 "http://www.ti.com/lit/gpn/sn74HC14" H 11100 7800 50  0001 C CNN
-	4    11100 7800
-	1    0    0    -1
-$EndComp
-$Comp
-L 74xx:74HC14 U15
-U 5 1 5CFF1027
-P 10800 10400
-F 0 "U15" H 10800 10717 50  0000 C CNN
-F 1 "74HC14" H 10800 10626 50  0000 C CNN
-F 2 "Package_DIP:DIP-14_W7.62mm_Socket" H 10800 10400 50  0001 C CNN
-F 3 "http://www.ti.com/lit/gpn/sn74HC14" H 10800 10400 50  0001 C CNN
-	5    10800 10400
+	5    11100 6800
 	1    0    0    -1
 $EndComp
@@
 L 74xx:74HC14 U15
 U 6 1 5DEEF6B3
-P 10800 10900
-F 0 "U15" H 10800 11217 50  0000 C CNN
-F 1 "74HC14" H 10800 11126 50  0000 C CNN
-F 2 "Package_DIP:DIP-14_W7.62mm_Socket" H 10800 10900 50  0001 C CNN
-F 3 "http://www.ti.com/lit/gpn/sn74HC14" H 10800 10900 50  0001 C CNN
-	6    10800 10900
+P 11100 6300
+F 0 "U15" H 11100 6617 50  0000 C CNN
+F 1 "74HC14" H 11100 6526 50  0000 C CNN
+F 2 "Package_DIP:DIP-14_W7.62mm_Socket" H 11100 6300 50  0001 C CNN
+F 3 "http://www.ti.com/lit/gpn/sn74HC14" H 11100 6300 50  0001 C CNN
+	6    11100 6300
 	1    0    0    -1
 $EndComp
@@
 Wire Bus Line
 	4600 3800 4600 10050
+$Comp
+L 74xx:74HC14 U15
+U 2 1 5CFF1015
+P 10800 10400
+F 0 "U15" H 10800 10717 50  0000 C CNN
+F 1 "74HC14" H 10800 10626 50  0000 C CNN
+F 2 "Package_DIP:DIP-14_W7.62mm_Socket" H 10800 10400 50  0001 C CNN
+F 3 "http://www.ti.com/lit/gpn/sn74HC14" H 10800 10400 50  0001 C CNN
+	2    10800 10400
+	1    0    0    -1
+$EndComp
+$Comp
+L 74xx:74HC14 U15
+U 3 1 5CFF101B
+P 11100 7800
+F 0 "U15" H 11100 8117 50  0000 C CNN
+F 1 "74HC14" H 11100 8026 50  0000 C CNN
+F 2 "Package_DIP:DIP-14_W7.62mm_Socket" H 11100 7800 50  0001 C CNN
+F 3 "http://www.ti.com/lit/gpn/sn74HC14" H 11100 7800 50  0001 C CNN
+	3    11100 7800
+	1    0    0    -1
+$EndComp
 $EndSCHEMATC

Commit message: Rotate U5 footprint 180 degrees
Connections:
- net a0: now also U5.6; no longer U5.11
- net f0: now also U5.9; no longer U5.1
- net f1: now also U5.12; no longer U5.4
- net f6: now also U5.10; no longer U5.2
- net f7: now also U5.13; no longer U5.5
- net usr: now also U5.2; no longer U5.10
- net at U5.3: now also U3.14 (SER); no longer U1.9
- net at U5.8: now also U1.9; no longer U3.14 (SER)
- net at U6.8: now also U5.5; no longer U5.13
- net at U6.11: now also U5.4; no longer U5.12
- new net: U5.1, U5.11
Other:
- moved on the sheet: U5A, U5B, U5C, U5D
Changed lines of the file:
@@
 L 74xx:74HC86 U5
 U 1 1 5CBA3DAB
+P 4900 3050
+F 0 "U5" H 4900 3375 50  0000 C CNN
+F 1 "74HC86" H 4900 3284 50  0000 C CNN
+F 2 "Package_DIP:DIP-14_W7.62mm_Socket" H 4900 3050 50  0001 C CNN
+F 3 "http://www.ti.com/lit/gpn/sn74HC86" H 4900 3050 50  0001 C CNN
+	1    4900 3050
+	1    0    0    -1
+$EndComp
+$Comp
+L 74xx:74HC86 U5
+U 3 1 5CBAF438
 P 4900 2050
-F 0 "U5" H 4900 2375 50  0000 C CNN
-F 1 "74HC86" H 4900 2284 50  0000 C CNN
+F 0 "U5" H 4900 1733 50  0000 C CNN
+F 1 "74HC86" H 4900 1824 50  0000 C CNN
 F 2 "Package_DIP:DIP-14_W7.62mm_Socket" H 4900 2050 50  0001 C CNN
 F 3 "http://www.ti.com/lit/gpn/sn74HC86" H 4900 2050 50  0001 C CNN
-	1    4900 2050
-	1    0    0    -1
-$EndComp
-$Comp
-L 74xx:74HC86 U5
-U 3 1 5CBAF438
-P 4900 3050
-F 0 "U5" H 4900 2733 50  0000 C CNN
-F 1 "74HC86" H 4900 2824 50  0000 C CNN
-F 2 "Package_DIP:DIP-14_W7.62mm_Socket" H 4900 3050 50  0001 C CNN
-F 3 "http://www.ti.com/lit/gpn/sn74HC86" H 4900 3050 50  0001 C CNN
-	3    4900 3050
+	3    4900 2050
 	1    0    0    -1
 $EndComp
@@
 L 74xx:74HC86 U5
 U 2 1 5CBA75FB
-P 4900 2600
-F 0 "U5" H 4900 2925 50  0000 C CNN
-F 1 "74HC86" H 4900 2834 50  0000 C CNN
-F 2 "Package_DIP:DIP-14_W7.62mm_Socket" H 4900 2600 50  0001 C CNN
-F 3 "http://www.ti.com/lit/gpn/sn74HC86" H 4900 2600 50  0001 C CNN
-	2    4900 2600
+P 7600 2150
+F 0 "U5" H 7600 2475 50  0000 C CNN
+F 1 "74HC86" H 7600 2384 50  0000 C CNN
+F 2 "Package_DIP:DIP-14_W7.62mm_Socket" H 7600 2150 50  0001 C CNN
+F 3 "http://www.ti.com/lit/gpn/sn74HC86" H 7600 2150 50  0001 C CNN
+	2    7600 2150
 	1    0    0    -1
 $EndComp
@@
 L 74xx:74HC86 U5
 U 4 1 5D9CE81B
-P 7600 2150
-F 0 "U5" H 7600 2475 50  0000 C CNN
-F 1 "74HC86" H 7600 2384 50  0000 C CNN
-F 2 "Package_DIP:DIP-14_W7.62mm_Socket" H 7600 2150 50  0001 C CNN
-F 3 "http://www.ti.com/lit/gpn/sn74HC86" H 7600 2150 50  0001 C CNN
-	4    7600 2150
-	1    0    0    -1
-$EndComp
+P 4900 2600
+F 0 "U5" H 4900 2925 50  0000 C CNN
+F 1 "74HC86" H 4900 2834 50  0000 C CNN
+F 2 "Package_DIP:DIP-14_W7.62mm_Socket" H 4900 2600 50  0001 C CNN
+F 3 "http://www.ti.com/lit/gpn/sn74HC86" H 4900 2600 50  0001 C CNN
+	4    4900 2600
+	1    0    0    -1
+$EndComp

Commit message: Fix polarity of push buttons
Connections:
- net GND: now also SW2.3 (C), SW3.3 (C); no longer SW2.1 (A), SW3.1 (A)
- net VCC: now also SW2.1 (A), SW3.1 (A); no longer SW2.3 (C), SW3.3 (C)
Changed lines of the file:
@@
 L power:GND #PWR08
 U 1 1 5CC74554
-P 950 3300
-F 0 "#PWR08" H 950 3050 50  0001 C CNN
-F 1 "GND" V 955 3172 50  0000 R CNN
-F 2 "" H 950 3300 50  0001 C CNN
-F 3 "" H 950 3300 50  0001 C CNN
-	1    950  3300
+P 950 3500
+F 0 "#PWR08" H 950 3250 50  0001 C CNN
+F 1 "GND" V 955 3372 50  0000 R CNN
+F 2 "" H 950 3500 50  0001 C CNN
+F 3 "" H 950 3500 50  0001 C CNN
+	1    950  3500
 	0    1    1    0
 $EndComp
@@
 L power:GND #PWR011
 U 1 1 5CC7D179
-P 950 4600
-F 0 "#PWR011" H 950 4350 50  0001 C CNN
-F 1 "GND" V 955 4472 50  0000 R CNN
-F 2 "" H 950 4600 50  0001 C CNN
-F 3 "" H 950 4600 50  0001 C CNN
-	1    950  4600
+P 950 4800
+F 0 "#PWR011" H 950 4550 50  0001 C CNN
+F 1 "GND" V 955 4672 50  0000 R CNN
+F 2 "" H 950 4800 50  0001 C CNN
+F 3 "" H 950 4800 50  0001 C CNN
+	1    950  4800
 	0    1    1    0
 $EndComp
@@
 L power:VCC #PWR012
 U 1 1 5D05C98D
-P 950 4800
-F 0 "#PWR012" H 950 4650 50  0001 C CNN
-F 1 "VCC" V 968 4927 50  0000 L CNN
-F 2 "" H 950 4800 50  0001 C CNN
-F 3 "" H 950 4800 50  0001 C CNN
-	1    950  4800
+P 950 4600
+F 0 "#PWR012" H 950 4450 50  0001 C CNN
+F 1 "VCC" V 968 4727 50  0000 L CNN
+F 2 "" H 950 4600 50  0001 C CNN
+F 3 "" H 950 4600 50  0001 C CNN
+	1    950  4600
 	0    -1   -1   0
 $EndComp
@@
 L power:VCC #PWR09
 U 1 1 5D05D785
-P 950 3500
-F 0 "#PWR09" H 950 3350 50  0001 C CNN
-F 1 "VCC" V 968 3627 50  0000 L CNN
-F 2 "" H 950 3500 50  0001 C CNN
-F 3 "" H 950 3500 50  0001 C CNN
-	1    950  3500
+P 950 3300
+F 0 "#PWR09" H 950 3150 50  0001 C CNN
+F 1 "VCC" V 968 3427 50  0000 L CNN
+F 2 "" H 950 3300 50  0001 C CNN
+F 3 "" H 950 3300 50  0001 C CNN
+	1    950  3300
 	0    -1   -1   0
 $EndComp
