File: midnight-sun-2019/midnight-sun-2019.sch (KiCad schematic (older format))
At the start: 73 parts, among them J1 Conn_02x02_Odd_Even, J2 USB_B_Micro, SW1 SW_SPDT, SW2 SW_SPDT, SW3 SW_SPDT, U1 74HC14, U10 74HC14, U11 74HC86, U12 74HC86, U13 74HC86, U14 74HC86, U15 74HC14, U16 74HC14, U2 74HC595, U3 74HC595, U4 74HC595, U5 74HC86, U6 74HC86, U7 74HC86, U8 74HC86, U9 74HC14

Commit message: Fix polarity of SW3
Connections:
- net GND: now also SW3.1 (A); no longer SW3.3 (C)
- net VCC: now also SW3.3 (C); no longer SW3.1 (A)
Changed lines of the file:
@@
 L power:GND #PWR011
 U 1 1 5CC7D179
-P 950 4800
-F 0 "#PWR011" H 950 4550 50  0001 C CNN
-F 1 "GND" V 955 4672 50  0000 R CNN
-F 2 "" H 950 4800 50  0001 C CNN
-F 3 "" H 950 4800 50  0001 C CNN
-	1    950  4800
+P 950 4600
+F 0 "#PWR011" H 950 4350 50  0001 C CNN
+F 1 "GND" V 955 4472 50  0000 R CNN
+F 2 "" H 950 4600 50  0001 C CNN
+F 3 "" H 950 4600 50  0001 C CNN
+	1    950  4600
 	0    1    1    0
 $EndComp
@@
 L power:VCC #PWR012
 U 1 1 5D05C98D
-P 950 4600
-F 0 "#PWR012" H 950 4450 50  0001 C CNN
-F 1 "VCC" V 968 4727 50  0000 L CNN
-F 2 "" H 950 4600 50  0001 C CNN
-F 3 "" H 950 4600 50  0001 C CNN
-	1    950  4600
+P 950 4800
+F 0 "#PWR012" H 950 4650 50  0001 C CNN
+F 1 "VCC" V 968 4927 50  0000 L CNN
+F 2 "" H 950 4800 50  0001 C CNN
+F 3 "" H 950 4800 50  0001 C CNN
+	1    950  4800
 	0    -1   -1   0
 $EndComp
@@
 NoConn ~ 12550 8800
 NoConn ~ 12550 8350
-Wire Wire Line
-	6450 9800 7300 9800
-Wire Wire Line
-	6450 9300 7300 9300
-Wire Wire Line
-	6450 8800 7300 8800
-Wire Wire Line
-	6450 8300 7300 8300
-Wire Wire Line
-	6450 7800 7300 7800
-Wire Wire Line
-	6450 6800 7300 6800
-Wire Wire Line
-	6450 7300 7300 7300
-Wire Wire Line
-	6450 6300 7300 6300
-Wire Bus Line
-	9200 2250 9200 5450
-Wire Bus Line
-	9800 2250 9800 2450
-Wire Bus Line
-	11050 2850 11050 3550
-Wire Bus Line
-	6350 1150 6350 3800
-Wire Bus Line
-	9650 5800 9650 9900
-Wire Bus Line
-	11500 3550 11500 9900
-Wire Bus Line
-	11050 3750 11050 5800
-Wire Bus Line
-	4300 3800 4300 6150
-Wire Bus Line
-	7050 6400 7050 11100
-Wire Bus Line
-	8750 6100 8750 10050
-Wire Bus Line
-	10000 6100 10000 10050
-Wire Bus Line
-	6350 3800 6350 10800
-Wire Bus Line
-	8100 5650 8100 11000
-Wire Bus Line
-	9800 2650 9800 5650
-Wire Bus Line
-	4600 3800 4600 10050
 $Comp
 L 74xx:74HC14 U15
@@
 	1    0    0    -1
 $EndComp
+Wire Wire Line
+	6450 9800 7300 9800
+Wire Wire Line
+	6450 9300 7300 9300
+Wire Wire Line
+	6450 8800 7300 8800
+Wire Wire Line
+	6450 8300 7300 8300
+Wire Wire Line
+	6450 7800 7300 7800
+Wire Wire Line
+	6450 6800 7300 6800
+Wire Wire Line
+	6450 7300 7300 7300
+Wire Wire Line
+	6450 6300 7300 6300
+Wire Bus Line
+	9200 2250 9200 5450
+Wire Bus Line
+	9800 2250 9800 2450
+Wire Bus Line
+	11050 2850 11050 3550
+Wire Bus Line
+	6350 1150 6350 3800
+Wire Bus Line
+	9650 5800 9650 9900
+Wire Bus Line
+	11500 3550 11500 9900
+Wire Bus Line
+	11050 3750 11050 5800
+Wire Bus Line
+	4300 3800 4300 6150
+Wire Bus Line
+	8750 6100 8750 10050
+Wire Bus Line
+	10000 6100 10000 10050
+Wire Bus Line
+	6350 3800 6350 10800
+Wire Bus Line
+	8100 5650 8100 11000
+Wire Bus Line
+	9800 2650 9800 5650
+Wire Bus Line
+	4600 3800 4600 10050
+Wire Bus Line
+	7050 6400 7050 11100
 $EndSCHEMATC
